File: hdw/Analog_Clock/Meter1.sch (KiCad schematic (older format))
At the start: 0 parts

Commit message: big sch push
Parts:
- added C1901, C1902, C1906, C1907, C1908, C1911, C1912: 0.1uF, Capacitors_SMD:C_0603, symbol Custom_Library:C_Custom
- added C1903, C1904: 4.7uF, Capacitors_SMD:C_0805, symbol Custom_Library:C_Custom
- added C1905: 47pF, Capacitors_SMD:C_0603, symbol Custom_Library:C_Custom
- added C1909: 10nF, Capacitors_SMD:C_0603, symbol Custom_Library:C_Custom
- added C1910: 1nF, Capacitors_SMD:C_0603, symbol Custom_Library:C_Custom
- added D1901: Green, LEDs:LED_0603, symbol Device:LED
- added D1902: ASMB-MTB0-0A3A2, LED_SMD:LED_Avago_PLCC4_3.2x2.8mm_CW, symbol LED:ASMB-MTB0-0A3A2
- added D1903: BZX384-B3V3,115, Diode_SMD:D_SOD-323, symbol Diode:DZ2S033X0L
- added L1901: 600R 0.5A, Inductors_SMD:L_0603, symbol Device:Ferrite_Bead
- added MES1901: Voltmeter_DC, symbol Device:Voltmeter_DC
- added MK1901, MK1902, MK1905, MK1906, MK1907, MK1908, MK1911, MK1912: #4-40 Screw, symbol Custom_Library:Screw
- added MK1903, MK1904, MK1909, MK1910: #4-40 Standoff, symbol Custom_Library:Standoff
- added R1901, R1902, R1903: 10, Resistors_SMD:R_0603, symbol Custom_Library:R_Custom
- added R1904, R1905, R1907: 10k, Resistors_SMD:R_0603, symbol Custom_Library:R_Custom
- added R1906, R1912: 1k, Resistors_SMD:R_0603, symbol Custom_Library:R_Custom
- added R1908, R1909: 1.01k, Resistors_SMD:R_0603, symbol Custom_Library:R_Custom
- added R1910, R1911: 9.09k, Resistors_SMD:R_0603, symbol Custom_Library:R_Custom
- added TP1901: TP_Pad, Custom Footprints Library:Test_Point, symbol Custom_Library:TP_Pad
- added U1901: 74LVC1G07, TO_SOT_Packages_SMD:SOT-353_SC-70-5, symbol Custom_Library:74LVC1G07_Power
- added U1902: LT1790-2.048, Package_TO_SOT_SMD:TSOT-23-6, symbol Reference_Voltage:LT1790-2.048
- added U1903: DAC8551, Package_SO:VSSOP-8_3.0x3.0mm_P0.65mm, symbol Custom_Library:DAC8551
- added U1904: OPA2197xDGK, Package_SO:VSSOP-8_3.0x3.0mm_P0.65mm, symbol Amplifier_Operational:OPA2197xDGK
Connections:
- new net: R1903.2, R1907.1, U1903.6 (SCLK)
- new net: R1902.2, R1905.1, U1903.7 (DIN)
- new net: C1904.1, C1906.1, L1901.1, U1903.1 (VDD)
- new net: C1911.1, MES1901.2 (+), R1910.1, R1911.1, U1904.1
- new net: C1907.1, R1908.1, R1910.2, U1904.5 (+)
- new net: U1903.3 (VFB), U1903.4 (VOUT), U1904.3 (+)
- new net: R1901.2, R1904.2, U1903.5 (~SYNC)
- new net: C1911.2, R1909.1, R1911.2, U1904.2 (-)
- new net: R1912.2, U1904.6 (-), U1904.7
- new net: D1901.1 (K), U1901.4
- new net: D1901.2 (A), R1906.2
- new net +20V: C1908.1, C1909.1, C1910.1, U1904.8 (V+)
- new net +3V3: C1901.1, C1902.1, D1902.1 (A), L1901.2, R1904.1, R1906.1, U1901.5 (VCC), U1902.4 (Vin)
- new net DAC1_VREF: C1903.1, C1905.1, TP1901.1 (TP), U1902.6 (Vout), U1903.2 (VREF)
- new net DAC_SPI_MOSI: R1902.1
- new net DAC_SPI_SCLK: R1903.1
- new net GND: C1901.2, C1902.2, C1903.2, C1904.2, C1905.2, C1906.2, C1907.2, C1908.2, C1909.2, C1910.2, C1912.2, D1903.2 (A), MES1901.1 (-), R1905.2, R1907.2, R1908.2, R1909.2, U1901.3 (GND), U1902.1 (GND), U1902.2 (GND), U1903.8 (GND), U1903.9 (GND), U1904.4 (V-)
- new net METER1_LED_B: D1902.2 (BK)
- new net METER1_LED_G: D1902.3 (GK)
- new net METER1_LED_R: D1902.4 (RK)
- new net VDAC_1_ADC: C1912.1, D1903.1 (K), R1912.1
- new net ~DAC_SPI_SYNC_1: R1901.1, U1901.2
Other:
- note added: "15V Full Scale"
- note added: "Gain = 0.1 V/V"
- note added: "Gain = 10 V/V"

Commit message: Much more schematic progress
Parts:
- MES1901: footprint (none) -> FIX ME
- R1901, R1902, R1903, R1904, R1905, R1907: Digi-Key PN (none) -> YAG2321CT-ND
- R1906, R1912: Digi-Key PN (none) -> 311-1.00KHRCT-ND
- R1908, R1909: Digi-Key PN (none) -> YAG4489CT-ND
- R1910, R1911: Digi-Key PN PN -> YAG1755CT-ND
Changed lines of the file:
@@
 encoding utf-8
 Sheet 19 25
-Title ""
-Date ""
-Rev ""
-Comp ""
+Title "Analog Clock"
+Date "2020-08-15"
+Rev "A"
+Comp "Drew Maatman"
 Comment1 ""
 Comment2 ""
@@
 F 5 "1%" V 2530 3680 50  0001 C CNN "Tolerance"
 F 6 "1/10W" V 2630 3680 50  0001 C CNN "Wattage"
+F 7 "YAG2321CT-ND" H 2330 3680 50  0001 C CNN "Digi-Key PN"
 	1    2330 3680
 	0    -1   1    0
@@
 F 5 "1%" V 2530 3580 50  0001 C CNN "Tolerance"
 F 6 "1/10W" V 2630 3580 50  0001 C CNN "Wattage"
+F 7 "YAG2321CT-ND" H 2330 3580 50  0001 C CNN "Digi-Key PN"
 	1    2330 3580
 	0    -1   1    0
@@
 F 5 "1%" V 2530 3480 50  0001 C CNN "Tolerance"
 F 6 "1/10W" V 2630 3480 50  0001 C CNN "Wattage"
+F 7 "YAG2321CT-ND" H 2330 3480 50  0001 C CNN "Digi-Key PN"
 	1    2330 3480
 	0    -1   1    0
@@
 F 5 "1%" H 2930 3250 50  0000 L CNN "Tolerance"
 F 6 "1/10W" H 2940 3170 50  0000 L CNN "Wattage"
-F 7 "" H 3130 3650 60  0001 C CNN "Digi-Key PN"
+F 7 "YAG2321CT-ND" H 3130 3650 60  0001 C CNN "Digi-Key PN"
 	1    2830 3250
 	1    0    0    -1
@@
 F 5 "1%" H 3670 3910 50  0000 L CNN "Tolerance"
 F 6 "1/10W" H 3680 3830 50  0000 L CNN "Wattage"
-F 7 "" H 3870 4310 60  0001 C CNN "Digi-Key PN"
+F 7 "YAG2321CT-ND" H 3870 4310 60  0001 C CNN "Digi-Key PN"
 	1    3570 3910
 	1    0    0    -1
@@
 F 5 "1%" H 2930 3910 50  0000 L CNN "Tolerance"
 F 6 "1/10W" H 2940 3830 50  0000 L CNN "Wattage"
-F 7 "" H 3130 4310 60  0001 C CNN "Digi-Key PN"
+F 7 "YAG2321CT-ND" H 3130 4310 60  0001 C CNN "Digi-Key PN"
 	1    2830 3910
 	1    0    0    -1
@@
 F 5 "0.1%" V 7110 2630 50  0000 C CNN "Tolerance"
 F 6 "1/10W" V 7210 2630 50  0000 C CNN "Wattage"
-F 7 "PN" H 7210 3030 60  0001 C CNN "Digi-Key PN"
+F 7 "YAG1755CT-ND" H 7210 3030 60  0001 C CNN "Digi-Key PN"
 	1    6910 2630
 	0    1    -1   0
@@
 F 5 "0.1%" H 6200 3210 50  0000 L CNN "Tolerance"
 F 6 "1/10W" H 6210 3130 50  0000 L CNN "Wattage"
+F 7 "YAG4489CT-ND" H 6100 3210 50  0001 C CNN "Digi-Key PN"
 	1    6100 3210
 	1    0    0    -1
@@
 F 5 "1%" V 7570 4510 50  0000 C CNN "Tolerance"
 F 6 "1/10W" V 7670 4510 50  0000 C CNN "Wattage"
-F 7 "" H 7670 4910 60  0001 C CNN "Digi-Key PN"
+F 7 "311-1.00KHRCT-ND" H 7670 4910 60  0001 C CNN "Digi-Key PN"
 	1    7370 4510
 	0    1    1    0
@@
 F 0 "MES1901" H 8270 2270 50  0000 R CNN
 F 1 "Voltmeter_DC" H 8270 2200 50  0000 R CNN
-F 2 "" V 8400 2330 50  0001 C CNN
+F 2 "FIX ME" V 8400 2330 50  0001 C CNN
 F 3 "~" V 8400 2330 50  0001 C CNN
 	1    8400 2230
@@
 F 5 "0.1%" H 5770 4740 50  0000 L CNN "Tolerance"
 F 6 "1/10W" H 5780 4660 50  0000 L CNN "Wattage"
+F 7 "YAG4489CT-ND" H 5670 4740 50  0001 C CNN "Digi-Key PN"
 	1    5670 4740
 	1    0    0    -1
@@
 F 5 "0.1%" V 6730 4020 50  0000 C CNN "Tolerance"
 F 6 "1/10W" V 6830 4020 50  0000 C CNN "Wattage"
-F 7 "PN" H 6830 4420 60  0001 C CNN "Digi-Key PN"
+F 7 "YAG1755CT-ND" H 6830 4420 60  0001 C CNN "Digi-Key PN"
 	1    6530 4020
 	0    1    -1   0
@@
 F 5 "1%" H 2960 5880 50  0000 L CNN "Tolerance"
 F 6 "1/10W" H 2960 5810 50  0000 L CNN "Wattage"
-F 7 "" H 3190 6280 60  0001 C CNN "Digi-Key PN"
+F 7 "311-1.00KHRCT-ND" H 3190 6280 60  0001 C CNN "Digi-Key PN"
 	1    2890 5880
 	-1   0    0    -1

Commit message: made netlist, started PCB
Parts:
- MES1901: footprint FIX ME -> (none)
Changed lines of the file:
@@
 F 0 "MES1901" H 8270 2270 50  0000 R CNN
 F 1 "Voltmeter_DC" H 8270 2200 50  0000 R CNN
-F 2 "FIX ME" V 8400 2330 50  0001 C CNN
+F 2 "" V 8400 2330 50  0001 C CNN
 F 3 "~" V 8400 2330 50  0001 C CNN
 	1    8400 2230

Commit message: more PCB grouping
Parts:
- MES1901: footprint (none) -> Custom Footprints Library:SO-45_Panel_Meter
Changed lines of the file:
@@
 F 0 "MES1901" H 8270 2270 50  0000 R CNN
 F 1 "Voltmeter_DC" H 8270 2200 50  0000 R CNN
-F 2 "" V 8400 2330 50  0001 C CNN
+F 2 "Custom Footprints Library:SO-45_Panel_Meter" V 8400 2330 50  0001 C CNN
 F 3 "~" V 8400 2330 50  0001 C CNN
 	1    8400 2230
