File: hdw/Analog_Clock/Meter1.sch (KiCad schematic (older format))
At the start: 46 parts, among them U1901 74LVC1G07, U1902 LT1790-2.048, U1903 DAC8551, U1904 OPA2197xDGK

Commit message: Major USB restructuring
Parts:
- U1904: symbol Amplifier_Operational:OPA2197xDGK -> Custom_Library:OPA2197xDGK
Changed lines of the file:
@@
 $Descr A 11000 8500
 encoding utf-8
-Sheet 19 24
+Sheet 15 25
 Title "Analog Clock"
 Date "2020-08-15"
@@
 Connection ~ 6100 2630
 $Comp
-L Amplifier_Operational:OPA2197xDGK U1904
+L Custom_Library:OPA2197xDGK U1904
 U 1 1 5F4617C5
 P 6480 1950
@@
 $EndComp
 $Comp
-L Amplifier_Operational:OPA2197xDGK U1904
+L Custom_Library:OPA2197xDGK U1904
 U 3 1 5F4617C8
 P 6480 1950
@@
 $EndComp
 $Comp
-L Amplifier_Operational:OPA2197xDGK U1904
+L Custom_Library:OPA2197xDGK U1904
 U 2 1 5F4617CA
 P 6480 4510
