File: hdw/Analog_Clock/Meter2.sch (KiCad schematic (older format))
At the start: 0 parts

Commit message: big sch push
Parts:
- added C2001, C2002, C2006, C2007, C2008, C2011, C2012: 0.1uF, Capacitors_SMD:C_0603, symbol Custom_Library:C_Custom
- added C2003, C2004: 4.7uF, Capacitors_SMD:C_0805, symbol Custom_Library:C_Custom
- added C2005: 47pF, Capacitors_SMD:C_0603, symbol Custom_Library:C_Custom
- added C2009: 10nF, Capacitors_SMD:C_0603, symbol Custom_Library:C_Custom
- added C2010: 1nF, Capacitors_SMD:C_0603, symbol Custom_Library:C_Custom
- added D2001: Green, LEDs:LED_0603, symbol Device:LED
- added D2002: ASMB-MTB0-0A3A2, LED_SMD:LED_Avago_PLCC4_3.2x2.8mm_CW, symbol LED:ASMB-MTB0-0A3A2
- added D2003: BZX384-B3V3,115, Diode_SMD:D_SOD-323, symbol Diode:DZ2S033X0L
- added L2001: 600R 0.5A, Inductors_SMD:L_0603, symbol Device:Ferrite_Bead
- added MES2001: Voltmeter_DC, symbol Device:Voltmeter_DC
- added MK2001, MK2002, MK2005, MK2006, MK2007, MK2008, MK2011, MK2012: #4-40 Screw, symbol Custom_Library:Screw
- added MK2003, MK2004, MK2009, MK2010: #4-40 Standoff, symbol Custom_Library:Standoff
- added R2001, R2002, R2003: 10, Resistors_SMD:R_0603, symbol Custom_Library:R_Custom
- added R2004, R2005, R2007: 10k, Resistors_SMD:R_0603, symbol Custom_Library:R_Custom
- added R2006, R2012: 1k, Resistors_SMD:R_0603, symbol Custom_Library:R_Custom
- added R2008, R2009: 1.01k, Resistors_SMD:R_0603, symbol Custom_Library:R_Custom
- added R2010, R2011: 9.09k, Resistors_SMD:R_0603, symbol Custom_Library:R_Custom
- added TP2001: TP_Pad, Custom Footprints Library:Test_Point, symbol Custom_Library:TP_Pad
- added U2001: 74LVC1G07, TO_SOT_Packages_SMD:SOT-353_SC-70-5, symbol Custom_Library:74LVC1G07_Power
- added U2002: LT1790-2.048, Package_TO_SOT_SMD:TSOT-23-6, symbol Reference_Voltage:LT1790-2.048
- added U2003: DAC8551, Package_SO:VSSOP-8_3.0x3.0mm_P0.65mm, symbol Custom_Library:DAC8551
- added U2004: OPA2197xDGK, Package_SO:VSSOP-8_3.0x3.0mm_P0.65mm, symbol Amplifier_Operational:OPA2197xDGK
Connections:
- new net: C2004.1, C2006.1, L2001.1, U2003.1 (VDD)
- new net: U2003.3 (VFB), U2003.4 (VOUT), U2004.3 (+)
- new net: R2001.2, R2004.2, U2003.5 (~SYNC)
- new net: R2003.2, R2007.1, U2003.6 (SCLK)
- new net: R2002.2, R2005.1, U2003.7 (DIN)
- new net: C2011.1, MES2001.2 (+), R2010.1, R2011.1, U2004.1
- new net: C2011.2, R2009.1, R2011.2, U2004.2 (-)
- new net: C2007.1, R2008.1, R2010.2, U2004.5 (+)
- new net: R2012.2, U2004.6 (-), U2004.7
- new net: D2001.2 (A), R2006.2
- new net: D2001.1 (K), U2001.4
- new net +20V: C2008.1, C2009.1, C2010.1, U2004.8 (V+)
- new net +3V3: C2001.1, C2002.1, D2002.1 (A), L2001.2, R2004.1, R2006.1, U2001.5 (VCC), U2002.4 (Vin)
- new net DAC2_VREF: C2003.1, C2005.1, TP2001.1 (TP), U2002.6 (Vout), U2003.2 (VREF)
- new net DAC_SPI_MOSI: R2002.1
- new net DAC_SPI_SCLK: R2003.1
- new net GND: C2001.2, C2002.2, C2003.2, C2004.2, C2005.2, C2006.2, C2007.2, C2008.2, C2009.2, C2010.2, C2012.2, D2003.2 (A), MES2001.1 (-), R2005.2, R2007.2, R2008.2, R2009.2, U2001.3 (GND), U2002.1 (GND), U2002.2 (GND), U2003.8 (GND), U2003.9 (GND), U2004.4 (V-)
- new net METER2_LED_B: D2002.2 (BK)
- new net METER2_LED_G: D2002.3 (GK)
- new net METER2_LED_R: D2002.4 (RK)
- new net VDAC_2_ADC: C2012.1, D2003.1 (K), R2012.1
- new net ~DAC_SPI_SYNC_2: R2001.1, U2001.2
Other:
- note added: "15V Full Scale"
- note added: "Gain = 0.1 V/V"
- note added: "Gain = 10 V/V"

Commit message: Much more schematic progress
Parts:
- MES2001: footprint (none) -> FIX ME
- R2001, R2002, R2003, R2004, R2005, R2007: Digi-Key PN (none) -> YAG2321CT-ND
- R2006, R2012: Digi-Key PN (none) -> 311-1.00KHRCT-ND
- R2008, R2009: Digi-Key PN (none) -> YAG4489CT-ND
- R2010, R2011: Digi-Key PN PN -> YAG1755CT-ND
Changed lines of the file:
@@
 encoding utf-8
 Sheet 20 25
-Title ""
-Date ""
-Rev ""
-Comp ""
+Title "Analog Clock"
+Date "2020-08-15"
+Rev "A"
+Comp "Drew Maatman"
 Comment1 ""
 Comment2 ""
@@
 F 5 "1%" V 2530 3680 50  0001 C CNN "Tolerance"
 F 6 "1/10W" V 2630 3680 50  0001 C CNN "Wattage"
+F 7 "YAG2321CT-ND" H 2330 3680 50  0001 C CNN "Digi-Key PN"
 	1    2330 3680
 	0    -1   1    0
@@
 F 5 "1%" V 2530 3580 50  0001 C CNN "Tolerance"
 F 6 "1/10W" V 2630 3580 50  0001 C CNN "Wattage"
+F 7 "YAG2321CT-ND" H 2330 3580 50  0001 C CNN "Digi-Key PN"
 	1    2330 3580
 	0    -1   1    0
@@
 F 5 "1%" V 2530 3480 50  0001 C CNN "Tolerance"
 F 6 "1/10W" V 2630 3480 50  0001 C CNN "Wattage"
+F 7 "YAG2321CT-ND" H 2330 3480 50  0001 C CNN "Digi-Key PN"
 	1    2330 3480
 	0    -1   1    0
@@
 F 5 "1%" H 2930 3250 50  0000 L CNN "Tolerance"
 F 6 "1/10W" H 2940 3170 50  0000 L CNN "Wattage"
-F 7 "" H 3130 3650 60  0001 C CNN "Digi-Key PN"
+F 7 "YAG2321CT-ND" H 3130 3650 60  0001 C CNN "Digi-Key PN"
 	1    2830 3250
 	1    0    0    -1
@@
 F 5 "1%" H 3670 3910 50  0000 L CNN "Tolerance"
 F 6 "1/10W" H 3680 3830 50  0000 L CNN "Wattage"
-F 7 "" H 3870 4310 60  0001 C CNN "Digi-Key PN"
+F 7 "YAG2321CT-ND" H 3870 4310 60  0001 C CNN "Digi-Key PN"
 	1    3570 3910
 	1    0    0    -1
@@
 F 5 "1%" H 2930 3910 50  0000 L CNN "Tolerance"
 F 6 "1/10W" H 2940 3830 50  0000 L CNN "Wattage"
-F 7 "" H 3130 4310 60  0001 C CNN "Digi-Key PN"
+F 7 "YAG2321CT-ND" H 3130 4310 60  0001 C CNN "Digi-Key PN"
 	1    2830 3910
 	1    0    0    -1
@@
 F 5 "0.1%" V 7110 2630 50  0000 C CNN "Tolerance"
 F 6 "1/10W" V 7210 2630 50  0000 C CNN "Wattage"
-F 7 "PN" H 7210 3030 60  0001 C CNN "Digi-Key PN"
+F 7 "YAG1755CT-ND" H 7210 3030 60  0001 C CNN "Digi-Key PN"
 	1    6910 2630
 	0    1    -1   0
@@
 F 5 "0.1%" H 6200 3210 50  0000 L CNN "Tolerance"
 F 6 "1/10W" H 6210 3130 50  0000 L CNN "Wattage"
+F 7 "YAG4489CT-ND" H 6100 3210 50  0001 C CNN "Digi-Key PN"
 	1    6100 3210
 	1    0    0    -1
@@
 F 5 "1%" V 7570 4510 50  0000 C CNN "Tolerance"
 F 6 "1/10W" V 7670 4510 50  0000 C CNN "Wattage"
-F 7 "" H 7670 4910 60  0001 C CNN "Digi-Key PN"
+F 7 "311-1.00KHRCT-ND" H 7670 4910 60  0001 C CNN "Digi-Key PN"
 	1    7370 4510
 	0    1    1    0
@@
 F 0 "MES2001" H 8270 2270 50  0000 R CNN
 F 1 "Voltmeter_DC" H 8270 2200 50  0000 R CNN
-F 2 "" V 8400 2330 50  0001 C CNN
+F 2 "FIX ME" V 8400 2330 50  0001 C CNN
 F 3 "~" V 8400 2330 50  0001 C CNN
 	1    8400 2230
@@
 F 5 "0.1%" H 5770 4740 50  0000 L CNN "Tolerance"
 F 6 "1/10W" H 5780 4660 50  0000 L CNN "Wattage"
+F 7 "YAG4489CT-ND" H 5670 4740 50  0001 C CNN "Digi-Key PN"
 	1    5670 4740
 	1    0    0    -1
@@
 F 5 "0.1%" V 6730 4020 50  0000 C CNN "Tolerance"
 F 6 "1/10W" V 6830 4020 50  0000 C CNN "Wattage"
-F 7 "PN" H 6830 4420 60  0001 C CNN "Digi-Key PN"
+F 7 "YAG1755CT-ND" H 6830 4420 60  0001 C CNN "Digi-Key PN"
 	1    6530 4020
 	0    1    -1   0
@@
 F 5 "1%" H 2960 5880 50  0000 L CNN "Tolerance"
 F 6 "1/10W" H 2960 5810 50  0000 L CNN "Wattage"
-F 7 "" H 3190 6280 60  0001 C CNN "Digi-Key PN"
+F 7 "311-1.00KHRCT-ND" H 3190 6280 60  0001 C CNN "Digi-Key PN"
 	1    2890 5880
 	-1   0    0    -1

Commit message: made netlist, started PCB
Parts:
- MES2001: footprint FIX ME -> (none)
Changed lines of the file:
@@
 F 0 "MES2001" H 8270 2270 50  0000 R CNN
 F 1 "Voltmeter_DC" H 8270 2200 50  0000 R CNN
-F 2 "FIX ME" V 8400 2330 50  0001 C CNN
+F 2 "" V 8400 2330 50  0001 C CNN
 F 3 "~" V 8400 2330 50  0001 C CNN
 	1    8400 2230

Commit message: more PCB grouping
Parts:
- MES2001: footprint (none) -> Custom Footprints Library:SO-45_Panel_Meter
Changed lines of the file:
@@
 F 0 "MES2001" H 8270 2270 50  0000 R CNN
 F 1 "Voltmeter_DC" H 8270 2200 50  0000 R CNN
-F 2 "" V 8400 2330 50  0001 C CNN
+F 2 "Custom Footprints Library:SO-45_Panel_Meter" V 8400 2330 50  0001 C CNN
 F 3 "~" V 8400 2330 50  0001 C CNN
 	1    8400 2230
