File: hdw/Analog_Clock/Meter2.sch (KiCad schematic (older format))
At the start: 46 parts, among them U2001 74LVC1G07, U2002 LT1790-2.048, U2003 DAC8551, U2004 OPA2197xDGK

Commit message: Major USB restructuring
Parts:
- U2004: symbol Amplifier_Operational:OPA2197xDGK -> Custom_Library:OPA2197xDGK
Changed lines of the file:
@@
 $Descr A 11000 8500
 encoding utf-8
-Sheet 20 24
+Sheet 16 25
 Title "Analog Clock"
 Date "2020-08-15"
@@
 Connection ~ 6100 2630
 $Comp
-L Amplifier_Operational:OPA2197xDGK U2004
+L Custom_Library:OPA2197xDGK U2004
 U 1 1 5EA45E04
 P 6480 1950
@@
 $EndComp
 $Comp
-L Amplifier_Operational:OPA2197xDGK U2004
+L Custom_Library:OPA2197xDGK U2004
 U 3 1 5EA4657D
 P 6480 1950
@@
 $EndComp
 $Comp
-L Amplifier_Operational:OPA2197xDGK U2004
+L Custom_Library:OPA2197xDGK U2004
 U 2 1 5EA49816
 P 6480 4510
