File: hdw/Analog_Clock/PIC32MZ_Bypass.sch (KiCad schematic (older format))
At the start: 24 parts

Commit message: a few sch adjustments
Parts:
- removed C? (x2): 0.1uF, Capacitors_SMD:C_0402, symbol Custom_Library:C_Custom
- removed C? (x2): 1nF, Capacitors_SMD:C_0402, symbol Custom_Library:C_Custom
- removed C? (x2): 10nF, Capacitors_SMD:C_0402, symbol Custom_Library:C_Custom
- removed C?: 22uF, Capacitors_SMD:C_1206, symbol Custom_Library:C_Custom
- added C? (x2): 0.1uF, Capacitors_SMD:C_0402, symbol Custom_Library:C_Custom
- added C? (x2): 1nF, Capacitors_SMD:C_0402, symbol Custom_Library:C_Custom
- added C? (x2): 10nF, Capacitors_SMD:C_0402, symbol Custom_Library:C_Custom
Connections:
- net +3.3VA_MZ: now also C?.1, C?.1, C?.1
- net +3V3: now also C?.1, C?.1, C?.1
- net GND: now also C?.2, C?.2, C?.2
- net GNDA_MZ: now also C?.2, C?.2, C?.2

Commit message: big sch push
Parts:
- C901, C902, C908, C912, C916, C917: renamed from C?; footprint Capacitors_SMD:C_0402 -> Capacitors_SMD:C_0603; Digi-Key PN 490-10701-1-ND -> 399-7845-1-ND; display_footprint 0402 -> 0603
- C903, C909, C913: renamed from C?; footprint Capacitors_SMD:C_0402 -> Capacitors_SMD:C_0603; Digi-Key PN 490-13211-1-ND -> 490-10474-1-ND; Voltage 6.3V -> 10V; display_footprint 0402 -> 0603
- C904, C905, C910, C914, C918, C919: renamed from C?; footprint Capacitors_SMD:C_0402 -> Capacitors_SMD:C_0603; Digi-Key PN 490-13295-1-ND -> 399-7842-1-ND; display_footprint 0402 -> 0603
- C906, C907, C911, C915, C920, C921: renamed from C?; footprint Capacitors_SMD:C_0402 -> Capacitors_SMD:C_0603; Digi-Key PN 399-1032-1-ND -> 399-1083-1-ND; display_footprint 0402 -> 0603
- L901, L902: renamed from L?; footprint Inductors_SMD:L_0402 -> Inductors_SMD:L_0603; Digi-Key PN 490-5441-1-ND -> 732-1593-1-ND
