File: hdw/Analog_Clock/POS12_Telemetry.sch (KiCad schematic (older format))
At the start: 7 parts

Commit message: a few sch adjustments
Parts:
- C? (x3): display_footprint 0402 -> (none)
- DOC?: value jahjahdslkjfhdsaf -> 0x40
- DOC?: value lkjasflkjasdf -> 0x18
- U? (x2): Configuration (none) -> Telemetry
Connections:
- net GND: now also U?.5 (A2), U?.6 (A1), U?.7 (A0), U?.7 (A0), U?.8 (A1)
Changed lines of the file:
@@
 encoding utf-8
 Sheet 3 20
-Title ""
-Date ""
-Rev ""
-Comp ""
+Title "Pulse Oximeter"
+Date "2020-08-01"
+Rev "A"
+Comp "Drew Maatman"
 Comment1 ""
 Comment2 ""
@@
 AR Path="/5E0A0E29/5E0ACFF2" Ref="#PWR?"  Part="1"
 AR Path="/5E052856/5E0ACFF2" Ref="#PWR?"  Part="1"
+AR Path="/5EAE2D84/5E0ACFF2" Ref="#PWR?"  Part="1"
 AR Path="/5E939D24/5E0ACFF2" Ref="#PWR?"  Part="1"
 F 0 "#PWR?" H 5110 2190 50  0001 C CNN
@@
 AR Path="/5E0A0E29/5E0AD665" Ref="#PWR?"  Part="1"
 AR Path="/5E052856/5E0AD665" Ref="#PWR?"  Part="1"
+AR Path="/5EAE2D84/5E0AD665" Ref="#PWR?"  Part="1"
 AR Path="/5E939D24/5E0AD665" Ref="#PWR?"  Part="1"
 F 0 "#PWR?" H 5110 1490 50  0001 C CNN
@@
 AR Path="/5E0A0E29/5E0B2427" Ref="C?"  Part="1"
 AR Path="/5E052856/5E0B2427" Ref="C?"  Part="1"
+AR Path="/5EAE2D84/5E0B2427" Ref="C?"  Part="1"
 AR Path="/5E939D24/5E0B2427" Ref="C?"  Part="1"
 F 0 "C?" H 5135 3110 50  0000 L CNN
@@
 F 2 "Capacitors_SMD:C_0402" H 5148 2860 50  0001 C CNN
 F 3 "" H 5135 3110 50  0001 C CNN
-F 4 "0402" H 4960 3110 50  0000 R CNN "display_footprint"
+F 4 "" H 4960 3110 50  0000 R CNN "display_footprint"
 F 5 "50V" H 4960 3010 50  0000 R CNN "Voltage"
 F 6 "X7R" H 4960 2910 50  0000 R CNN "Dielectric"
@@
 AR Path="/5E0A0E29/5E0B535B" Ref="#PWR?"  Part="1"
 AR Path="/5E052856/5E0B535B" Ref="#PWR?"  Part="1"
+AR Path="/5EAE2D84/5E0B535B" Ref="#PWR?"  Part="1"
 AR Path="/5E939D24/5E0B535B" Ref="#PWR?"  Part="1"
 F 0 "#PWR?" H 5110 2710 50  0001 C CNN
@@
 AR Path="/5E0A0E29/5E0B592B" Ref="#PWR?"  Part="1"
 AR Path="/5E052856/5E0B592B" Ref="#PWR?"  Part="1"
+AR Path="/5EAE2D84/5E0B592B" Ref="#PWR?"  Part="1"
 AR Path="/5E939D24/5E0B592B" Ref="#PWR?"  Part="1"
 F 0 "#PWR?" H 5110 2910 50  0001 C CNN
@@
 I2C_SDA
 $Comp
+L Custom_Library:I2C_Address DOC?
+U 1 1 5E0B8BC8
+P 6010 2880
+AR Path="/5E0652BA/5E0B8BC8" Ref="DOC?"  Part="1"
+AR Path="/5E0A0E29/5E0B8BC8" Ref="DOC?"  Part="1"
+AR Path="/5E052856/5E0B8BC8" Ref="DOC?"  Part="1"
+AR Path="/5EAE2D84/5E0B8BC8" Ref="DOC?"  Part="1"
+AR Path="/5E939D24/5E0B8BC8" Ref="DOC?"  Part="1"
+F 0 "DOC?" H 6010 3130 60  0001 C CNN
+F 1 "0x40" H 5560 2880 60  0000 L CNN
+F 2 "" H 6010 3230 60  0001 C CNN
+F 3 "" H 6010 3230 60  0001 C CNN
+	1    6010 2880
+	1    0    0    -1
+$EndComp
+$Comp
 L power:GND #PWR?
 U 1 1 5E2AA995
@@
 AR Path="/5E0A0E29/5E2AA995" Ref="#PWR?"  Part="1"
 AR Path="/5E052856/5E2AA995" Ref="#PWR?"  Part="1"
+AR Path="/5EAE2D84/5E2AA995" Ref="#PWR?"  Part="1"
 AR Path="/5E939D24/5E2AA995" Ref="#PWR?"  Part="1"
 F 0 "#PWR?" H 5110 4870 50  0001 C CNN
@@
 AR Path="/5E0A0E29/5E2AA99A" Ref="#PWR?"  Part="1"
 AR Path="/5E052856/5E2AA99A" Ref="#PWR?"  Part="1"
+AR Path="/5EAE2D84/5E2AA99A" Ref="#PWR?"  Part="1"
 AR Path="/5E939D24/5E2AA99A" Ref="#PWR?"  Part="1"
 F 0 "#PWR?" H 5110 3890 50  0001 C CNN
@@
 AR Path="/5E0A0E29/5E2AA99D" Ref="U?"  Part="1"
 AR Path="/5E052856/5E2AA99D" Ref="U?"  Part="1"
+AR Path="/5EAE2D84/5E2AA99D" Ref="U?"  Part="1"
 AR Path="/5E939D24/5E2AA99D" Ref="U?"  Part="1"
 F 0 "U?" H 4860 4990 50  0000 C CNN
@@
 F 3 "http://ww1.microchip.com/downloads/en/DeviceDoc/22203b.pdf" H 4860 4990 50  0001 C CNN
 F 4 "MCP9804T-E/MCCT-ND" H 5110 4540 50  0001 C CNN "Digi-Key PN"
+F 5 "Telemetry" H 5510 5070 50  0000 C CNN "Configuration"
 	1    5110 4540
 	-1   0    0    -1
@@
 AR Path="/5E0A0E29/5E2AA9A1" Ref="C?"  Part="1"
 AR Path="/5E052856/5E2AA9A1" Ref="C?"  Part="1"
+AR Path="/5EAE2D84/5E2AA9A1" Ref="C?"  Part="1"
 AR Path="/5E939D24/5E2AA9A1" Ref="C?"  Part="1"
 F 0 "C?" H 5135 5790 50  0000 L CNN
@@
 F 2 "Capacitors_SMD:C_0402" H 5148 5540 50  0001 C CNN
 F 3 "" H 5135 5790 50  0001 C CNN
-F 4 "0402" H 4960 5790 50  0000 R CNN "display_footprint"
+F 4 "" H 4960 5790 50  0000 R CNN "display_footprint"
 F 5 "50V" H 4960 5690 50  0000 R CNN "Voltage"
 F 6 "X7R" H 4960 5590 50  0000 R CNN "Dielectric"
@@
 AR Path="/5E0A0E29/5E2AA9A6" Ref="#PWR?"  Part="1"
 AR Path="/5E052856/5E2AA9A6" Ref="#PWR?"  Part="1"
+AR Path="/5EAE2D84/5E2AA9A6" Ref="#PWR?"  Part="1"
 AR Path="/5E939D24/5E2AA9A6" Ref="#PWR?"  Part="1"
 F 0 "#PWR?" H 5110 5390 50  0001 C CNN
@@
 AR Path="/5E0A0E29/5E2AA9AD" Ref="#PWR?"  Part="1"
 AR Path="/5E052856/5E2AA9AD" Ref="#PWR?"  Part="1"
+AR Path="/5EAE2D84/5E2AA9AD" Ref="#PWR?"  Part="1"
 AR Path="/5E939D24/5E2AA9AD" Ref="#PWR?"  Part="1"
 F 0 "#PWR?" H 5110 5590 50  0001 C CNN
@@
 F 3 "" H 5110 5840 50  0001 C CNN
 	1    5110 5840
+	1    0    0    -1
+$EndComp
+$Comp
+L Custom_Library:I2C_Address DOC?
+U 1 1 5E2AA9AF
+P 6010 5560
+AR Path="/5E0652BA/5E2AA9AF" Ref="DOC?"  Part="1"
+AR Path="/5E0A0E29/5E2AA9AF" Ref="DOC?"  Part="1"
+AR Path="/5E052856/5E2AA9AF" Ref="DOC?"  Part="1"
+AR Path="/5EAE2D84/5E2AA9AF" Ref="DOC?"  Part="1"
+AR Path="/5E939D24/5E2AA9AF" Ref="DOC?"  Part="1"
+F 0 "DOC?" H 6010 5810 60  0001 C CNN
+F 1 "0x18" H 5560 5560 60  0000 L CNN
+F 2 "" H 6010 5910 60  0001 C CNN
+F 3 "" H 6010 5910 60  0001 C CNN
+	1    6010 5560
 	1    0    0    -1
 $EndComp
@@
 AR Path="/5E0A0E29/5E07E0FD" Ref="C?"  Part="1"
 AR Path="/5E052856/5E07E0FD" Ref="C?"  Part="1"
+AR Path="/5EAE2D84/5E07E0FD" Ref="C?"  Part="1"
 AR Path="/5E939D24/5E07E0FD" Ref="C?"  Part="1"
 F 0 "C?" H 4255 2130 50  0000 L CNN
@@
 F 2 "Capacitors_SMD:C_0402" H 4268 1880 50  0001 C CNN
 F 3 "" H 4255 2130 50  0001 C CNN
-F 4 "0402" H 4080 2130 50  0000 R CNN "display_footprint"
+F 4 "" H 4080 2130 50  0000 R CNN "display_footprint"
 F 5 "50V" H 4080 2030 50  0000 R CNN "Voltage"
 F 6 "X7R" H 4080 1930 50  0000 R CNN "Dielectric"
@@
 F 3 "http://www.ti.com/lit/ds/symlink/ina219.pdf" H 5460 1940 50  0001 C CNN
 F 4 "296-46420-1-ND" H 5110 2040 50  0001 C CNN "Digi-Key PN"
+F 5 "Telemetry" H 5370 2470 50  0000 C CNN "Configuration"
 	1    5110 2040
 	1    0    0    -1
@@
 Connection ~ 4230 2260
 $Comp
-L Custom_Library:I2C_Address DOC?
-U 1 1 5E0B8BC8
-P 6010 2880
-AR Path="/5E0652BA/5E0B8BC8" Ref="DOC?"  Part="1"
-AR Path="/5E0A0E29/5E0B8BC8" Ref="DOC?"  Part="1"
-AR Path="/5E052856/5E0B8BC8" Ref="DOC?"  Part="1"
-AR Path="/5E939D24/5E0B8BC8" Ref="DOC?"  Part="1"
-F 0 "DOC?" H 6010 3130 60  0001 C CNN
-F 1 "jahjahdslkjfhdsaf" H 5560 2880 60  0000 L CNN
-F 2 "" H 6010 3230 60  0001 C CNN
-F 3 "" H 6010 3230 60  0001 C CNN
-	1    6010 2880
-	1    0    0    -1
-$EndComp
-$Comp
-L Custom_Library:I2C_Address DOC?
-U 1 1 5E2AA9AF
-P 6010 5560
-AR Path="/5E0652BA/5E2AA9AF" Ref="DOC?"  Part="1"
-AR Path="/5E0A0E29/5E2AA9AF" Ref="DOC?"  Part="1"
-AR Path="/5E052856/5E2AA9AF" Ref="DOC?"  Part="1"
-AR Path="/5E939D24/5E2AA9AF" Ref="DOC?"  Part="1"
-F 0 "DOC?" H 6010 5810 60  0001 C CNN
-F 1 "lkjasflkjasdf" H 5560 5560 60  0000 L CNN
-F 2 "" H 6010 5910 60  0001 C CNN
-F 3 "" H 6010 5910 60  0001 C CNN
-	1    6010 5560
-	1    0    0    -1
+L power:GND #PWR?
+U 1 1 5E320C53
+P 5510 2140
+AR Path="/5E0652BA/5E320C53" Ref="#PWR?"  Part="1"
+AR Path="/5E0A0E29/5E320C53" Ref="#PWR?"  Part="1"
+AR Path="/5E052856/5E320C53" Ref="#PWR?"  Part="1"
+AR Path="/5EAE2D84/5E320C53" Ref="#PWR?"  Part="1"
+AR Path="/5E939D24/5E320C53" Ref="#PWR?"  Part="1"
+F 0 "#PWR?" H 5510 1890 50  0001 C CNN
+F 1 "GND" V 5510 1990 50  0000 R CNN
+F 2 "" H 5510 2140 50  0001 C CNN
+F 3 "" H 5510 2140 50  0001 C CNN
+	1    5510 2140
+	0    -1   -1   0
+$EndComp
+$Comp
+L power:GND #PWR?
+U 1 1 5E321138
+P 5510 2240
+AR Path="/5E0652BA/5E321138" Ref="#PWR?"  Part="1"
+AR Path="/5E0A0E29/5E321138" Ref="#PWR?"  Part="1"
+AR Path="/5E052856/5E321138" Ref="#PWR?"  Part="1"
+AR Path="/5EAE2D84/5E321138" Ref="#PWR?"  Part="1"
+AR Path="/5E939D24/5E321138" Ref="#PWR?"  Part="1"
+F 0 "#PWR?" H 5510 1990 50  0001 C CNN
+F 1 "GND" V 5510 2090 50  0000 R CNN
+F 2 "" H 5510 2240 50  0001 C CNN
+F 3 "" H 5510 2240 50  0001 C CNN
+	1    5510 2240
+	0    -1   -1   0
+$EndComp
+$Comp
+L power:GND #PWR?
+U 1 1 5E35CA2A
+P 5510 4840
+AR Path="/5E0652BA/5E35CA2A" Ref="#PWR?"  Part="1"
+AR Path="/5E0A0E29/5E35CA2A" Ref="#PWR?"  Part="1"
+AR Path="/5E052856/5E35CA2A" Ref="#PWR?"  Part="1"
+AR Path="/5EAE2D84/5E35CA2A" Ref="#PWR?"  Part="1"
+AR Path="/5E939D24/5E35CA2A" Ref="#PWR?"  Part="1"
+F 0 "#PWR?" H 5510 4590 50  0001 C CNN
+F 1 "GND" V 5510 4690 50  0000 R CNN
+F 2 "" H 5510 4840 50  0001 C CNN
+F 3 "" H 5510 4840 50  0001 C CNN
+	1    5510 4840
+	0    -1   -1   0
+$EndComp
+$Comp
+L power:GND #PWR?
+U 1 1 5E35C74D
+P 5510 4740
+AR Path="/5E0652BA/5E35C74D" Ref="#PWR?"  Part="1"
+AR Path="/5E0A0E29/5E35C74D" Ref="#PWR?"  Part="1"
+AR Path="/5E052856/5E35C74D" Ref="#PWR?"  Part="1"
+AR Path="/5EAE2D84/5E35C74D" Ref="#PWR?"  Part="1"
+AR Path="/5E939D24/5E35C74D" Ref="#PWR?"  Part="1"
+F 0 "#PWR?" H 5510 4490 50  0001 C CNN
+F 1 "GND" V 5510 4590 50  0000 R CNN
+F 2 "" H 5510 4740 50  0001 C CNN
+F 3 "" H 5510 4740 50  0001 C CNN
+	1    5510 4740
+	0    -1   -1   0
+$EndComp
+$Comp
+L power:GND #PWR?
+U 1 1 5E35BF65
+P 5510 4640
+AR Path="/5E0652BA/5E35BF65" Ref="#PWR?"  Part="1"
+AR Path="/5E0A0E29/5E35BF65" Ref="#PWR?"  Part="1"
+AR Path="/5E052856/5E35BF65" Ref="#PWR?"  Part="1"
+AR Path="/5EAE2D84/5E35BF65" Ref="#PWR?"  Part="1"
+AR Path="/5E939D24/5E35BF65" Ref="#PWR?"  Part="1"
+F 0 "#PWR?" H 5510 4390 50  0001 C CNN
+F 1 "GND" V 5510 4490 50  0000 R CNN
+F 2 "" H 5510 4640 50  0001 C CNN
+F 3 "" H 5510 4640 50  0001 C CNN
+	1    5510 4640
+	0    -1   -1   0
 $EndComp
 $EndSCHEMATC

Commit message: More sch work
Parts:
- DOC?: value 0x40 -> FIX ME
- DOC?: value 0x18 -> FIX ME
Connections:
- net GND: no longer U?.5 (A2), U?.6 (A1), U?.7 (A0), U?.7 (A0), U?.8 (A1)
Changed lines of the file:
@@
 $Descr A 11000 8500
 encoding utf-8
-Sheet 3 20
+Sheet 3 21
 Title "Pulse Oximeter"
 Date "2020-08-01"
@@
 AR Path="/5E939D24/5E0B8BC8" Ref="DOC?"  Part="1"
 F 0 "DOC?" H 6010 3130 60  0001 C CNN
-F 1 "0x40" H 5560 2880 60  0000 L CNN
+F 1 "FIX ME" H 5560 2880 60  0000 L CNN
 F 2 "" H 6010 3230 60  0001 C CNN
 F 3 "" H 6010 3230 60  0001 C CNN
@@
 AR Path="/5E939D24/5E2AA9AF" Ref="DOC?"  Part="1"
 F 0 "DOC?" H 6010 5810 60  0001 C CNN
-F 1 "0x18" H 5560 5560 60  0000 L CNN
+F 1 "FIX ME" H 5560 5560 60  0000 L CNN
 F 2 "" H 6010 5910 60  0001 C CNN
 F 3 "" H 6010 5910 60  0001 C CNN
@@
 	4540 2260 4230 2260
 Connection ~ 4230 2260
-$Comp
-L power:GND #PWR?
-U 1 1 5E320C53
-P 5510 2140
-AR Path="/5E0652BA/5E320C53" Ref="#PWR?"  Part="1"
-AR Path="/5E0A0E29/5E320C53" Ref="#PWR?"  Part="1"
-AR Path="/5E052856/5E320C53" Ref="#PWR?"  Part="1"
-AR Path="/5EAE2D84/5E320C53" Ref="#PWR?"  Part="1"
-AR Path="/5E939D24/5E320C53" Ref="#PWR?"  Part="1"
-F 0 "#PWR?" H 5510 1890 50  0001 C CNN
-F 1 "GND" V 5510 1990 50  0000 R CNN
-F 2 "" H 5510 2140 50  0001 C CNN
-F 3 "" H 5510 2140 50  0001 C CNN
-	1    5510 2140
-	0    -1   -1   0
-$EndComp
-$Comp
-L power:GND #PWR?
-U 1 1 5E321138
-P 5510 2240
-AR Path="/5E0652BA/5E321138" Ref="#PWR?"  Part="1"
-AR Path="/5E0A0E29/5E321138" Ref="#PWR?"  Part="1"
-AR Path="/5E052856/5E321138" Ref="#PWR?"  Part="1"
-AR Path="/5EAE2D84/5E321138" Ref="#PWR?"  Part="1"
-AR Path="/5E939D24/5E321138" Ref="#PWR?"  Part="1"
-F 0 "#PWR?" H 5510 1990 50  0001 C CNN
-F 1 "GND" V 5510 2090 50  0000 R CNN
-F 2 "" H 5510 2240 50  0001 C CNN
-F 3 "" H 5510 2240 50  0001 C CNN
-	1    5510 2240
-	0    -1   -1   0
-$EndComp
-$Comp
-L power:GND #PWR?
-U 1 1 5E35CA2A
-P 5510 4840
-AR Path="/5E0652BA/5E35CA2A" Ref="#PWR?"  Part="1"
-AR Path="/5E0A0E29/5E35CA2A" Ref="#PWR?"  Part="1"
-AR Path="/5E052856/5E35CA2A" Ref="#PWR?"  Part="1"
-AR Path="/5EAE2D84/5E35CA2A" Ref="#PWR?"  Part="1"
-AR Path="/5E939D24/5E35CA2A" Ref="#PWR?"  Part="1"
-F 0 "#PWR?" H 5510 4590 50  0001 C CNN
-F 1 "GND" V 5510 4690 50  0000 R CNN
-F 2 "" H 5510 4840 50  0001 C CNN
-F 3 "" H 5510 4840 50  0001 C CNN
-	1    5510 4840
-	0    -1   -1   0
-$EndComp
-$Comp
-L power:GND #PWR?
-U 1 1 5E35C74D
-P 5510 4740
-AR Path="/5E0652BA/5E35C74D" Ref="#PWR?"  Part="1"
-AR Path="/5E0A0E29/5E35C74D" Ref="#PWR?"  Part="1"
-AR Path="/5E052856/5E35C74D" Ref="#PWR?"  Part="1"
-AR Path="/5EAE2D84/5E35C74D" Ref="#PWR?"  Part="1"
-AR Path="/5E939D24/5E35C74D" Ref="#PWR?"  Part="1"
-F 0 "#PWR?" H 5510 4490 50  0001 C CNN
-F 1 "GND" V 5510 4590 50  0000 R CNN
-F 2 "" H 5510 4740 50  0001 C CNN
-F 3 "" H 5510 4740 50  0001 C CNN
-	1    5510 4740
-	0    -1   -1   0
-$EndComp
-$Comp
-L power:GND #PWR?
-U 1 1 5E35BF65
-P 5510 4640
-AR Path="/5E0652BA/5E35BF65" Ref="#PWR?"  Part="1"
-AR Path="/5E0A0E29/5E35BF65" Ref="#PWR?"  Part="1"
-AR Path="/5E052856/5E35BF65" Ref="#PWR?"  Part="1"
-AR Path="/5EAE2D84/5E35BF65" Ref="#PWR?"  Part="1"
-AR Path="/5E939D24/5E35BF65" Ref="#PWR?"  Part="1"
-F 0 "#PWR?" H 5510 4390 50  0001 C CNN
-F 1 "GND" V 5510 4490 50  0000 R CNN
-F 2 "" H 5510 4640 50  0001 C CNN
-F 3 "" H 5510 4640 50  0001 C CNN
-	1    5510 4640
-	0    -1   -1   0
-$EndComp
 $EndSCHEMATC

Commit message: big sch push
Parts:
- removed C? (x2): 0.1uF, Capacitors_SMD:C_0402, symbol Custom_Library:C_Custom
- removed DOC? (x2): FIX ME, symbol Custom_Library:I2C_Address
- removed U?: INA219BxDCN, Package_TO_SOT_SMD:SOT-23-8, symbol Analog_ADC:INA219BxDCN
- removed U?: MCP9804, Package_DFN_QFN:DFN-8-1EP_3x2mm_P0.5mm_EP1.3x1.5mm, symbol Sensor_Temperature:MCP9804_DFN
- added C301, C302: 0.1uF, Capacitors_SMD:C_0603, symbol Custom_Library:C_Custom
- added DOC301: 0x40, symbol Custom_Library:I2C_Address
- added DOC302: 0x18, symbol Custom_Library:I2C_Address
- added U301: INA219BxDCN, Package_TO_SOT_SMD:SOT-23-8, symbol Analog_ADC:INA219BxDCN
- added U302: MCP9804, Package_DFN_QFN:DFN-8-1EP_3x2mm_P0.5mm_EP1.3x1.5mm, symbol Sensor_Temperature:MCP9804_DFN
- C303: renamed from C?; footprint Capacitors_SMD:C_0402 -> Capacitors_SMD:C_0603; Digi-Key PN 490-10701-1-ND -> 399-7845-1-ND; display_footprint (none) -> 0603
Connections:
- net +3V3: now also C302.1, U301.4 (VS), U302.8 (VDD)
- net GND: now also C302.2, U301.3 (GND), U301.7 (A0), U301.8 (A1), U302.4 (GND), U302.5 (A2), U302.6 (A1), U302.7 (A0), U302.9 (EP/GND)
- net I2C_SCL: now also U301.5 (SCL), U302.2 (SCL)
- net I2C_SDA: now also U301.6 (SDA), U302.1 (SDA)
- net POS12_SNS+: now also C301.1, U301.1 (IN+)
- net POS12_SNS-: now also C301.2, U301.2 (IN-)
Other:
- note added: "RSHUNT = 0.02\nCLSB = 60uA"
