File: hdw/Analog_Clock/POS3P3_Power_Supply.sch (KiCad schematic (older format))
At the start: 18 parts

Commit message: More schematic work
Parts:
- added D?: DZ2S033X0L, Diode_SMD:D_SOD-523, symbol Diode:DZ2S033X0L
- added Q?: BSS214NW, Package_TO_SOT_SMD:SOT-323_SC-70, symbol Transistor_FET:BSS214NW
- added Q?: Si1442DH, Package_TO_SOT_SMD:SOT-363_SC-70-6, symbol Transistor_FET:Si1442DH
- added R?: 0, Resistors_SMD:R_0402, symbol Custom_Library:R_Custom
- added R?: 10k, Resistors_SMD:R_0402, symbol Custom_Library:R_Custom
- added R?: 27, Resistors_SMD:R_0402, symbol Custom_Library:R_Custom
Connections:
- net labels added: POS12_PGOOD
- wire segments 47 -> 52
Changed lines of the file:
@@
 EESchema Schematic File Version 4
+LIBS:Analog_Clock-cache
 EELAYER 30 0
 EELAYER END
@@
 	-1   0    0    -1
 $EndComp
+$Comp
+L Custom_Library:R_Custom R?
+U 1 1 5E94EEC8
+P 1770 5610
+AR Path="/5E939CFF/5E94EEC8" Ref="R?"  Part="1"
+AR Path="/5E939D31/5E94EEC8" Ref="R?"  Part="1"
+F 0 "R?" V 1670 5610 50  0000 C CNN
+F 1 "0" V 1770 5610 50  0000 C CNN
+F 2 "Resistors_SMD:R_0402" H 1770 5610 50  0001 C CNN
+F 3 "" H 1770 5610 50  0001 C CNN
+F 4 "0402" V 1870 5610 50  0000 C CNN "display_footprint"
+F 5 "1%" V 1970 5610 50  0000 C CNN "Tolerance"
+F 6 "1/16W" V 2070 5610 50  0000 C CNN "Wattage"
+	1    1770 5610
+	0    1    1    0
+$EndComp
+Text GLabel 1920 5610 2    50   Output ~ 0
+POS3P3_RUN
+Text GLabel 1620 5610 0    50   Input ~ 0
+POS12_PGOOD
+$Comp
+L Transistor_FET:BSS214NW Q?
+U 1 1 5E951F4A
+P 3190 7350
+F 0 "Q?" H 3390 7425 50  0000 L CNN
+F 1 "BSS214NW" H 3390 7350 50  0000 L CNN
+F 2 "Package_TO_SOT_SMD:SOT-323_SC-70" H 3390 7275 50  0001 L CIN
+F 3 "https://www.infineon.com/dgdl/Infineon-BSS214NW-DS-v02_02-en.pdf?fileId=db3a30431b3e89eb011b695aebc01bde" H 3190 7350 50  0001 L CNN
+	1    3190 7350
+	1    0    0    -1
+$EndComp
+$Comp
+L Custom_Library:R_Custom R?
+U 1 1 5E954057
+P 3290 6720
+AR Path="/5BB27BA3/5E954057" Ref="R?"  Part="1"
+AR Path="/5BB27BF7/5E954057" Ref="R?"  Part="1"
+AR Path="/5C1DE17A/5E954057" Ref="R?"  Part="1"
+AR Path="/5C1E3A08/5E954057" Ref="R?"  Part="1"
+AR Path="/5D779AE1/5E954057" Ref="R?"  Part="1"
+AR Path="/5CB7718D/5E954057" Ref="R?"  Part="1"
+AR Path="/5E0DC082/5E954057" Ref="R?"  Part="1"
+AR Path="/5E0F263A/5E954057" Ref="R?"  Part="1"
+AR Path="/5E939D31/5E954057" Ref="R?"  Part="1"
+F 0 "R?" H 3210 6720 50  0000 R CNN
+F 1 "10k" V 3290 6720 50  0000 C CNN
+F 2 "Resistors_SMD:R_0402" H 3290 6720 50  0001 C CNN
+F 3 "" H 3290 6720 50  0001 C CNN
+F 4 "0402" H 3390 6800 50  0000 L CNN "display_footprint"
+F 5 "1%" H 3390 6720 50  0000 L CNN "Tolerance"
+F 6 "1/16W" H 3400 6640 50  0000 L CNN "Wattage"
+F 7 "RMCF0402FT10K0CT-ND" H 3590 7120 60  0001 C CNN "Digi-Key PN"
+	1    3290 6720
+	1    0    0    -1
+$EndComp
+$Comp
+L power:GND #PWR?
+U 1 1 5E954CDC
+P 3290 7550
+F 0 "#PWR?" H 3290 7300 50  0001 C CNN
+F 1 "GND" H 3290 7400 50  0000 C CNN
+F 2 "" H 3290 7550 50  0001 C CNN
+F 3 "" H 3290 7550 50  0001 C CNN
+	1    3290 7550
+	1    0    0    -1
+$EndComp
+$Comp
+L power:+12V #PWR?
+U 1 1 5E9552D1
+P 3290 6570
+AR Path="/5CB7718D/5E9552D1" Ref="#PWR?"  Part="1"
+AR Path="/5E0DC082/5E9552D1" Ref="#PWR?"  Part="1"
+AR Path="/5E0F263A/5E9552D1" Ref="#PWR?"  Part="1"
+AR Path="/5E939D31/5E9552D1" Ref="#PWR?"  Part="1"
+F 0 "#PWR?" H 3290 6420 50  0001 C CNN
+F 1 "+12V" H 3290 6710 50  0000 C CNN
+F 2 "" H 3290 6570 50  0001 C CNN
+F 3 "" H 3290 6570 50  0001 C CNN
+	1    3290 6570
+	1    0    0    -1
+$EndComp
+Wire Wire Line
+	3290 6870 3290 7070
+Text GLabel 2990 7350 0    50   Input ~ 0
+POS3P3_RUN
+$Comp
+L Transistor_FET:Si1442DH Q?
+U 1 1 5E960022
+P 4650 7070
+F 0 "Q?" H 4850 7120 50  0000 L CNN
+F 1 "Si1442DH" H 4850 7020 50  0000 L CNN
+F 2 "Package_TO_SOT_SMD:SOT-363_SC-70-6" H 4750 6670 50  0001 C CNN
+F 3 "http://www.vishay.com/docs/63772/si1442dh.pdf" H 4650 7070 50  0001 C CNN
+	1    4650 7070
+	1    0    0    -1
+$EndComp
+$Comp
+L Diode:DZ2S033X0L D?
+U 1 1 5E965C70
+P 3950 7400
+AR Path="/5E98CF45/5E965C70" Ref="D?"  Part="1"
+AR Path="/5E939D31/5E965C70" Ref="D?"  Part="1"
+F 0 "D?" V 3890 7510 50  0000 L CNN
+F 1 "DZ2S033X0L" V 3990 7510 50  0000 L CNN
+F 2 "Diode_SMD:D_SOD-523" H 3950 7225 50  0001 C CNN
+F 3 "https://industrial.panasonic.com/content/data/SC/ds/ds4/DZ2S03300L_E.pdf" H 3950 7400 50  0001 C CNN
+	1    3950 7400
+	0    1    1    0
+$EndComp
+$Comp
+L power:GND #PWR?
+U 1 1 5E966579
+P 3950 7550
+F 0 "#PWR?" H 3950 7300 50  0001 C CNN
+F 1 "GND" H 3950 7400 50  0000 C CNN
+F 2 "" H 3950 7550 50  0001 C CNN
+F 3 "" H 3950 7550 50  0001 C CNN
+	1    3950 7550
+	1    0    0    -1
+$EndComp
+$Comp
+L power:GND #PWR?
+U 1 1 5E9674AD
+P 4750 7270
+F 0 "#PWR?" H 4750 7020 50  0001 C CNN
+F 1 "GND" H 4750 7120 50  0000 C CNN
+F 2 "" H 4750 7270 50  0001 C CNN
+F 3 "" H 4750 7270 50  0001 C CNN
+	1    4750 7270
+	1    0    0    -1
+$EndComp
+Wire Wire Line
+	4450 7070 3950 7070
+Connection ~ 3290 7070
+Wire Wire Line
+	3290 7070 3290 7150
+Wire Wire Line
+	3950 7250 3950 7070
+Connection ~ 3950 7070
+Wire Wire Line
+	3950 7070 3290 7070
+$Comp
+L power:+3.3V #PWR?
+U 1 1 5E96D7A6
+P 4750 6570
+AR Path="/5CB7718D/5E96D7A6" Ref="#PWR?"  Part="1"
+AR Path="/5E0DC082/5E96D7A6" Ref="#PWR?"  Part="1"
+AR Path="/5E0F263A/5E96D7A6" Ref="#PWR?"  Part="1"
+AR Path="/5E939D31/5E96D7A6" Ref="#PWR?"  Part="1"
+F 0 "#PWR?" H 4750 6420 50  0001 C CNN
+F 1 "+3.3V" H 4750 6710 50  0000 C CNN
+F 2 "" H 4750 6570 50  0001 C CNN
+F 3 "" H 4750 6570 50  0001 C CNN
+	1    4750 6570
+	1    0    0    -1
+$EndComp
+$Comp
+L Custom_Library:R_Custom R?
+U 1 1 5E971822
+P 4750 6720
+AR Path="/5BB27BA3/5E971822" Ref="R?"  Part="1"
+AR Path="/5BB27BF7/5E971822" Ref="R?"  Part="1"
+AR Path="/5C1DE17A/5E971822" Ref="R?"  Part="1"
+AR Path="/5C1E3A08/5E971822" Ref="R?"  Part="1"
+AR Path="/5D779AE1/5E971822" Ref="R?"  Part="1"
+AR Path="/5CB7718D/5E971822" Ref="R?"  Part="1"
+AR Path="/5E0DC082/5E971822" Ref="R?"  Part="1"
+AR Path="/5E0F263A/5E971822" Ref="R?"  Part="1"
+AR Path="/5E939D31/5E971822" Ref="R?"  Part="1"
+F 0 "R?" H 4670 6720 50  0000 R CNN
+F 1 "27" V 4750 6720 50  0000 C CNN
+F 2 "Resistors_SMD:R_0402" H 4750 6720 50  0001 C CNN
+F 3 "" H 4750 6720 50  0001 C CNN
+F 4 "0402" H 4850 6800 50  0000 L CNN "display_footprint"
+F 5 "1%" H 4850 6720 50  0000 L CNN "Tolerance"
+F 6 "1/16W" H 4860 6640 50  0000 L CNN "Wattage"
+	1    4750 6720
+	1    0    0    -1
+$EndComp
 $EndSCHEMATC

Commit message: a few sch adjustments
Parts:
- removed C?: 22uF, Capacitors_SMD:C_1206, symbol Custom_Library:C_Custom
- removed D?: DZ2S033X0L, Diode_SMD:D_SOD-523, symbol Diode:DZ2S033X0L
- removed Q?: BSS214NW, Package_TO_SOT_SMD:SOT-323_SC-70, symbol Transistor_FET:BSS214NW
- removed Q?: Si1442DH, Package_TO_SOT_SMD:SOT-363_SC-70-6, symbol Transistor_FET:Si1442DH
- removed R?: 0.02, Resistors_SMD:R_0612, symbol Custom_Library:R_Custom
- removed R?: 0, Resistors_SMD:R_0402, symbol Custom_Library:R_Custom
- removed R? (x4): 10, Resistors_SMD:R_0402, symbol Custom_Library:R_Custom
- removed R?: 10k, Resistors_SMD:R_0402, symbol Custom_Library:R_Custom
- removed R?: 27, Resistors_SMD:R_0402, symbol Custom_Library:R_Custom
- removed U?: TPS62130, Housings_DFN_QFN:QFN-16-1EP_3x3mm_Pitch0.5mm, symbol Custom_Library:TPS62130
- added C?: 10uF, Capacitors_SMD:C_0402, symbol Custom_Library:C_Custom
- added D?: BAT48JFILM, Diode_SMD:D_SOD-323, symbol Diode:BAT48JFILM
- added Q?: ZXMS6004FFTA, Package_TO_SOT_SMD:SOT-23, symbol Custom_Library:ZXMS6004FFTA
- added Q?: BSS214NW, Package_TO_SOT_SMD:SOT-323_SC-70, symbol Transistor_FET:BSS214NW
- added R? (x3): 10, Resistors_SMD:R_0402, symbol Custom_Library:R_Custom
- added R?: 10k, Resistors_SMD:R_0402, symbol Custom_Library:R_Custom
- added U?: TPS62150, Package_DFN_QFN:QFN-16-1EP_3x3mm_P0.5mm_EP1.8x1.8mm, symbol Custom_Library:TPS62150
- C?: value 22uF -> 100uF; Dielectric X7R -> X5R; Digi-Key PN 1276-3148-1-ND -> 587-1963-1-ND; Voltage 10V -> 6.3V
- C? (x3): display_footprint 0402 -> (none)
- L?: value 2.2u -> 3.3uH; footprint Inductors_SMD:L_Vishay_IHLP-2020 -> Inductors_SMD:L_Vishay_IHLP-1212; Ampacity 5.5A -> 2.7A; Digi-Key PN 541-1236-1-ND -> 541-2567-1-ND; display_footprint IHLP2020 -> IHLP1212
- R?: Digi-Key PN (none) -> 311-562KLRCT-ND
- R?: Digi-Key PN (none) -> A129654CT-ND
Connections:
- net labels removed: POS3P3_SNS_IN+, POS3P3_SNS_IN-
- wire segments 52 -> 46
Other:
- moved on the sheet: C?, L?, R?, TP?

Commit message: big sch push
Parts:
- C402: renamed from C?; footprint Capacitors_SMD:C_0402 -> Capacitors_SMD:C_0603; Digi-Key PN 490-13211-1-ND -> 490-10474-1-ND; Voltage 6.3V -> 10V; display_footprint 0402 -> 0603
- C403: renamed from C?; footprint Capacitors_SMD:C_0402 -> Capacitors_SMD:C_0603; Digi-Key PN 490-13295-1-ND -> 399-7842-1-ND; display_footprint (none) -> 0603
- C404, C406: renamed from C?; footprint Capacitors_SMD:C_0402 -> Capacitors_SMD:C_0603; Digi-Key PN 490-10701-1-ND -> 399-7845-1-ND; display_footprint (none) -> 0603
- R401, R404, R406: renamed from R?; footprint Resistors_SMD:R_0402 -> Resistors_SMD:R_0603; Digi-Key PN 541-3964-1-ND -> (none); Wattage 1/16W -> 1/10W; display_footprint 0402 -> 0603
- R402, R403: renamed from R?; footprint Resistors_SMD:R_0402 -> Resistors_SMD:R_0603; Digi-Key PN RMCF0402FT10K0CT-ND -> (none); Wattage 1/16W -> 1/10W; display_footprint 0402 -> 0603
- R407: renamed from R?; footprint Resistors_SMD:R_0402 -> Resistors_SMD:R_0603; Digi-Key PN 311-562KLRCT-ND -> (none); Wattage 1/16W -> 1/10W; display_footprint 0402 -> 0603
- R408: renamed from R?; footprint Resistors_SMD:R_0402 -> Resistors_SMD:R_0603; Digi-Key PN A129654CT-ND -> (none); Wattage 1/16W -> 1/10W; display_footprint 0402 -> 0603
- gave numbers to parts that had none: 9
Connections:
- net POS3P3_SNS_OUT+ renamed POS3P3_SNS+
- net POS3P3_SNS_OUT- renamed POS3P3_SNS-

Commit message: Much more schematic progress
Parts:
- R401, R402, R403, R404, R406: Digi-Key PN (none) -> YAG2321CT-ND
- R407: Digi-Key PN (none) -> 311-562KHRCT-ND
- R408: Digi-Key PN (none) -> 311-180KHRCT-ND
Changed lines of the file:
@@
 encoding utf-8
 Sheet 4 25
-Title "Pulse Oximeter"
-Date "2020-08-01"
+Title "Analog Clock"
+Date "2020-08-15"
 Rev "A"
 Comp "Drew Maatman"
@@
 F 5 "1%" H 8320 3810 50  0000 L CNN "Tolerance"
 F 6 "1/10W" H 8330 3730 50  0000 L CNN "Wattage"
-F 7 "" H 8220 3810 50  0001 C CNN "Digi-Key PN"
+F 7 "311-562KHRCT-ND" H 8220 3810 50  0001 C CNN "Digi-Key PN"
 	1    8220 3810
 	1    0    0    -1
@@
 F 5 "1%" H 8320 4720 50  0000 L CNN "Tolerance"
 F 6 "1/10W" H 8330 4640 50  0000 L CNN "Wattage"
-F 7 "" H 8220 4720 50  0001 C CNN "Digi-Key PN"
+F 7 "311-180KHRCT-ND" H 8220 4720 50  0001 C CNN "Digi-Key PN"
 	1    8220 4720
 	1    0    0    -1
@@
 F 5 "1%" V 7490 2710 50  0001 C CNN "Tolerance"
 F 6 "1/10W" V 7590 2710 50  0001 C CNN "Wattage"
-F 7 "" H 7290 2710 50  0001 C CNN "Digi-Key PN"
+F 7 "YAG2321CT-ND" H 7290 2710 50  0001 C CNN "Digi-Key PN"
 	1    7290 2710
 	-1   0    0    -1
@@
 F 5 "1%" V 7950 2710 50  0001 C CNN "Tolerance"
 F 6 "1/10W" V 8050 2710 50  0001 C CNN "Wattage"
-F 7 "" H 7750 2710 50  0001 C CNN "Digi-Key PN"
+F 7 "YAG2321CT-ND" H 7750 2710 50  0001 C CNN "Digi-Key PN"
 	1    7750 2710
 	-1   0    0    -1
@@
 F 5 "1%" H 4490 6980 50  0000 L CNN "Tolerance"
 F 6 "1/10W" H 4500 6900 50  0000 L CNN "Wattage"
-F 7 "" H 4690 7380 60  0001 C CNN "Digi-Key PN"
+F 7 "YAG2321CT-ND" H 4690 7380 60  0001 C CNN "Digi-Key PN"
 	1    4390 6980
 	1    0    0    -1
@@
 F 2 "Resistors_SMD:R_0603" H 2130 6700 50  0001 C CNN
 F 3 "" H 2130 6700 50  0001 C CNN
-F 4 "" H 2430 7100 60  0001 C CNN "Digi-Key PN"
+F 4 "YAG2321CT-ND" H 2430 7100 60  0001 C CNN "Digi-Key PN"
 F 5 "0603" V 2230 6700 50  0000 C CNN "display_footprint"
 F 6 "1%" V 2330 6700 50  0000 C CNN "Tolerance"
@@
 F 5 "1%" H 2870 3810 50  0000 L CNN "Tolerance"
 F 6 "1/10W" H 2880 3730 50  0000 L CNN "Wattage"
-F 7 "" H 3070 4210 60  0001 C CNN "Digi-Key PN"
+F 7 "YAG2321CT-ND" H 3070 4210 60  0001 C CNN "Digi-Key PN"
 	1    2770 3810
 	1    0    0    -1
