File: hdw/Analog_Clock/Function_LEDs.sch (KiCad schematic (older format))
At the start: 0 parts

Commit message: more analog work, added some more sch stuff
Parts:
- added C? (x4): 0.1uF, Capacitors_SMD:C_0402, symbol Custom_Library:C_Custom
- added R? (x4): 1k, Resistors_SMD:R_0402, symbol Custom_Library:R_Custom
- added R? (x4): 10k, Resistors_SMD:R_0402, symbol Custom_Library:R_Custom
- added U? (x4): 74LVC1G06, TO_SOT_Packages_SMD:SOT-353_SC-70-5, symbol Custom_Library:74LVC1G06_Power
Connections:
- net labels added: +3.3V, Function_Date_LED, Function_Time_LED, GND
- wire segments 0 -> 20

Commit message: big sch push
Parts:
- added D2301, D2302, D2303: Green, LEDs:LED_0603, symbol Device:LED
- added D2304: Yellow, LEDs:LED_0603, symbol Device:LED
- C2301, C2302, C2303, C2304: renamed from C?; footprint Capacitors_SMD:C_0402 -> Capacitors_SMD:C_0603; Digi-Key PN 490-10701-1-ND -> 399-7845-1-ND; display_footprint 0402 -> 0603
- R2301, R2302, R2305, R2306: renamed from R?; footprint Resistors_SMD:R_0402 -> Resistors_SMD:R_0603; Digi-Key PN RMCF0402FT10K0CT-ND -> (none); Wattage 1/16W -> 1/10W; display_footprint 0402 -> 0603
- R2303, R2304, R2307, R2308: renamed from R?; footprint Resistors_SMD:R_0402 -> Resistors_SMD:R_0603; Digi-Key PN 541-1.00KLCT-ND -> (none); Wattage 1/16W -> 1/10W; display_footprint 0402 -> 0603
- gave numbers to parts that had none: 4
Connections:
- net labels added: Alarm_Arm_LED, Function_Weekday_LED

Commit message: Much more schematic progress
Parts:
- R2301, R2302, R2305, R2306: Digi-Key PN (none) -> YAG2321CT-ND
- R2303, R2304, R2307, R2308: Digi-Key PN (none) -> 311-1.00KHRCT-ND
Changed lines of the file:
@@
 encoding utf-8
 Sheet 23 25
-Title ""
-Date ""
-Rev ""
-Comp ""
+Title "Analog Clock"
+Date "2020-08-15"
+Rev "A"
+Comp "Drew Maatman"
 Comment1 ""
 Comment2 ""
@@
 F 5 "1%" H 4790 2300 50  0000 L CNN "Tolerance"
 F 6 "1/10W" H 4790 2230 50  0000 L CNN "Wattage"
-F 7 "" H 5020 2700 60  0001 C CNN "Digi-Key PN"
+F 7 "311-1.00KHRCT-ND" H 5020 2700 60  0001 C CNN "Digi-Key PN"
 	1    4720 2300
 	-1   0    0    -1
@@
 F 5 "1%" H 3670 3100 50  0000 L CNN "Tolerance"
 F 6 "1/10W" H 3670 3030 50  0000 L CNN "Wattage"
-F 7 "" H 3600 3100 50  0001 C CNN "Digi-Key PN"
+F 7 "YAG2321CT-ND" H 3600 3100 50  0001 C CNN "Digi-Key PN"
 	1    3600 3100
 	-1   0    0    -1
@@
 F 5 "1%" H 6790 2300 50  0000 L CNN "Tolerance"
 F 6 "1/10W" H 6790 2230 50  0000 L CNN "Wattage"
-F 7 "" H 7020 2700 60  0001 C CNN "Digi-Key PN"
+F 7 "311-1.00KHRCT-ND" H 7020 2700 60  0001 C CNN "Digi-Key PN"
 	1    6720 2300
 	-1   0    0    -1
@@
 F 5 "1%" H 4790 4300 50  0000 L CNN "Tolerance"
 F 6 "1/10W" H 4790 4230 50  0000 L CNN "Wattage"
-F 7 "" H 5020 4700 60  0001 C CNN "Digi-Key PN"
+F 7 "311-1.00KHRCT-ND" H 5020 4700 60  0001 C CNN "Digi-Key PN"
 	1    4720 4300
 	-1   0    0    -1
@@
 F 5 "1%" H 3670 5100 50  0000 L CNN "Tolerance"
 F 6 "1/10W" H 3670 5030 50  0000 L CNN "Wattage"
-F 7 "" H 3600 5100 50  0001 C CNN "Digi-Key PN"
+F 7 "YAG2321CT-ND" H 3600 5100 50  0001 C CNN "Digi-Key PN"
 	1    3600 5100
 	-1   0    0    -1
@@
 F 5 "1%" H 6790 4300 50  0000 L CNN "Tolerance"
 F 6 "1/10W" H 6790 4230 50  0000 L CNN "Wattage"
-F 7 "" H 7020 4700 60  0001 C CNN "Digi-Key PN"
+F 7 "311-1.00KHRCT-ND" H 7020 4700 60  0001 C CNN "Digi-Key PN"
 	1    6720 4300
 	-1   0    0    -1
@@
 F 5 "1%" H 5670 5100 50  0000 L CNN "Tolerance"
 F 6 "1/10W" H 5670 5030 50  0000 L CNN "Wattage"
-F 7 "" H 5600 5100 50  0001 C CNN "Digi-Key PN"
+F 7 "YAG2321CT-ND" H 5600 5100 50  0001 C CNN "Digi-Key PN"
 	1    5600 5100
 	-1   0    0    -1
@@
 F 5 "1%" H 5670 3100 50  0000 L CNN "Tolerance"
 F 6 "1/10W" H 5670 3030 50  0000 L CNN "Wattage"
-F 7 "" H 5600 3100 50  0001 C CNN "Digi-Key PN"
+F 7 "YAG2321CT-ND" H 5600 3100 50  0001 C CNN "Digi-Key PN"
 	1    5600 3100
 	-1   0    0    -1
