File: hdw/Analog_Clock/LED_Driver.sch (KiCad schematic (older format))
At the start: 7 parts

Commit message: more analog work, added some more sch stuff
Parts:
- R?: value R -> 3.65k
Changed lines of the file:
@@
 $Descr A 11000 8500
 encoding utf-8
-Sheet 21 23
+Sheet 21 24
 Title ""
 Date ""
@@
 AR Path="/5F280E04/5F33A0D6" Ref="R?"  Part="1"
 F 0 "R?" H 4850 4430 50  0000 R CNN
-F 1 "R" V 4930 4430 40  0000 C CNN
+F 1 "3.65k" V 4930 4430 40  0000 C CNN
 F 2 "Resistors_SMD:R_0402" H 4930 4430 50  0001 C CNN
 F 3 "" H 4930 4430 50  0001 C CNN

Commit message: big sch push
Parts:
- C2101, C2102: renamed from C?; footprint Capacitors_SMD:C_0402 -> Capacitors_SMD:C_0603; Digi-Key PN 490-13211-1-ND -> 490-10474-1-ND; Voltage 6.3V -> 10V; display_footprint 0402 -> 0603
- C2103: renamed from C?; footprint Capacitors_SMD:C_0402 -> Capacitors_SMD:C_0603; Digi-Key PN 490-10701-1-ND -> 399-7845-1-ND; display_footprint (none) -> 0603
- R2101: renamed from R?; footprint Resistors_SMD:R_0402 -> Resistors_SMD:R_0603; Digi-Key PN RMCF0402FT10K0CT-ND -> (none); Wattage 1/16W -> 1/10W; display_footprint 0402 -> 0603
- R2102: renamed from R?; footprint Resistors_SMD:R_0402 -> Resistors_SMD:R_0603; Wattage 1/16W -> 1/10W; display_footprint 0402 -> 0603
- gave numbers to parts that had none: 2
Changed lines of the file:
@@
 $Descr A 11000 8500
 encoding utf-8
-Sheet 21 24
+Sheet 21 25
 Title ""
 Date ""
@@
 P 5690 3800
 AR Path="/5E98CF45/5F281117" Ref="U?"  Part="1"
-AR Path="/5F280E04/5F281117" Ref="U?"  Part="1"
-F 0 "U?" H 5390 4350 50  0000 L CNN
+AR Path="/5F280E04/5F281117" Ref="U2101"  Part="1"
+F 0 "U2101" H 5390 4350 50  0000 L CNN
 F 1 "LP5009" H 5740 4350 50  0000 L CNN
 F 2 "Housings_DFN_QFN:UQFN-20-1EP_3x3mm_Pitch0.4mm" H 5690 3700 50  0001 C CNN
@@
 METER0_LED_B
 $Comp
-L Custom_Library:I2C_Address DOC?
+L Custom_Library:I2C_Address DOC2101
 U 1 1 5F33042D
 P 6580 4660
-F 0 "DOC?" H 6580 4910 60  0001 C CNN
+F 0 "DOC2101" H 6580 4910 60  0001 C CNN
 F 1 "0x14" H 6130 4660 60  0000 L CNN
 F 2 "" H 6580 5010 60  0001 C CNN
@@
 $EndComp
 $Comp
-L power:GND #PWR?
+L power:GND #PWR02109
 U 1 1 5F3308CA
 P 5690 4400
-F 0 "#PWR?" H 5690 4150 50  0001 C CNN
+F 0 "#PWR02109" H 5690 4150 50  0001 C CNN
 F 1 "GND" H 5690 4250 50  0000 C CNN
 F 2 "" H 5690 4400 50  0001 C CNN
@@
 $EndComp
 $Comp
-L power:+3.3V #PWR?
+L power:+3.3V #PWR02108
 U 1 1 5F330E0D
 P 5690 3200
-F 0 "#PWR?" H 5690 3050 50  0001 C CNN
+F 0 "#PWR02108" H 5690 3050 50  0001 C CNN
 F 1 "+3.3V" H 5690 3340 50  0000 C CNN
 F 2 "" H 5690 3200 50  0001 C CNN
@@
 METER2_LED_B
 $Comp
-L power:GND #PWR?
+L power:GND #PWR02104
 U 1 1 5F3356DC
 P 5290 3800
-F 0 "#PWR?" H 5290 3550 50  0001 C CNN
+F 0 "#PWR02104" H 5290 3550 50  0001 C CNN
 F 1 "GND" V 5290 3650 50  0000 R CNN
 F 2 "" H 5290 3800 50  0001 C CNN
@@
 $EndComp
 $Comp
-L power:GND #PWR?
+L power:GND #PWR02105
 U 1 1 5F335B6C
 P 5290 3900
-F 0 "#PWR?" H 5290 3650 50  0001 C CNN
+F 0 "#PWR02105" H 5290 3650 50  0001 C CNN
 F 1 "GND" V 5290 3750 50  0000 R CNN
 F 2 "" H 5290 3900 50  0001 C CNN
@@
 AR Path="/5E939D31/5F33A0D6" Ref="R?"  Part="1"
 AR Path="/5E98CF45/5F33A0D6" Ref="R?"  Part="1"
-AR Path="/5F280E04/5F33A0D6" Ref="R?"  Part="1"
-F 0 "R?" H 4850 4430 50  0000 R CNN
+AR Path="/5F280E04/5F33A0D6" Ref="R2102"  Part="1"
+F 0 "R2102" H 4850 4430 50  0000 R CNN
 F 1 "3.65k" V 4930 4430 40  0000 C CNN
-F 2 "Resistors_SMD:R_0402" H 4930 4430 50  0001 C CNN
+F 2 "Resistors_SMD:R_0603" H 4930 4430 50  0001 C CNN
 F 3 "" H 4930 4430 50  0001 C CNN
-F 4 "0402" H 5030 4510 50  0000 L CNN "display_footprint"
+F 4 "0603" H 5030 4510 50  0000 L CNN "display_footprint"
 F 5 "0.1%" H 5030 4430 50  0000 L CNN "Tolerance"
-F 6 "1/16W" H 5040 4350 50  0000 L CNN "Wattage"
+F 6 "1/10W" H 5040 4350 50  0000 L CNN "Wattage"
 	1    4930 4430
 	1    0    0    -1
@@
 P 4930 4580
 AR Path="/5E98CF45/5F33A0DC" Ref="#PWR?"  Part="1"
-AR Path="/5F280E04/5F33A0DC" Ref="#PWR?"  Part="1"
-F 0 "#PWR?" H 4930 4330 50  0001 C CNN
+AR Path="/5F280E04/5F33A0DC" Ref="#PWR02103"  Part="1"
+F 0 "#PWR02103" H 4930 4330 50  0001 C CNN
 F 1 "GND" H 4930 4430 50  0000 C CNN
 F 2 "" H 4930 4580 50  0001 C CNN
@@
 P 4350 4580
 AR Path="/5E98CF45/5F33A0EC" Ref="#PWR?"  Part="1"
-AR Path="/5F280E04/5F33A0EC" Ref="#PWR?"  Part="1"
-F 0 "#PWR?" H 4350 4330 50  0001 C CNN
+AR Path="/5F280E04/5F33A0EC" Ref="#PWR02102"  Part="1"
+F 0 "#PWR02102" H 4350 4330 50  0001 C CNN
 F 1 "GND" H 4350 4430 50  0000 C CNN
 F 2 "" H 4350 4580 50  0001 C CNN
@@
 AR Path="/5EAE2D8A/5F33CF88" Ref="C?"  Part="1"
 AR Path="/5E939D31/5F33CF88" Ref="C?"  Part="1"
-AR Path="/5F280E04/5F33CF88" Ref="C?"  Part="1"
-F 0 "C?" H 4375 4530 50  0000 L CNN
+AR Path="/5F280E04/5F33CF88" Ref="C2101"  Part="1"
+F 0 "C2101" H 4375 4530 50  0000 L CNN
 F 1 "10uF" H 4375 4330 50  0000 L CNN
-F 2 "Capacitors_SMD:C_0402" H 4388 4280 50  0001 C CNN
+F 2 "Capacitors_SMD:C_0603" H 4388 4280 50  0001 C CNN
 F 3 "" H 4375 4530 50  0001 C CNN
-F 4 "0402" H 4200 4530 50  0000 R CNN "display_footprint"
-F 5 "6.3V" H 4200 4430 50  0000 R CNN "Voltage"
+F 4 "0603" H 4200 4530 50  0000 R CNN "display_footprint"
+F 5 "10V" H 4200 4430 50  0000 R CNN "Voltage"
 F 6 "X5R" H 4200 4330 50  0000 R CNN "Dielectric"
-F 7 "490-13211-1-ND" H 4350 4430 50  0001 C CNN "Digi-Key PN"
+F 7 "490-10474-1-ND" H 4350 4430 50  0001 C CNN "Digi-Key PN"
 	1    4350 4430
 	1    0    0    -1
@@
 P 3550 4580
 AR Path="/5E98CF45/5F3402F2" Ref="#PWR?"  Part="1"
-AR Path="/5F280E04/5F3402F2" Ref="#PWR?"  Part="1"
-F 0 "#PWR?" H 3550 4330 50  0001 C CNN
+AR Path="/5F280E04/5F3402F2" Ref="#PWR02101"  Part="1"
+F 0 "#PWR02101" H 3550 4330 50  0001 C CNN
 F 1 "GND" H 3550 4430 50  0000 C CNN
 F 2 "" H 3550 4580 50  0001 C CNN
@@
 AR Path="/5E939D31/5F342C1F" Ref="R?"  Part="1"
 AR Path="/5E98CF45/5F342C1F" Ref="R?"  Part="1"
-AR Path="/5F280E04/5F342C1F" Ref="R?"  Part="1"
-F 0 "R?" H 3470 4430 50  0000 R CNN
+AR Path="/5F280E04/5F342C1F" Ref="R2101"  Part="1"
+F 0 "R2101" H 3470 4430 50  0000 R CNN
 F 1 "10k" V 3550 4430 50  0000 C CNN
-F 2 "Resistors_SMD:R_0402" H 3550 4430 50  0001 C CNN
+F 2 "Resistors_SMD:R_0603" H 3550 4430 50  0001 C CNN
 F 3 "" H 3550 4430 50  0001 C CNN
-F 4 "0402" H 3650 4510 50  0000 L CNN "display_footprint"
+F 4 "0603" H 3650 4510 50  0000 L CNN "display_footprint"
 F 5 "1%" H 3650 4430 50  0000 L CNN "Tolerance"
-F 6 "1/16W" H 3660 4350 50  0000 L CNN "Wattage"
-F 7 "RMCF0402FT10K0CT-ND" H 3850 4830 60  0001 C CNN "Digi-Key PN"
+F 6 "1/10W" H 3660 4350 50  0000 L CNN "Wattage"
+F 7 "" H 3850 4830 60  0001 C CNN "Digi-Key PN"
 	1    3550 4430
 	1    0    0    -1
@@
 AR Path="/5E939D24/5F348653" Ref="C?"  Part="1"
 AR Path="/5E939D42/5F348653" Ref="C?"  Part="1"
-AR Path="/5F280E04/5F348653" Ref="C?"  Part="1"
-F 0 "C?" H 6095 2680 50  0000 L CNN
+AR Path="/5F280E04/5F348653" Ref="C2103"  Part="1"
+F 0 "C2103" H 6095 2680 50  0000 L CNN
 F 1 "0.1uF" H 6095 2480 50  0000 L CNN
-F 2 "Capacitors_SMD:C_0402" H 6108 2430 50  0001 C CNN
+F 2 "Capacitors_SMD:C_0603" H 6108 2430 50  0001 C CNN
 F 3 "" H 6095 2680 50  0001 C CNN
-F 4 "" H 5920 2680 50  0000 R CNN "display_footprint"
+F 4 "0603" H 5920 2680 50  0000 R CNN "display_footprint"
 F 5 "50V" H 5920 2580 50  0000 R CNN "Voltage"
 F 6 "X7R" H 5920 2480 50  0000 R CNN "Dielectric"
-F 7 "490-10701-1-ND" H 2160 -4300 50  0001 C CNN "Digi-Key PN"
+F 7 "399-7845-1-ND" H 2160 -4300 50  0001 C CNN "Digi-Key PN"
 	1    6070 2580
 	1    0    0    -1
@@
 AR Path="/5E939D24/5F348659" Ref="#PWR?"  Part="1"
 AR Path="/5E939D42/5F348659" Ref="#PWR?"  Part="1"
-AR Path="/5F280E04/5F348659" Ref="#PWR?"  Part="1"
-F 0 "#PWR?" H 6070 2280 50  0001 C CNN
+AR Path="/5F280E04/5F348659" Ref="#PWR02110"  Part="1"
+F 0 "#PWR02110" H 6070 2280 50  0001 C CNN
 F 1 "+3.3V" H 6070 2570 50  0000 C CNN
 F 2 "" H 6070 2430 50  0001 C CNN
@@
 AR Path="/5E939D24/5F34865F" Ref="#PWR?"  Part="1"
 AR Path="/5E939D42/5F34865F" Ref="#PWR?"  Part="1"
-AR Path="/5F280E04/5F34865F" Ref="#PWR?"  Part="1"
-F 0 "#PWR?" H 6070 2480 50  0001 C CNN
+AR Path="/5F280E04/5F34865F" Ref="#PWR02111"  Part="1"
+F 0 "#PWR02111" H 6070 2480 50  0001 C CNN
 F 1 "GND" H 6070 2580 50  0000 C CNN
 F 2 "" H 6070 2730 50  0001 C CNN
@@
 $EndComp
 $Comp
-L power:GND #PWR?
+L power:GND #PWR02107
 U 1 1 5F34ADB6
 P 5300 2730
-F 0 "#PWR?" H 5300 2480 50  0001 C CNN
+F 0 "#PWR02107" H 5300 2480 50  0001 C CNN
 F 1 "GND" H 5300 2580 50  0000 C CNN
 F 2 "" H 5300 2730 50  0001 C CNN
@@
 AR Path="/5EAE2D8A/5F34ADC0" Ref="C?"  Part="1"
 AR Path="/5E939D31/5F34ADC0" Ref="C?"  Part="1"
-AR Path="/5F280E04/5F34ADC0" Ref="C?"  Part="1"
-F 0 "C?" H 5325 2680 50  0000 L CNN
+AR Path="/5F280E04/5F34ADC0" Ref="C2102"  Part="1"
+F 0 "C2102" H 5325 2680 50  0000 L CNN
 F 1 "10uF" H 5325 2480 50  0000 L CNN
-F 2 "Capacitors_SMD:C_0402" H 5338 2430 50  0001 C CNN
+F 2 "Capacitors_SMD:C_0603" H 5338 2430 50  0001 C CNN
 F 3 "" H 5325 2680 50  0001 C CNN
-F 4 "0402" H 5150 2680 50  0000 R CNN "display_footprint"
-F 5 "6.3V" H 5150 2580 50  0000 R CNN "Voltage"
+F 4 "0603" H 5150 2680 50  0000 R CNN "display_footprint"
+F 5 "10V" H 5150 2580 50  0000 R CNN "Voltage"
 F 6 "X5R" H 5150 2480 50  0000 R CNN "Dielectric"
-F 7 "490-13211-1-ND" H 5300 2580 50  0001 C CNN "Digi-Key PN"
+F 7 "490-10474-1-ND" H 5300 2580 50  0001 C CNN "Digi-Key PN"
 	1    5300 2580
 	1    0    0    -1
@@
 AR Path="/5E939D24/5F34AE43" Ref="#PWR?"  Part="1"
 AR Path="/5E939D42/5F34AE43" Ref="#PWR?"  Part="1"
-AR Path="/5F280E04/5F34AE43" Ref="#PWR?"  Part="1"
-F 0 "#PWR?" H 5300 2280 50  0001 C CNN
+AR Path="/5F280E04/5F34AE43" Ref="#PWR02106"  Part="1"
+F 0 "#PWR02106" H 5300 2280 50  0001 C CNN
 F 1 "+3.3V" H 5300 2570 50  0000 C CNN
 F 2 "" H 5300 2430 50  0001 C CNN

Commit message: Much more schematic progress
Parts:
- R2101: Digi-Key PN (none) -> YAG2321CT-ND
- R2102: Digi-Key PN (none) -> YAG4547CT-ND
Changed lines of the file:
@@
 encoding utf-8
 Sheet 21 25
-Title ""
-Date ""
-Rev ""
-Comp ""
+Title "Analog Clock"
+Date "2020-08-15"
+Rev "A"
+Comp "Drew Maatman"
 Comment1 ""
 Comment2 ""
@@
 F 5 "0.1%" H 5030 4430 50  0000 L CNN "Tolerance"
 F 6 "1/10W" H 5040 4350 50  0000 L CNN "Wattage"
+F 7 "YAG4547CT-ND" H 4930 4430 50  0001 C CNN "Digi-Key PN"
 	1    4930 4430
 	1    0    0    -1
@@
 F 5 "1%" H 3650 4430 50  0000 L CNN "Tolerance"
 F 6 "1/10W" H 3660 4350 50  0000 L CNN "Wattage"
-F 7 "" H 3850 4830 60  0001 C CNN "Digi-Key PN"
+F 7 "YAG2321CT-ND" H 3850 4830 60  0001 C CNN "Digi-Key PN"
 	1    3550 4430
 	1    0    0    -1
