File: hdw/Analog_Clock/Meter0.sch (KiCad schematic (older format))
At the start: 43 parts

Commit message: more analog work, added some more sch stuff
Connections:
- net DAC0_VREF: now reaches C?.1, C?.1, U?.2 (VREF), U?.6 (Vout)
Changed lines of the file:
@@
 $Descr A 11000 8500
 encoding utf-8
-Sheet 18 23
+Sheet 18 24
 Title ""
 Date ""
@@
 Text GLabel 3250 6740 3    50   UnSpc ~ 0
 METER0_LED_B
+Text GLabel 4880 1850 2    50   Output ~ 0
+DAC0_VREF
+Wire Wire Line
+	4880 1850 4800 1850
+Connection ~ 4800 1850
 $EndSCHEMATC

Commit message: big sch push
Parts:
- removed C? (x2): 47pF, symbol Custom_Library:C_Custom
- removed C? (x3): 0.1uF, Capacitors_SMD:C_0402, symbol Custom_Library:C_Custom
- removed C?: 4.7uF, Capacitors_SMD:C_0805, symbol Custom_Library:C_Custom
- removed C?: 1nF, Capacitors_SMD:C_0402, symbol Custom_Library:C_Custom
- removed C?: 10nF, Capacitors_SMD:C_0402, symbol Custom_Library:C_Custom
- removed D?: DZ2S033X0L, Diode_SMD:D_SOD-523, symbol Diode:DZ2S033X0L
- removed L?: 600R 0.5A, Inductors_SMD:L_0402, symbol Device:Ferrite_Bead
- removed MK? (x4): Standoff, symbol Custom_Library:Standoff
- removed MK? (x8): Screw, symbol Custom_Library:Screw
- removed R? (x2): 10, Resistors_SMD:R_0402, symbol Custom_Library:R_Custom
- removed R?: 10k, Resistors_SMD:R_0402, symbol Custom_Library:R_Custom
- removed R?: 1k, Resistors_SMD:R_0402, symbol Custom_Library:R_Custom
- removed R?: 1.01k, Resistors_SMD:R_0402, symbol Custom_Library:R_Custom
- removed R?: 9.09k, symbol Custom_Library:R_Custom
- removed U?: DAC8551, Package_SO:VSSOP-8_3.0x3.0mm_P0.65mm, symbol Custom_Library:DAC8551
- removed U?: LT1790-2.048, Package_TO_SOT_SMD:TSOT-23-6, symbol Reference_Voltage:LT1790-2.048
- removed U? (x3): OPA2197xDGK, Package_SO:VSSOP-8_3.0x3.0mm_P0.65mm, symbol Amplifier_Operational:OPA2197xDGK
- added C1801, C1802, C1806, C1807, C1812: 0.1uF, Capacitors_SMD:C_0603, symbol Custom_Library:C_Custom
- added C1804: 4.7uF, Capacitors_SMD:C_0805, symbol Custom_Library:C_Custom
- added C1805: 47pF, Capacitors_SMD:C_0603, symbol Custom_Library:C_Custom
- added C1809: 10nF, Capacitors_SMD:C_0603, symbol Custom_Library:C_Custom
- added C1810: 1nF, Capacitors_SMD:C_0603, symbol Custom_Library:C_Custom
- added D1801: Green, LEDs:LED_0603, symbol Device:LED
- added D1803: BZX384-B3V3,115, Diode_SMD:D_SOD-323, symbol Diode:DZ2S033X0L
- added L1801: 600R 0.5A, Inductors_SMD:L_0603, symbol Device:Ferrite_Bead
- added MK1801, MK1802, MK1805, MK1806, MK1807, MK1808, MK1811, MK1812: #4-40 Screw, symbol Custom_Library:Screw
- added MK1803, MK1804, MK1809, MK1810: #4-40 Standoff, symbol Custom_Library:Standoff
- added R1802, R1803: 10, Resistors_SMD:R_0603, symbol Custom_Library:R_Custom
- added R1806, R1812: 1k, Resistors_SMD:R_0603, symbol Custom_Library:R_Custom
- added R1807: 10k, Resistors_SMD:R_0603, symbol Custom_Library:R_Custom
- added R1808: 1.01k, Resistors_SMD:R_0603, symbol Custom_Library:R_Custom
- added R1810: 9.09k, Resistors_SMD:R_0603, symbol Custom_Library:R_Custom
- added TP1801: TP_Pad, Custom Footprints Library:Test_Point, symbol Custom_Library:TP_Pad
- added U1801: 74LVC1G07, TO_SOT_Packages_SMD:SOT-353_SC-70-5, symbol Custom_Library:74LVC1G07_Power
- added U1802: LT1790-2.048, Package_TO_SOT_SMD:TSOT-23-6, symbol Reference_Voltage:LT1790-2.048
- added U1803: DAC8551, Package_SO:VSSOP-8_3.0x3.0mm_P0.65mm, symbol Custom_Library:DAC8551
- added U1804: OPA2197xDGK, Package_SO:VSSOP-8_3.0x3.0mm_P0.65mm, symbol Amplifier_Operational:OPA2197xDGK
- C1808, C1811: renamed from C?; footprint Capacitors_SMD:C_0402 -> Capacitors_SMD:C_0603; Digi-Key PN 490-10701-1-ND -> 399-7845-1-ND; display_footprint 0402 -> 0603
- D1802: renamed from D?; Digi-Key PN (none) -> 516-3279-1-ND
- R1801, R1809: renamed from R?; footprint Resistors_SMD:R_0402 -> Resistors_SMD:R_0603; Wattage 1/16W -> 1/10W; display_footprint 0402 -> 0603
- R1804, R1805: renamed from R?; footprint Resistors_SMD:R_0402 -> Resistors_SMD:R_0603; Digi-Key PN RMCF0402FT10K0CT-ND -> (none); Wattage 1/16W -> 1/10W; display_footprint 0402 -> 0603
- R1811: renamed from R?; footprint (none) -> Resistors_SMD:R_0603; Wattage 1/16W -> 1/10W; display_footprint 0402 -> 0603
- gave numbers to parts that had none: 2
Connections:
- net +20V: now also C1809.1, C1810.1, U1804.8 (V+)
- net +3V3: now also C1801.1, C1802.1, L1801.2, R1806.1, U1801.5 (VCC), U1802.4 (Vin)
- net DAC0_VREF: now also C1805.1, TP1801.1 (TP), U1802.6 (Vout), U1803.2 (VREF)
- net DAC_SPI_MOSI: now also R1802.1
- net DAC_SPI_SCLK: now also R1803.1
- net GND: now also C1801.2, C1802.2, C1804.2, C1805.2, C1806.2, C1807.2, C1809.2, C1810.2, C1812.2, D1803.2 (A), R1807.2, R1808.2, U1801.3 (GND), U1802.1 (GND), U1802.2 (GND), U1803.8 (GND), U1803.9 (GND), U1804.4 (V-)
- net VDAC_0_ADC: now also C1812.1, D1803.1 (K), R1812.1
- net ~DAC_SPI_SYNC_0: now also U1801.2
- net at R1801.2, R1804.2: now also U1803.5 (~SYNC)
- net at R1805.1: now also R1802.2, U1803.7 (DIN)
- net at C1811.1, MES1801.2 (+), R1811.1: now also R1810.1, U1804.1
- net at C1811.2, R1809.1, R1811.2: now also U1804.2 (-)
- new net: D1801.1 (K), U1801.4
- new net: C1804.1, C1806.1, L1801.1, U1803.1 (VDD)
- new net: U1803.3 (VFB), U1803.4 (VOUT), U1804.3 (+)
- new net: R1803.2, R1807.1, U1803.6 (SCLK)
- new net: C1807.1, R1808.1, R1810.2, U1804.5 (+)
- new net: R1812.2, U1804.6 (-), U1804.7
- new net: D1801.2 (A), R1806.2
Other:
- note added: "15V Full Scale"
- moved on the sheet: D1802

Commit message: Much more schematic progress
Parts:
- MES1801: footprint (none) -> FIX ME
- R1801, R1802, R1803, R1804, R1805, R1807: Digi-Key PN (none) -> YAG2321CT-ND
- R1806, R1812: Digi-Key PN (none) -> 311-1.00KHRCT-ND
- R1808, R1809: Digi-Key PN (none) -> YAG4489CT-ND
- R1810, R1811: Digi-Key PN PN -> YAG1755CT-ND
Changed lines of the file:
@@
 encoding utf-8
 Sheet 18 25
-Title ""
-Date ""
-Rev ""
-Comp ""
+Title "Analog Clock"
+Date "2020-08-15"
+Rev "A"
+Comp "Drew Maatman"
 Comment1 ""
 Comment2 ""
@@
 F 5 "1%" V 2530 3680 50  0001 C CNN "Tolerance"
 F 6 "1/10W" V 2630 3680 50  0001 C CNN "Wattage"
+F 7 "YAG2321CT-ND" H 2330 3680 50  0001 C CNN "Digi-Key PN"
 	1    2330 3680
 	0    -1   1    0
@@
 F 5 "1%" V 2530 3580 50  0001 C CNN "Tolerance"
 F 6 "1/10W" V 2630 3580 50  0001 C CNN "Wattage"
+F 7 "YAG2321CT-ND" H 2330 3580 50  0001 C CNN "Digi-Key PN"
 	1    2330 3580
 	0    -1   1    0
@@
 F 5 "1%" V 2530 3480 50  0001 C CNN "Tolerance"
 F 6 "1/10W" V 2630 3480 50  0001 C CNN "Wattage"
+F 7 "YAG2321CT-ND" H 2330 3480 50  0001 C CNN "Digi-Key PN"
 	1    2330 3480
 	0    -1   1    0
@@
 F 5 "1%" H 2930 3250 50  0000 L CNN "Tolerance"
 F 6 "1/10W" H 2940 3170 50  0000 L CNN "Wattage"
-F 7 "" H 3130 3650 60  0001 C CNN "Digi-Key PN"
+F 7 "YAG2321CT-ND" H 3130 3650 60  0001 C CNN "Digi-Key PN"
 	1    2830 3250
 	1    0    0    -1
@@
 F 5 "1%" H 3670 3910 50  0000 L CNN "Tolerance"
 F 6 "1/10W" H 3680 3830 50  0000 L CNN "Wattage"
-F 7 "" H 3870 4310 60  0001 C CNN "Digi-Key PN"
+F 7 "YAG2321CT-ND" H 3870 4310 60  0001 C CNN "Digi-Key PN"
 	1    3570 3910
 	1    0    0    -1
@@
 F 5 "1%" H 2930 3910 50  0000 L CNN "Tolerance"
 F 6 "1/10W" H 2940 3830 50  0000 L CNN "Wattage"
-F 7 "" H 3130 4310 60  0001 C CNN "Digi-Key PN"
+F 7 "YAG2321CT-ND" H 3130 4310 60  0001 C CNN "Digi-Key PN"
 	1    2830 3910
 	1    0    0    -1
@@
 F 5 "0.1%" V 7110 2630 50  0000 C CNN "Tolerance"
 F 6 "1/10W" V 7210 2630 50  0000 C CNN "Wattage"
-F 7 "PN" H 7210 3030 60  0001 C CNN "Digi-Key PN"
+F 7 "YAG1755CT-ND" H 7210 3030 60  0001 C CNN "Digi-Key PN"
 	1    6910 2630
 	0    1    -1   0
@@
 F 5 "0.1%" H 6200 3210 50  0000 L CNN "Tolerance"
 F 6 "1/10W" H 6210 3130 50  0000 L CNN "Wattage"
+F 7 "YAG4489CT-ND" H 6100 3210 50  0001 C CNN "Digi-Key PN"
 	1    6100 3210
 	1    0    0    -1
@@
 F 5 "1%" V 7570 4510 50  0000 C CNN "Tolerance"
 F 6 "1/10W" V 7670 4510 50  0000 C CNN "Wattage"
-F 7 "" H 7670 4910 60  0001 C CNN "Digi-Key PN"
+F 7 "311-1.00KHRCT-ND" H 7670 4910 60  0001 C CNN "Digi-Key PN"
 	1    7370 4510
 	0    1    1    0
@@
 F 0 "MES1801" H 8270 2270 50  0000 R CNN
 F 1 "Voltmeter_DC" H 8270 2200 50  0000 R CNN
-F 2 "" V 8400 2330 50  0001 C CNN
+F 2 "FIX ME" V 8400 2330 50  0001 C CNN
 F 3 "~" V 8400 2330 50  0001 C CNN
 	1    8400 2230
@@
 F 5 "0.1%" H 5770 4740 50  0000 L CNN "Tolerance"
 F 6 "1/10W" H 5780 4660 50  0000 L CNN "Wattage"
+F 7 "YAG4489CT-ND" H 5670 4740 50  0001 C CNN "Digi-Key PN"
 	1    5670 4740
 	1    0    0    -1
@@
 F 5 "0.1%" V 6730 4020 50  0000 C CNN "Tolerance"
 F 6 "1/10W" V 6830 4020 50  0000 C CNN "Wattage"
-F 7 "PN" H 6830 4420 60  0001 C CNN "Digi-Key PN"
+F 7 "YAG1755CT-ND" H 6830 4420 60  0001 C CNN "Digi-Key PN"
 	1    6530 4020
 	0    1    -1   0
@@
 F 5 "1%" H 2960 5880 50  0000 L CNN "Tolerance"
 F 6 "1/10W" H 2960 5810 50  0000 L CNN "Wattage"
-F 7 "" H 3190 6280 60  0001 C CNN "Digi-Key PN"
+F 7 "311-1.00KHRCT-ND" H 3190 6280 60  0001 C CNN "Digi-Key PN"
 	1    2890 5880
 	-1   0    0    -1

Commit message: made netlist, started PCB
Parts:
- MES1801: footprint FIX ME -> (none)
Changed lines of the file:
@@
 F 0 "MES1801" H 8270 2270 50  0000 R CNN
 F 1 "Voltmeter_DC" H 8270 2200 50  0000 R CNN
-F 2 "FIX ME" V 8400 2330 50  0001 C CNN
+F 2 "" V 8400 2330 50  0001 C CNN
 F 3 "~" V 8400 2330 50  0001 C CNN
 	1    8400 2230

Commit message: more PCB grouping
Parts:
- MES1801: footprint (none) -> Custom Footprints Library:SO-45_Panel_Meter
Changed lines of the file:
@@
 F 0 "MES1801" H 8270 2270 50  0000 R CNN
 F 1 "Voltmeter_DC" H 8270 2200 50  0000 R CNN
-F 2 "" V 8400 2330 50  0001 C CNN
+F 2 "Custom Footprints Library:SO-45_Panel_Meter" V 8400 2330 50  0001 C CNN
 F 3 "~" V 8400 2330 50  0001 C CNN
 	1    8400 2230

Commit message: Major USB restructuring
Parts:
- U1804: symbol Amplifier_Operational:OPA2197xDGK -> Custom_Library:OPA2197xDGK
Changed lines of the file:
@@
 $Descr A 11000 8500
 encoding utf-8
-Sheet 18 24
+Sheet 15 25
 Title "Analog Clock"
 Date "2020-08-15"
@@
 Connection ~ 6100 2630
 $Comp
-L Amplifier_Operational:OPA2197xDGK U1804
-U 1 1 5F4617C6
-P 6480 1950
-F 0 "U1804" H 6480 2310 50  0000 L CNN
-F 1 "OPA2197xDGK" H 6480 2150 50  0000 L CNN
-F 2 "Package_SO:VSSOP-8_3.0x3.0mm_P0.65mm" H 6480 1950 50  0001 C CNN
-F 3 "http://www.ti.com/lit/ds/symlink/opa2197.pdf" H 6480 1950 50  0001 C CNN
-F 4 "296-44774-1-ND" H 6480 1950 50  0001 C CNN "Digi-Key PN"
-	1    6480 1950
-	1    0    0    -1
-$EndComp
-$Comp
-L Amplifier_Operational:OPA2197xDGK U1804
+L Custom_Library:OPA2197xDGK U1804
 U 3 1 5F4617C7
 P 6480 1950
@@
 $EndComp
 $Comp
-L Amplifier_Operational:OPA2197xDGK U1804
+L Custom_Library:OPA2197xDGK U1804
 U 2 1 5F4617C9
 P 6480 4510
@@
 	4600 2600 4600 2680
 Connection ~ 4600 2680
+$Comp
+L Custom_Library:OPA2197xDGK U1804
+U 1 1 5F4617C6
+P 6480 1950
+F 0 "U1804" H 6480 2310 50  0000 L CNN
+F 1 "OPA2197xDGK" H 6480 2150 50  0000 L CNN
+F 2 "Package_SO:VSSOP-8_3.0x3.0mm_P0.65mm" H 6480 1950 50  0001 C CNN
+F 3 "http://www.ti.com/lit/ds/symlink/opa2197.pdf" H 6480 1950 50  0001 C CNN
+F 4 "296-44774-1-ND" H 6480 1950 50  0001 C CNN "Digi-Key PN"
+	1    6480 1950
+	1    0    0    -1
+$EndComp
 $EndSCHEMATC
