File: hdw/Analog_Clock/Misc_Circuits.sch (KiCad schematic (older format))
At the start: 5 parts

Commit message: big sch push
Parts:
- removed C?: 0.1uF, Capacitors_SMD:C_0402, symbol Custom_Library:C_Custom
- removed DOC?: FIX ME, symbol Custom_Library:I2C_Address
- removed R?: 10k, Resistors_SMD:R_0402, symbol Custom_Library:R_Custom
- removed R?: 10, Resistors_SMD:R_0402, symbol Custom_Library:R_Custom
- removed U?: MCP9804, Package_DFN_QFN:DFN-8-1EP_3x2mm_P0.5mm_EP1.3x1.5mm, symbol Sensor_Temperature:MCP9804_DFN
- added BZ2401: CST-931RP-A, Buzzer_Beeper:MagneticBuzzer_CUI_CST-931RP-A, symbol Device:Buzzer
- added C2401, C2402, C2403: 0.1uF, Capacitors_SMD:C_0603, symbol Custom_Library:C_Custom
- added D2401: MBR0580, Diode_SMD:D_SOD-123, symbol Diode:MBR0580
- added DOC2401: 0x1C, symbol Custom_Library:I2C_Address
- added J2401: I2C, Pin_Headers:Pin_Header_Straight_1x03_Pitch2.54mm, symbol Connector_Generic:Conn_01x03
- added J2402: USB UART, Pin_Headers:Pin_Header_Straight_1x03_Pitch2.54mm, symbol Connector_Generic:Conn_01x03
- added J2403: DAC SPI, Pin_Headers:Pin_Header_Straight_1x03_Pitch2.54mm, symbol Connector_Generic:Conn_01x03
- added Q2401: BSS214NW, TO_SOT_Packages_SMD:SOT-323_SC-70, symbol Transistor_FET:BSS214NW
- added R2401: 1.07M, Resistors_SMD:R_0603, symbol Custom_Library:R_Custom
- added R2402, R2403, R2405, R2407: 10k, Resistors_SMD:R_0603, symbol Custom_Library:R_Custom
- added R2404, R2406: 10, Resistors_SMD:R_0603, symbol Custom_Library:R_Custom
- added U2401: LTC6900, Package_TO_SOT_SMD:SOT-23-5, symbol Custom_Library:LTC6900
- added U2402: 74LVC1G08, Package_TO_SOT_SMD:SOT-353_SC-70-5, symbol Custom_Library:74LVC1G08_Power
- added U2403: MCP9804, Package_DFN_QFN:DFN-8-1EP_3x2mm_P0.5mm_EP1.3x1.5mm, symbol Sensor_Temperature:MCP9804_DFN
Connections:
- net +3V3: now also BZ2401.1 (-), C2401.1, C2402.1, C2403.1, D2401.1 (K), R2401.1, R2403.1, U2401.1 (V+), U2401.4 (DIV), U2402.5 (VCC), U2403.5 (A2), U2403.8 (VDD)
- net GND: now also C2401.2, C2402.2, C2403.2, J2401.3 (Pin_3), J2402.3 (Pin_3), J2403.3 (Pin_3), Q2401.2 (S), R2402.1, R2404.2, R2405.1, R2407.1, U2401.2 (GND), U2402.3 (GND), U2403.4 (GND), U2403.6 (A1), U2403.7 (A0), U2403.9 (EP/GND)
- net I2C_SCL: now also J2401.1 (Pin_1), U2403.2 (SCL)
- net I2C_SDA: now also J2401.2 (Pin_2), U2403.1 (SDA)
- net Telemetry_Hardstrap: now also R2403.2, R2404.1
- new net: BZ2401.2 (+), D2401.2 (A), Q2401.3 (D)
- new net: Q2401.1 (G), R2406.1, R2407.2
- new net: R2402.2, U2401.5 (OUT), U2402.1
- new net: R2406.2, U2402.4
- new net: R2401.2, U2401.3 (SET)
- new net Buzzer_Enable: R2405.2, U2402.2
- new net DAC_SPI_MOSI: J2403.1 (Pin_1)
- new net DAC_SPI_SCLK: J2403.2 (Pin_2)
- new net USB_UART_RX: J2402.2 (Pin_2)
- new net USB_UART_TX: J2402.1 (Pin_1)
Other:
- note added: "Fosc ~~ 2kHz"
- note added: "Place away from power components"
- note removed: "Add alarm?"
- note removed: "High for no telemetry installed,\nLow for telemetry sensors installed"

Commit message: Much more schematic progress
Parts:
- R2401: Digi-Key PN (none) -> RMCF0603FT1M07CT-ND
- R2402, R2403, R2405, R2406, R2407: Digi-Key PN (none) -> YAG2321CT-ND
Changed lines of the file:
@@
 encoding utf-8
 Sheet 24 25
-Title ""
-Date ""
-Rev ""
-Comp ""
+Title "Analog Clock"
+Date "2020-08-15"
+Rev "A"
+Comp "Drew Maatman"
 Comment1 ""
 Comment2 ""
@@
 F 5 "1%" H 5450 5490 50  0000 L CNN "Tolerance"
 F 6 "1/10W" H 5450 5420 50  0000 L CNN "Wattage"
-F 7 "" H 1290 -100 50  0001 C CNN "Digi-Key PN"
+F 7 "YAG2321CT-ND" H 1290 -100 50  0001 C CNN "Digi-Key PN"
 	1    5380 5490
 	-1   0    0    1
@@
 F 5 "1%" H 4820 5490 50  0000 L CNN "Tolerance"
 F 6 "1/10W" H 4820 5420 50  0000 L CNN "Wattage"
-F 7 "" H 660 -100 50  0001 C CNN "Digi-Key PN"
+F 7 "YAG2321CT-ND" H 660 -100 50  0001 C CNN "Digi-Key PN"
 	1    4750 5490
 	-1   0    0    1
@@
 F 5 "1%" H 7600 5440 50  0000 L CNN "Tolerance"
 F 6 "1/10W" H 7600 5370 50  0000 L CNN "Wattage"
-F 7 "" H 3440 -150 50  0001 C CNN "Digi-Key PN"
+F 7 "YAG2321CT-ND" H 3440 -150 50  0001 C CNN "Digi-Key PN"
 	1    7530 5440
 	-1   0    0    1
@@
 F 2 "Resistors_SMD:R_0603" H 6900 5210 50  0001 C CNN
 F 3 "" H 6900 5210 50  0001 C CNN
-F 4 "" H 7200 5610 60  0001 C CNN "Digi-Key PN"
+F 4 "YAG2321CT-ND" H 7200 5610 60  0001 C CNN "Digi-Key PN"
 F 5 "0603" V 7000 5210 50  0000 C CNN "display_footprint"
 F 6 "1%" V 7100 5210 50  0000 C CNN "Tolerance"
@@
 F 5 "1%" H 2540 4830 50  0000 L CNN "Tolerance"
 F 6 "1/10W" H 2550 4750 50  0000 L CNN "Wattage"
-F 7 "" H 2440 4830 50  0001 C CNN "Digi-Key PN"
+F 7 "RMCF0603FT1M07CT-ND" H 2440 4830 50  0001 C CNN "Digi-Key PN"
 	1    2440 4830
 	-1   0    0    -1
@@
 F 5 "1%" H 5010 3200 50  0000 L CNN "Tolerance"
 F 6 "1/10W" H 5020 3120 50  0000 L CNN "Wattage"
-F 7 "" H 5210 3600 60  0001 C CNN "Digi-Key PN"
+F 7 "YAG2321CT-ND" H 5210 3600 60  0001 C CNN "Digi-Key PN"
 	1    4910 3200
 	1    0    0    -1
