File: hdw/Analog_Clock/PGOOD_LEDs.sch (KiCad schematic (older format))
At the start: 22 parts

Commit message: More schematic work
Parts:
- removed C?: 4.7uF, Capacitors_SMD:C_0805, symbol Custom_Library:C_Custom
- removed U? (x4): 74LVC1G97, Package_TO_SOT_SMD:SOT-363_SC-70-6, symbol Custom_Library:74LVC1G97_Power_NOT
- removed U?: 74LVC1G97, Package_TO_SOT_SMD:SOT-363_SC-70-6, symbol Custom_Library:74LVC1G97_Power_BUF
- added C?: 4.7uF, Capacitors_SMD:C_0603, symbol Custom_Library:C_Custom
- added U? (x5): 74LVC1G06, TO_SOT_Packages_SMD:SOT-353_SC-70-5, symbol Custom_Library:74LVC1G06_Power
Other:
- moved on the sheet: C?, D?, R?

Commit message: More sch work
Parts:
- removed C?: 0.1uF, Capacitors_SMD:C_0402, symbol Custom_Library:C_Custom
- removed C?: 4.7uF, Capacitors_SMD:C_0603, symbol Custom_Library:C_Custom
- removed U?: TPS71533, Package_TO_SOT_SMD:SOT-353_SC-70-5, symbol Regulator_Linear:TPS71533__SC70
- added C?: 0.1uF, Capacitors_SMD:C_0402, symbol Custom_Library:C_Custom
- added C? (x2): 4.7uF, Capacitors_SMD:C_0805, symbol Custom_Library:C_Custom
- added Q?: BSS214NW, Package_TO_SOT_SMD:SOT-323_SC-70, symbol Transistor_FET:BSS214NW
- added R? (x2): 10k, Resistors_SMD:R_0402, symbol Custom_Library:R_Custom
- added R?: 10, Resistors_SMD:R_0402, symbol Custom_Library:R_Custom
- added U?: LP2985-3.3, Package_TO_SOT_SMD:SOT-23-5, symbol Regulator_Linear:LP2985-3.3
Connections:
- net labels added: +3.3V_PGL, POS3P3_PGL_SHDN
- wire segments 19 -> 22
- no-connect marks 0 -> 1

Commit message: more sch progress
Parts:
- removed U?: 74LVC1G06, TO_SOT_Packages_SMD:SOT-353_SC-70-5, symbol Custom_Library:74LVC1G06_Power
- added U?: 74LVC1G07, TO_SOT_Packages_SMD:SOT-353_SC-70-5, symbol Custom_Library:74LVC1G07_Power
Connections:
- net +3V3: now also U?.5 (VCC)
- net GND: now also U?.3 (GND)
- net VBAT_PGOOD: now also U?.2
- net at D?.1 (K): now also U?.4
- net POS5_PGOOD renamed POS20_PGOOD

Commit message: big sch push
Parts:
- C1602, C1603, C1605, C1606, C1607: renamed from C?; footprint Capacitors_SMD:C_0402 -> Capacitors_SMD:C_0603; Digi-Key PN 490-10701-1-ND -> 399-7845-1-ND; display_footprint 0402 -> 0603
- D1601, D1602, D1603, D1605: renamed from D?; footprint (none) -> LEDs:LED_0603; Digi-Key PN (none) -> 754-1121-1-ND
- D1604: renamed from D?; footprint (none) -> LEDs:LED_0603; Digi-Key PN (none) -> 754-1117-1-ND
- R1601: renamed from R?; footprint Resistors_SMD:R_0402 -> Resistors_SMD:R_0603; Digi-Key PN 541-3964-1-ND -> (none); Wattage 1/16W -> 1/10W; display_footprint 0402 -> 0603
- R1602, R1603: renamed from R?; footprint Resistors_SMD:R_0402 -> Resistors_SMD:R_0603; Digi-Key PN RMCF0402FT10K0CT-ND -> (none); Wattage 1/16W -> 1/10W; display_footprint 0402 -> 0603
- R1604, R1605, R1606, R1607, R1608: renamed from R?; footprint Resistors_SMD:R_0402 -> Resistors_SMD:R_0603; Digi-Key PN 541-1.00KLCT-ND -> (none); Wattage 1/16W -> 1/10W; display_footprint 0402 -> 0603
- U1603: renamed from U?; Digi-Key PN (none) -> LP2985IM5X-3.3/NOPBCT-ND
- gave numbers to parts that had none: 8

Commit message: Much more schematic progress
Parts:
- R1601, R1602, R1603: Digi-Key PN (none) -> YAG2321CT-ND
- R1604, R1605, R1606, R1607, R1608: Digi-Key PN (none) -> 311-1.00KHRCT-ND
Changed lines of the file:
@@
 encoding utf-8
 Sheet 16 25
-Title ""
-Date ""
-Rev ""
-Comp ""
+Title "Analog Clock"
+Date "2020-08-15"
+Rev "A"
+Comp "Drew Maatman"
 Comment1 ""
 Comment2 ""
@@
 F 5 "1%" H 3620 2300 50  0000 L CNN "Tolerance"
 F 6 "1/10W" H 3620 2230 50  0000 L CNN "Wattage"
-F 7 "" H 3850 2700 60  0001 C CNN "Digi-Key PN"
+F 7 "311-1.00KHRCT-ND" H 3850 2700 60  0001 C CNN "Digi-Key PN"
 	1    3550 2300
 	-1   0    0    -1
@@
 F 5 "1%" H 9620 2300 50  0000 L CNN "Tolerance"
 F 6 "1/10W" H 9620 2230 50  0000 L CNN "Wattage"
-F 7 "" H 9850 2700 60  0001 C CNN "Digi-Key PN"
+F 7 "311-1.00KHRCT-ND" H 9850 2700 60  0001 C CNN "Digi-Key PN"
 	1    9550 2300
 	-1   0    0    -1
@@
 F 5 "1%" H 5620 2300 50  0000 L CNN "Tolerance"
 F 6 "1/10W" H 5620 2230 50  0000 L CNN "Wattage"
-F 7 "" H 5850 2700 60  0001 C CNN "Digi-Key PN"
+F 7 "311-1.00KHRCT-ND" H 5850 2700 60  0001 C CNN "Digi-Key PN"
 	1    5550 2300
 	-1   0    0    -1
@@
 F 5 "1%" H 7620 2300 50  0000 L CNN "Tolerance"
 F 6 "1/10W" H 7620 2230 50  0000 L CNN "Wattage"
-F 7 "" H 7850 2700 60  0001 C CNN "Digi-Key PN"
+F 7 "311-1.00KHRCT-ND" H 7850 2700 60  0001 C CNN "Digi-Key PN"
 	1    7550 2300
 	-1   0    0    -1
@@
 F 5 "1%" H 3250 5940 50  0000 L CNN "Tolerance"
 F 6 "1/10W" H 3260 5860 50  0000 L CNN "Wattage"
-F 7 "" H 3450 6340 60  0001 C CNN "Digi-Key PN"
+F 7 "YAG2321CT-ND" H 3450 6340 60  0001 C CNN "Digi-Key PN"
 	1    3150 5940
 	1    0    0    -1
@@
 F 5 "1%" V 2310 7060 50  0000 C CNN "Tolerance"
 F 6 "1/10W" V 2410 7060 50  0000 C CNN "Wattage"
-F 7 "" H 2410 7460 60  0001 C CNN "Digi-Key PN"
+F 7 "YAG2321CT-ND" H 2410 7460 60  0001 C CNN "Digi-Key PN"
 	1    2110 7060
 	0    -1   -1   0
@@
 F 5 "1%" H 2740 7290 50  0000 C CNN "Tolerance"
 F 6 "1/10W" H 2770 7220 50  0000 C CNN "Wattage"
-F 7 "" H 2860 7690 60  0001 C CNN "Digi-Key PN"
+F 7 "YAG2321CT-ND" H 2860 7690 60  0001 C CNN "Digi-Key PN"
 	1    2560 7290
 	1    0    0    -1
@@
 F 5 "1%" H 3620 3800 50  0000 L CNN "Tolerance"
 F 6 "1/10W" H 3620 3730 50  0000 L CNN "Wattage"
-F 7 "" H 3850 4200 60  0001 C CNN "Digi-Key PN"
+F 7 "311-1.00KHRCT-ND" H 3850 4200 60  0001 C CNN "Digi-Key PN"
 	1    3550 3800
 	-1   0    0    -1
