File: hdw/Analog_Clock/POS20_Telemetry.sch (KiCad schematic (older format))
At the start: 0 parts

Commit message: More sch work
Parts:
- added C? (x3): 0.1uF, Capacitors_SMD:C_0402, symbol Custom_Library:C_Custom
- added DOC? (x2): FIX ME, symbol Custom_Library:I2C_Address
- added U?: INA219BxDCN, Package_TO_SOT_SMD:SOT-23-8, symbol Analog_ADC:INA219BxDCN
- added U?: MCP9804, Package_DFN_QFN:DFN-8-1EP_3x2mm_P0.5mm_EP1.3x1.5mm, symbol Sensor_Temperature:MCP9804_DFN
Connections:
- new net +3V3: C?.1, C?.1, U?.4 (VS), U?.8 (VDD)
- new net GND: C?.2, C?.2, U?.3 (GND), U?.4 (GND), U?.9 (EP/GND)
- new net I2C_SCL: U?.2 (SCL), U?.5 (SCL)
- new net I2C_SDA: U?.1 (SDA), U?.6 (SDA)
- new net POS20_SNS+: C?.1, U?.1 (IN+)
- new net POS20_SNS-: C?.2, U?.2 (IN-)
- no-connect marks 0 -> 1

Commit message: big sch push
Parts:
- removed C? (x2): 0.1uF, Capacitors_SMD:C_0402, symbol Custom_Library:C_Custom
- removed DOC? (x2): FIX ME, symbol Custom_Library:I2C_Address
- removed U?: INA219BxDCN, Package_TO_SOT_SMD:SOT-23-8, symbol Analog_ADC:INA219BxDCN
- added C702, C703: 0.1uF, Capacitors_SMD:C_0603, symbol Custom_Library:C_Custom
- added DOC701: 0x42, symbol Custom_Library:I2C_Address
- added DOC702: 0x1A, symbol Custom_Library:I2C_Address
- added U701: INA219BxDCN, Package_TO_SOT_SMD:SOT-23-8, symbol Analog_ADC:INA219BxDCN
- C701: renamed from C?; footprint Capacitors_SMD:C_0402 -> Capacitors_SMD:C_0603; Digi-Key PN 490-10701-1-ND -> 399-7845-1-ND; display_footprint (none) -> 0603
- gave numbers to parts that had none: 1
Connections:
- net +3V3: now also U702.6 (A1), C702.1, C703.1, U701.4 (VS)
- net GND: now also U702.5 (A2), U702.7 (A0), C702.2, C703.2, U701.3 (GND), U701.8 (A1)
- net I2C_SCL: now also U701.5 (SCL)
- net I2C_SDA: now also U701.6 (SDA), U701.7 (A0)
- net POS20_SNS+: now also U701.1 (IN+)
- net POS20_SNS-: now also U701.2 (IN-)
Other:
- note added: "RSHUNT = 1.0\nCLSB = 60uA"
