File: hdw/Analog_Clock/Pushbuttons.sch (KiCad schematic (older format))
At the start: 26 parts

Commit message: big sch push
Parts:
- removed C? (x2): 0.1uF, Capacitors_SMD:C_0603, symbol Custom_Library:C_Custom
- removed U? (x2): TLV71333PDBV, Package_TO_SOT_SMD:SOT-23-5, symbol Regulator_Linear:TLV71333PDBV
- C2201, C2202, C2207, C2208: renamed from C?; Digi-Key PN 311-1344-1-ND -> 399-7845-1-ND
- C2203, C2204: renamed from C?; Digi-Key PN 1276-1921-1-ND -> 399-7842-1-ND
- C2205, C2206: renamed from C?; Digi-Key PN 490-14372-1-ND -> 490-10474-1-ND
- R2201, R2202: renamed from R?; Digi-Key PN P499HCT-ND -> (none)
- R2203, R2204, R2205, R2206, R2207, R2208: renamed from R?; Digi-Key PN RMCF0603FT10K0CT-ND -> (none)
- gave numbers to parts that had none: 6
Connections:
- wire segments 56 -> 30

Commit message: Much more schematic progress
Parts:
- R2201, R2202: Digi-Key PN (none) -> RMCF0603FT499RCT-ND
- R2203, R2204, R2205, R2206, R2207, R2208: Digi-Key PN (none) -> YAG2321CT-ND
Changed lines of the file:
@@
 encoding utf-8
 Sheet 22 25
-Title "Incrementor"
-Date "2019-09-03"
+Title "Analog Clock"
+Date "2020-08-15"
 Rev "A"
 Comp "Drew Maatman"
@@
 F 2 "Resistors_SMD:R_0603" H 3200 2260 50  0001 C CNN
 F 3 "" H 3200 2260 50  0001 C CNN
-F 4 "" H 3500 2660 60  0001 C CNN "Digi-Key PN"
+F 4 "RMCF0603FT499RCT-ND" H 3500 2660 60  0001 C CNN "Digi-Key PN"
 F 5 "0603" V 3300 2260 50  0000 C CNN "display_footprint"
 F 6 "1%" V 3400 2260 50  0000 C CNN "Tolerance"
@@
 F 5 "1%" H 5670 2720 50  0000 L CNN "Tolerance"
 F 6 "1/10W" H 5670 2620 50  0000 L CNN "Wattage"
-F 7 "" H 5870 3150 60  0001 C CNN "Digi-Key PN"
+F 7 "YAG2321CT-ND" H 5870 3150 60  0001 C CNN "Digi-Key PN"
 	1    5570 2750
 	1    0    0    -1
@@
 F 5 "1%" V 6390 2460 50  0000 C CNN "Tolerance"
 F 6 "1/10W" V 6490 2460 50  0000 C CNN "Wattage"
-F 7 "" H 6190 2460 50  0001 C CNN "Digi-Key PN"
+F 7 "YAG2321CT-ND" H 6190 2460 50  0001 C CNN "Digi-Key PN"
 	1    6190 2460
 	0    1    -1   0
@@
 F 5 "1%" H 7780 2720 50  0000 L CNN "Tolerance"
 F 6 "1/10W" H 7780 2620 50  0000 L CNN "Wattage"
-F 7 "" H 7980 3150 60  0001 C CNN "Digi-Key PN"
+F 7 "YAG2321CT-ND" H 7980 3150 60  0001 C CNN "Digi-Key PN"
 	1    7680 2750
 	1    0    0    -1
@@
 F 2 "Resistors_SMD:R_0603" H 3200 4790 50  0001 C CNN
 F 3 "" H 3200 4790 50  0001 C CNN
-F 4 "" H 3500 5190 60  0001 C CNN "Digi-Key PN"
+F 4 "RMCF0603FT499RCT-ND" H 3500 5190 60  0001 C CNN "Digi-Key PN"
 F 5 "0603" V 3300 4790 50  0000 C CNN "display_footprint"
 F 6 "1%" V 3400 4790 50  0000 C CNN "Tolerance"
@@
 F 5 "1%" H 5670 5250 50  0000 L CNN "Tolerance"
 F 6 "1/10W" H 5670 5150 50  0000 L CNN "Wattage"
-F 7 "" H 5870 5680 60  0001 C CNN "Digi-Key PN"
+F 7 "YAG2321CT-ND" H 5870 5680 60  0001 C CNN "Digi-Key PN"
 	1    5570 5280
 	1    0    0    -1
@@
 F 5 "1%" V 6390 4990 50  0000 C CNN "Tolerance"
 F 6 "1/10W" V 6490 4990 50  0000 C CNN "Wattage"
-F 7 "" H 6190 4990 50  0001 C CNN "Digi-Key PN"
+F 7 "YAG2321CT-ND" H 6190 4990 50  0001 C CNN "Digi-Key PN"
 	1    6190 4990
 	0    1    -1   0
@@
 F 5 "1%" H 7780 5250 50  0000 L CNN "Tolerance"
 F 6 "1/10W" H 7780 5150 50  0000 L CNN "Wattage"
-F 7 "" H 7980 5680 60  0001 C CNN "Digi-Key PN"
+F 7 "YAG2321CT-ND" H 7980 5680 60  0001 C CNN "Digi-Key PN"
 	1    7680 5280
 	1    0    0    -1
