File: hdw/Analog_Clock/Time_of_Flight.sch (KiCad schematic (older format))
At the start: 6 parts

Commit message: More sch work
Parts:
- added D?: BAT48JFILM, Diode_SMD:D_SOD-323, symbol Diode:BAT48JFILM
Other:
- note removed: "find smaller diode"
Changed lines of the file:
@@
 $Descr A 11000 8500
 encoding utf-8
-Sheet 15 20
+Sheet 15 21
 Title ""
 Date ""
@@
 	5320 2810 5320 2890
 Connection ~ 5320 2890
-Text Notes 2580 2690 0    50   ~ 0
-find smaller diode
+$Comp
+L Diode:BAT48JFILM D?
+U 1 1 5F32DF32
+P 2880 2660
+AR Path="/5E939D31/5F32DF32" Ref="D?"  Part="1"
+AR Path="/5E93A1E8/5F32DF32" Ref="D?"  Part="1"
+F 0 "D?" V 2950 2540 50  0000 R CNN
+F 1 "BAT48JFILM" V 2850 2540 50  0000 R CNN
+F 2 "Diode_SMD:D_SOD-323" H 2880 2485 50  0001 C CNN
+F 3 "www.st.com/resource/en/datasheet/bat48.pdf" H 2880 2660 50  0001 C CNN
+F 4 "497-5711-1-ND" H 2880 2660 50  0001 C CNN "Digi-Key PN"
+	1    2880 2660
+	0    -1   -1   0
+$EndComp
 $EndSCHEMATC

Commit message: big sch push
Parts:
- C1501, C1502, C1503: renamed from C?; footprint Capacitors_SMD:C_0402 -> Capacitors_SMD:C_0603; Digi-Key PN 490-13211-1-ND -> 490-10474-1-ND; Voltage 6.3V -> 10V; display_footprint 0402 -> 0603
- C1504: renamed from C?; footprint Capacitors_SMD:C_0402 -> Capacitors_SMD:C_0603; Digi-Key PN 490-10701-1-ND -> 399-7845-1-ND; display_footprint 0402 -> 0603
- DOC1501: renamed from DOC?; value kjhjfhdsaf -> 0x6B
- gave numbers to parts that had none: 2
Changed lines of the file:
@@
 $Descr A 11000 8500
 encoding utf-8
-Sheet 15 24
+Sheet 15 25
 Title ""
 Date ""
@@
 $EndDescr
 $Comp
-L Custom_Library:DS1683 U?
+L Custom_Library:DS1683 U1501
 U 1 1 5B5039F7
 P 4840 4100
-F 0 "U?" H 4840 3750 60  0000 C CNN
+F 0 "U1501" H 4840 3750 60  0000 C CNN
 F 1 "DS1683" H 4840 4450 60  0000 C CNN
 F 2 "Housings_SOIC:SOIC-8_3.9x4.9mm_Pitch1.27mm" H 4740 4400 60  0001 C CNN
@@
 NoConn ~ 4440 3900
 $Comp
-L power:GND #PWR?
+L power:GND #PWR01505
 U 1 1 5B50444E
 P 4360 4380
-F 0 "#PWR?" H 4360 4130 50  0001 C CNN
+F 0 "#PWR01505" H 4360 4130 50  0001 C CNN
 F 1 "GND" H 4360 4230 50  0000 C CNN
 F 2 "" H 4360 4380 50  0001 C CNN
@@
 	5320 3900 5240 3900
 $Comp
-L Custom_Library:C_Custom C?
+L Custom_Library:C_Custom C1504
 U 1 1 5B507AC7
 P 4830 3120
-F 0 "C?" H 4855 3220 50  0000 L CNN
+F 0 "C1504" H 4855 3220 50  0000 L CNN
 F 1 "0.1uF" H 4855 3020 50  0000 L CNN
-F 2 "Capacitors_SMD:C_0402" H 4868 2970 50  0001 C CNN
+F 2 "Capacitors_SMD:C_0603" H 4868 2970 50  0001 C CNN
 F 3 "" H 4855 3220 50  0001 C CNN
-F 4 "0402" H 4680 3220 50  0000 R CNN "display_footprint"
+F 4 "0603" H 4680 3220 50  0000 R CNN "display_footprint"
 F 5 "50V" H 4680 3120 50  0000 R CNN "Voltage"
 F 6 "X7R" H 4680 3020 50  0000 R CNN "Dielectric"
-F 7 "490-10701-1-ND" H 4830 3120 50  0001 C CNN "Digi-Key PN"
+F 7 "399-7845-1-ND" H 4830 3120 50  0001 C CNN "Digi-Key PN"
 	1    4830 3120
 	1    0    0    -1
 $EndComp
 $Comp
-L power:GND #PWR?
+L power:GND #PWR01507
 U 1 1 5B507BED
 P 4830 3270
-F 0 "#PWR?" H 4830 3020 50  0001 C CNN
+F 0 "#PWR01507" H 4830 3020 50  0001 C CNN
 F 1 "GND" H 4830 3120 50  0000 C CNN
 F 2 "" H 4830 3270 50  0001 C CNN
@@
 $EndComp
 $Comp
-L Custom_Library:I2C_Address DOC?
+L Custom_Library:I2C_Address DOC1501
 U 1 1 5E383387
 P 5040 5100
-F 0 "DOC?" H 5040 5350 60  0001 C CNN
-F 1 "kjhjfhdsaf" H 4590 5100 60  0000 L CNN
+F 0 "DOC1501" H 5040 5350 60  0001 C CNN
+F 1 "0x6B" H 4590 5100 60  0000 L CNN
 F 2 "" H 5040 5450 60  0001 C CNN
 F 3 "" H 5040 5450 60  0001 C CNN
@@
 AR Path="/5E2A7EE3/5E2AFB8F" Ref="C?"  Part="1"
 AR Path="/5E07B870/5E2AFB8F" Ref="C?"  Part="1"
-AR Path="/5E93A1E8/5E2AFB8F" Ref="C?"  Part="1"
-F 0 "C?" H 4205 3220 50  0000 L CNN
+AR Path="/5E93A1E8/5E2AFB8F" Ref="C1503"  Part="1"
+F 0 "C1503" H 4205 3220 50  0000 L CNN
 F 1 "10uF" H 4205 3020 50  0000 L CNN
-F 2 "Capacitors_SMD:C_0402" H 4218 2970 50  0001 C CNN
+F 2 "Capacitors_SMD:C_0603" H 4218 2970 50  0001 C CNN
 F 3 "" H 4205 3220 50  0001 C CNN
-F 4 "490-13211-1-ND" H 4605 3620 60  0001 C CNN "Digi-Key PN"
-F 5 "0402" H 4030 3220 50  0000 R CNN "display_footprint"
-F 6 "6.3V" H 4030 3120 50  0000 R CNN "Voltage"
+F 4 "490-10474-1-ND" H 4605 3620 60  0001 C CNN "Digi-Key PN"
+F 5 "0603" H 4030 3220 50  0000 R CNN "display_footprint"
+F 6 "10V" H 4030 3120 50  0000 R CNN "Voltage"
 F 7 "X5R" H 4030 3020 50  0000 R CNN "Dielectric"
 	1    4180 3120
@@
 AR Path="/5E2A7EE3/5E2AFBB1" Ref="C?"  Part="1"
 AR Path="/5E07B870/5E2AFBB1" Ref="C?"  Part="1"
-AR Path="/5E93A1E8/5E2AFBB1" Ref="C?"  Part="1"
-F 0 "C?" H 3555 3220 50  0000 L CNN
+AR Path="/5E93A1E8/5E2AFBB1" Ref="C1502"  Part="1"
+F 0 "C1502" H 3555 3220 50  0000 L CNN
 F 1 "10uF" H 3555 3020 50  0000 L CNN
-F 2 "Capacitors_SMD:C_0402" H 3568 2970 50  0001 C CNN
+F 2 "Capacitors_SMD:C_0603" H 3568 2970 50  0001 C CNN
 F 3 "" H 3555 3220 50  0001 C CNN
-F 4 "490-13211-1-ND" H 3955 3620 60  0001 C CNN "Digi-Key PN"
-F 5 "0402" H 3380 3220 50  0000 R CNN "display_footprint"
-F 6 "6.3V" H 3380 3120 50  0000 R CNN "Voltage"
+F 4 "490-10474-1-ND" H 3955 3620 60  0001 C CNN "Digi-Key PN"
+F 5 "0603" H 3380 3220 50  0000 R CNN "display_footprint"
+F 6 "10V" H 3380 3120 50  0000 R CNN "Voltage"
 F 7 "X5R" H 3380 3020 50  0000 R CNN "Dielectric"
 	1    3530 3120
@@
 AR Path="/5E2A7EE3/5E2B068F" Ref="C?"  Part="1"
 AR Path="/5E07B870/5E2B068F" Ref="C?"  Part="1"
-AR Path="/5E93A1E8/5E2B068F" Ref="C?"  Part="1"
-F 0 "C?" H 2905 3220 50  0000 L CNN
+AR Path="/5E93A1E8/5E2B068F" Ref="C1501"  Part="1"
+F 0 "C1501" H 2905 3220 50  0000 L CNN
 F 1 "10uF" H 2905 3020 50  0000 L CNN
-F 2 "Capacitors_SMD:C_0402" H 2918 2970 50  0001 C CNN
+F 2 "Capacitors_SMD:C_0603" H 2918 2970 50  0001 C CNN
 F 3 "" H 2905 3220 50  0001 C CNN
-F 4 "490-13211-1-ND" H 3305 3620 60  0001 C CNN "Digi-Key PN"
-F 5 "0402" H 2730 3220 50  0000 R CNN "display_footprint"
-F 6 "6.3V" H 2730 3120 50  0000 R CNN "Voltage"
+F 4 "490-10474-1-ND" H 3305 3620 60  0001 C CNN "Digi-Key PN"
+F 5 "0603" H 2730 3220 50  0000 R CNN "display_footprint"
+F 6 "10V" H 2730 3120 50  0000 R CNN "Voltage"
 F 7 "X5R" H 2730 3020 50  0000 R CNN "Dielectric"
 	1    2880 3120
@@
 $EndComp
 $Comp
-L power:GND #PWR?
+L power:GND #PWR01504
 U 1 1 5E2B2965
 P 4180 3270
-F 0 "#PWR?" H 4180 3020 50  0001 C CNN
+F 0 "#PWR01504" H 4180 3020 50  0001 C CNN
 F 1 "GND" H 4180 3120 50  0000 C CNN
 F 2 "" H 4180 3270 50  0001 C CNN
@@
 $EndComp
 $Comp
-L power:GND #PWR?
+L power:GND #PWR01503
 U 1 1 5E2B2CA6
 P 3530 3270
-F 0 "#PWR?" H 3530 3020 50  0001 C CNN
+F 0 "#PWR01503" H 3530 3020 50  0001 C CNN
 F 1 "GND" H 3530 3120 50  0000 C CNN
 F 2 "" H 3530 3270 50  0001 C CNN
@@
 $EndComp
 $Comp
-L power:GND #PWR?
+L power:GND #PWR01502
 U 1 1 5E2B305D
 P 2880 3270
-F 0 "#PWR?" H 2880 3020 50  0001 C CNN
+F 0 "#PWR01502" H 2880 3020 50  0001 C CNN
 F 1 "GND" H 2880 3120 50  0000 C CNN
 F 2 "" H 2880 3270 50  0001 C CNN
@@
 I2C_SDA
 $Comp
-L power:+3.3V #PWR?
+L power:+3.3V #PWR01506
 U 1 1 5E36CA22
 P 4440 4100
-F 0 "#PWR?" H 4440 3950 50  0001 C CNN
+F 0 "#PWR01506" H 4440 3950 50  0001 C CNN
 F 1 "+3.3V" V 4440 4240 50  0000 L CNN
 F 2 "" H 4440 4100 50  0001 C CNN
@@
 $EndComp
 $Comp
-L power:+3.3V #PWR?
+L power:+3.3V #PWR01501
 U 1 1 5E36D120
 P 2880 2510
-F 0 "#PWR?" H 2880 2360 50  0001 C CNN
+F 0 "#PWR01501" H 2880 2360 50  0001 C CNN
 F 1 "+3.3V" H 2880 2650 50  0000 C CNN
 F 2 "" H 2880 2510 50  0001 C CNN
@@
 $EndComp
 $Comp
-L power:PWR_FLAG #FLG?
+L power:PWR_FLAG #FLG01501
 U 1 1 5E4BADF7
 P 5320 2810
-F 0 "#FLG?" H 5320 2885 50  0001 C CNN
+F 0 "#FLG01501" H 5320 2885 50  0001 C CNN
 F 1 "PWR_FLAG" H 5320 2960 50  0000 C CNN
 F 2 "" H 5320 2810 50  0001 C CNN
@@
 P 2880 2660
 AR Path="/5E939D31/5F32DF32" Ref="D?"  Part="1"
-AR Path="/5E93A1E8/5F32DF32" Ref="D?"  Part="1"
-F 0 "D?" V 2950 2540 50  0000 R CNN
+AR Path="/5E93A1E8/5F32DF32" Ref="D1501"  Part="1"
+F 0 "D1501" V 2950 2540 50  0000 R CNN
 F 1 "BAT48JFILM" V 2850 2540 50  0000 R CNN
 F 2 "Diode_SMD:D_SOD-323" H 2880 2485 50  0001 C CNN
