File: hdw/Analog_Clock/USB_Telemetry.sch (KiCad schematic (older format))
At the start: 7 parts

Commit message: More schematic work
Connections:
- net labels added: +3.3V, GND
Changed lines of the file:
@@
 EESchema Schematic File Version 4
+LIBS:Analog_Clock-cache
 EELAYER 30 0
 EELAYER END
@@
 Text GLabel 3790 1860 0    50   UnSpc ~ 0
 POS5_USB_SNS+
+$Comp
+L power:GND #PWR?
+U 1 1 5E9C5D8F
+P 5110 5120
+F 0 "#PWR?" H 5110 4870 50  0001 C CNN
+F 1 "GND" H 5110 4970 50  0000 C CNN
+F 2 "" H 5110 5120 50  0001 C CNN
+F 3 "" H 5110 5120 50  0001 C CNN
+	1    5110 5120
+	1    0    0    -1
+$EndComp
+$Comp
+L power:GND #PWR?
+U 1 1 5E9C60FF
+P 5110 5840
+F 0 "#PWR?" H 5110 5590 50  0001 C CNN
+F 1 "GND" H 5110 5690 50  0000 C CNN
+F 2 "" H 5110 5840 50  0001 C CNN
+F 3 "" H 5110 5840 50  0001 C CNN
+	1    5110 5840
+	1    0    0    -1
+$EndComp
+$Comp
+L power:GND #PWR?
+U 1 1 5E9C64E1
+P 5110 3220
+F 0 "#PWR?" H 5110 2970 50  0001 C CNN
+F 1 "GND" H 5110 3070 50  0000 C CNN
+F 2 "" H 5110 3220 50  0001 C CNN
+F 3 "" H 5110 3220 50  0001 C CNN
+	1    5110 3220
+	1    0    0    -1
+$EndComp
+$Comp
+L power:GND #PWR?
+U 1 1 5E9C6E65
+P 5110 2500
+F 0 "#PWR?" H 5110 2250 50  0001 C CNN
+F 1 "GND" H 5110 2350 50  0000 C CNN
+F 2 "" H 5110 2500 50  0001 C CNN
+F 3 "" H 5110 2500 50  0001 C CNN
+	1    5110 2500
+	1    0    0    -1
+$EndComp
+$Comp
+L power:+3.3V #PWR?
+U 1 1 5E9C850A
+P 5110 1700
+F 0 "#PWR?" H 5110 1550 50  0001 C CNN
+F 1 "+3.3V" H 5110 1840 50  0000 C CNN
+F 2 "" H 5110 1700 50  0001 C CNN
+F 3 "" H 5110 1700 50  0001 C CNN
+	1    5110 1700
+	1    0    0    -1
+$EndComp
+$Comp
+L power:+3.3V #PWR?
+U 1 1 5E9C8B3B
+P 5110 2920
+F 0 "#PWR?" H 5110 2770 50  0001 C CNN
+F 1 "+3.3V" H 5110 3060 50  0000 C CNN
+F 2 "" H 5110 2920 50  0001 C CNN
+F 3 "" H 5110 2920 50  0001 C CNN
+	1    5110 2920
+	1    0    0    -1
+$EndComp
+$Comp
+L power:+3.3V #PWR?
+U 1 1 5E9C962A
+P 5110 4040
+F 0 "#PWR?" H 5110 3890 50  0001 C CNN
+F 1 "+3.3V" H 5110 4180 50  0000 C CNN
+F 2 "" H 5110 4040 50  0001 C CNN
+F 3 "" H 5110 4040 50  0001 C CNN
+	1    5110 4040
+	1    0    0    -1
+$EndComp
 $EndSCHEMATC

Commit message: More sch work
Parts:
- removed C? (x3): 0.1uF, Capacitors_SMD:C_0402, symbol Custom_Library:C_Custom
- removed DOC?: ljasdflkjafds, symbol Custom_Library:I2C_Address
- removed DOC?: aljhdslkfjasdf, symbol Custom_Library:I2C_Address
- removed U?: INA219BxDCN, Package_TO_SOT_SMD:SOT-23-8, symbol Analog_ADC:INA219BxDCN
- removed U?: MCP9804, Package_DFN_QFN:DFN-8-1EP_3x2mm_P0.5mm_EP1.3x1.5mm, symbol Sensor_Temperature:MCP9804_DFN
- added C? (x3): 0.1uF, Capacitors_SMD:C_0402, symbol Custom_Library:C_Custom
- added DOC? (x2): FIX ME, symbol Custom_Library:I2C_Address
- added U?: INA219BxDCN, Package_TO_SOT_SMD:SOT-23-8, symbol Analog_ADC:INA219BxDCN
- added U?: MCP9804, Package_DFN_QFN:DFN-8-1EP_3x2mm_P0.5mm_EP1.3x1.5mm, symbol Sensor_Temperature:MCP9804_DFN
Connections:
- net +3V3: now also C?.1, C?.1, U?.4 (VS), U?.8 (VDD)
- net GND: now also C?.2, C?.2, U?.3 (GND), U?.4 (GND), U?.9 (EP/GND)
- net I2C_SCL: now also U?.2 (SCL), U?.5 (SCL)
- net I2C_SDA: now also U?.1 (SDA), U?.6 (SDA)
- net POS5_USB_SNS+: now also C?.1, U?.1 (IN+)
- net POS5_USB_SNS-: now also C?.2, U?.2 (IN-)

Commit message: big sch push
Parts:
- removed C? (x3): 0.1uF, Capacitors_SMD:C_0402, symbol Custom_Library:C_Custom
- removed DOC?: FIX ME, symbol Custom_Library:I2C_Address
- removed U?: MCP9804, Package_DFN_QFN:DFN-8-1EP_3x2mm_P0.5mm_EP1.3x1.5mm, symbol Sensor_Temperature:MCP9804_DFN
- added C1401, C1402, C1403: 0.1uF, Capacitors_SMD:C_0603, symbol Custom_Library:C_Custom
- added DOC1402: 0x1B, symbol Custom_Library:I2C_Address
- added U1402: MCP9804, Package_DFN_QFN:DFN-8-1EP_3x2mm_P0.5mm_EP1.3x1.5mm, symbol Sensor_Temperature:MCP9804_DFN
- DOC1401: renamed from DOC?; value FIX ME -> 0x43
- gave numbers to parts that had none: 1
Connections:
- net +3V3: now also C1402.1, C1403.1, U1402.6 (A1), U1402.7 (A0), U1402.8 (VDD)
- net GND: now also U1401.8 (A1), C1402.2, C1403.2, U1402.4 (GND), U1402.5 (A2), U1402.9 (EP/GND)
- net I2C_SCL: now also U1401.7 (A0), U1402.2 (SCL)
- net I2C_SDA: now also U1402.1 (SDA)
- net POS5_USB_SNS+: now also C1401.1
- net POS5_USB_SNS-: now also C1401.2
Other:
- note added: "RSHUNT = 0.02\nCLSB = 60uA"

Commit message: More PCB arrangement
Parts:
- removed C1401, C1402, C1403: 0.1uF, Capacitors_SMD:C_0603, symbol Custom_Library:C_Custom
- removed DOC1401: 0x43, symbol Custom_Library:I2C_Address
- removed DOC1402: 0x1B, symbol Custom_Library:I2C_Address
- removed U1401: INA219BxDCN, Package_TO_SOT_SMD:SOT-23-8, symbol Analog_ADC:INA219BxDCN
- removed U1402: MCP9804, Package_DFN_QFN:DFN-8-1EP_3x2mm_P0.5mm_EP1.3x1.5mm, symbol Sensor_Temperature:MCP9804_DFN
Connections:
- no-connect marks 1 -> 0
Other:
- note removed: "RSHUNT = 0.02\nCLSB = 60uA"

Commit message: Major USB restructuring
Parts:
- added C1401, C1402, C1403: 0.1uF, Capacitors_SMD:C_0603, symbol Custom_Library:C_Custom
- added DOC1401: 0x43, symbol Custom_Library:I2C_Address
- added DOC1402: 0x1B, symbol Custom_Library:I2C_Address
- added U1401: INA219BxDCN, Package_TO_SOT_SMD:SOT-23-8, symbol Analog_ADC:INA219BxDCN
- added U1402: MCP9804, Package_DFN_QFN:DFN-8-1EP_3x2mm_P0.5mm_EP1.3x1.5mm, symbol Sensor_Temperature:MCP9804_DFN
Connections:
- new net +3V3: C1402.1, C1403.1, U1401.4 (VS), U1402.6 (A1), U1402.7 (A0), U1402.8 (VDD)
- new net GND: C1402.2, C1403.2, U1401.3 (GND), U1401.8 (A1), U1402.4 (GND), U1402.5 (A2), U1402.9 (EP/GND)
- new net I2C_SCL: U1401.5 (SCL), U1401.7 (A0), U1402.2 (SCL)
- new net I2C_SDA: U1401.6 (SDA), U1402.1 (SDA)
- new net POS5_USB_SNS+: C1401.1, U1401.1 (IN+)
- new net POS5_USB_SNS-: C1401.2, U1401.2 (IN-)
- no-connect marks 0 -> 1
Other:
- note added: "RSHUNT = 0.02\nCLSB = 60uA"
