File: hdw/Analog_Clock/POS20_Power_Supply.sch (KiCad schematic (older format))
At the start: 0 parts

Commit message: Added +20V power supply, updated input power sheet
Parts:
- added C?: 4.7uF, Capacitors_SMD:C_0805, symbol Custom_Library:C_Custom
- added C?: 0.1uF, Capacitors_SMD:C_0805, symbol Custom_Library:C_Custom
- added C? (x3): 0.1uF, Capacitors_SMD:C_0603, symbol Custom_Library:C_Custom
- added C?: 1nF, Capacitors_SMD:C_0603, symbol Custom_Library:C_Custom
- added C?: 10nF, Capacitors_SMD:C_0603, symbol Custom_Library:C_Custom
- added C? (x2): 10uF, Capacitors_SMD:C_1206, symbol Custom_Library:C_Custom
- added C?: 6.8nF, Capacitors_SMD:C_0603, symbol Custom_Library:C_Custom
- added C?: C_Custom, symbol Custom_Library:C_Custom
- added D?: MBR0580, Diode_SMD:D_SOD-123, symbol Diode:MBR0580
- added L?: L_Custom, symbol Custom_Library:L_Custom
- added R? (x2): 10k, Resistors_SMD:R_0603, symbol Custom_Library:R_Custom
- added R?: 1, Resistors_SMD:R_0612, symbol Custom_Library:R_Custom
- added R? (x6): R, Resistors_SMD:R_0603, symbol Custom_Library:R_Custom
- added R?: R, Resistors_SMD:R_0805, symbol Custom_Library:R_Custom
- added R?: 22k, Resistors_SMD:R_0603, symbol Custom_Library:R_Custom
- added R? (x2): 100, Resistors_SMD:R_0603, symbol Custom_Library:R_Custom
- added TP?: TP, Custom Footprints Library:Test_Point, symbol Custom_Library:TP
- added U?: LT3757, Housings_DFN_QFN:DFN-10-1EP_3x3mm_Pitch0.5mm, symbol Custom_Library:LT3757
- added U?: TLV6700, Package_TO_SOT_SMD:SOT-23-6, symbol Custom_Library:TLV6700
Connections:
- net labels added: +12V, +3.3V, +60VAN, GND, POS20_PGOOD, POS20_RUN, POS20_SNS+, POS20_SNS-
- wire segments 0 -> 71
Other:
- note added: "fsw = 650 kHz"

Commit message: some +20V boost supply work
Parts:
- removed C?: 4.7uF, Capacitors_SMD:C_0805, symbol Custom_Library:C_Custom
- added C?: 10uF, symbol Custom_Library:C_Custom
- added Q?: FDC5612, TO_SOT_Packages_SMD:SOT-23-6, symbol Custom_Library:FDC5612
- added R?: 10, Resistors_SMD:R_0402, symbol Custom_Library:R_Custom
- C?: value C_Custom -> 10uF; Dielectric Er -> X5R; Digi-Key PN PN -> 490-18664-1-ND; Voltage V -> 50V; display_footprint Foot -> 0805
- L?: value L_Custom -> 10uH; Ampacity A -> 3A; Digi-Key PN (none) -> 541-1013-1-ND; Tolerance Tol -> 20%; display_footprint Foot -> IHLP2525
- R? (x2): value R -> 11.5k
- R?: value R -> 1k
- R?: value R -> 140m
Connections:
- net labels added: +20V
- net labels removed: +60VAN
- wire segments 71 -> 72
Other:
- note added: "fsw = 950 kHz"
- note removed: "fsw = 650 kHz"
Changed lines of the file:
@@
 	5440 2540 5440 3190
-Wire Wire Line
-	4760 2340 4800 2340
 Wire Wire Line
 	3710 4130 3710 4090
@@
 	4210 4330 4210 4090
 Text Notes 1540 3210 0    60   ~ 0
-fsw = 650 kHz
+fsw = 950 kHz
 $Comp
 L power:GND #PWR?
@@
 $EndComp
 $Comp
-L Custom_Library:C_Custom C?
-U 1 1 5A174CC6
-P 4210 4480
-F 0 "C?" H 4235 4580 50  0000 L CNN
-F 1 "4.7uF" H 4235 4380 50  0000 L CNN
-F 2 "Capacitors_SMD:C_0805" H 4248 4330 50  0001 C CNN
-F 3 "" H 4235 4580 50  0001 C CNN
-F 4 "0805" H 4060 4580 50  0000 R CNN "display_footprint"
-F 5 "16V" H 4060 4480 50  0000 R CNN "Voltage"
-F 6 "X7R" H 4060 4380 50  0000 R CNN "Dielectric"
-F 7 "1276-2970-1-ND" H -1690 -80 50  0001 C CNN "Digi-Key PN"
-	1    4210 4480
-	1    0    0    -1
-$EndComp
-$Comp
 L power:GND #PWR?
 U 1 1 5A0BD1B1
@@
 F 3 "" H 3960 4090 50  0001 C CNN
 	1    3960 4090
-	1    0    0    -1
-$EndComp
-$Comp
-L Custom_Library:LT3757 U?
-U 1 1 5A0BD080
-P 3960 2890
-F 0 "U?" H 4460 1840 50  0000 C CNN
-F 1 "LT3757" H 3960 2890 50  0000 C CNN
-F 2 "Housings_DFN_QFN:DFN-10-1EP_3x3mm_Pitch0.5mm" H 3960 3590 60  0001 C CNN
-F 3 "" H 3960 3590 60  0001 C CNN
-F 4 "LT3757EDD#PBF-ND" H -1690 -80 50  0001 C CNN "Digi-Key PN"
-	1    3960 2890
 	1    0    0    -1
 $EndComp
@@
 P 2460 3570
 F 0 "R?" H 2530 3700 50  0000 L CNN
-F 1 "R" V 2460 3570 40  0000 C CNN
+F 1 "11.5k" V 2460 3570 40  0000 C CNN
 F 2 "Resistors_SMD:R_0603" H 2460 3570 50  0001 C CNN
 F 3 "" H 2460 3570 50  0001 C CNN
@@
 P 9310 4110
 F 0 "R?" H 9380 4240 50  0000 L CNN
-F 1 "R" V 9310 4110 50  0000 C CNN
+F 1 "1k" V 9310 4110 50  0000 C CNN
 F 2 "Resistors_SMD:R_0603" H 9310 4110 50  0001 C CNN
 F 3 "" H 9310 4110 50  0001 C CNN
@@
 P 5440 3380
 F 0 "R?" H 5510 3510 50  0000 L CNN
-F 1 "R" V 5440 3380 40  0000 C CNN
+F 1 "140m" V 5440 3380 40  0000 C CNN
 F 2 "Resistors_SMD:R_0805" H 5440 3380 50  0001 C CNN
 F 3 "" H 5440 3380 50  0001 C CNN
@@
 Wire Wire Line
 	4760 3790 9310 3790
-$Comp
-L Custom_Library:+60VAN #PWR?
-U 1 1 5E121BE1
-P 2050 5950
-F 0 "#PWR?" H 2050 5800 50  0001 C CNN
-F 1 "+60VAN" H 2050 6090 50  0000 C CNN
-F 2 "" H 2050 5950 50  0000 C CNN
-F 3 "" H 2050 5950 50  0000 C CNN
-	1    2050 5950
-	1    0    0    -1
-$EndComp
 Wire Wire Line
 	5440 1500 5440 2140
@@
 P 9310 2760
 F 0 "R?" H 9380 2890 50  0000 L CNN
-F 1 "R" V 9310 2760 40  0000 C CNN
+F 1 "11.5k" V 9310 2760 40  0000 C CNN
 F 2 "Resistors_SMD:R_0603" H 9310 2760 50  0001 C CNN
 F 3 "" H 9310 2760 50  0001 C CNN
@@
 P 4670 1500
 F 0 "L?" V 4620 1500 50  0000 C CNN
-F 1 "L_Custom" V 4745 1500 50  0000 C CNN
+F 1 "10uH" V 4745 1500 50  0000 C CNN
 F 2 "" H 4670 1500 50  0001 C CNN
 F 3 "" H 4670 1500 50  0001 C CNN
-F 4 "Foot" V 4820 1500 50  0000 C CNN "display_footprint"
-F 5 "A" V 4920 1500 50  0000 C CNN "Ampacity"
-F 6 "Tol" V 5020 1500 50  0000 C CNN "Tolerance"
+F 4 "IHLP2525" V 4820 1500 50  0000 C CNN "display_footprint"
+F 5 "3A" V 4920 1500 50  0000 C CNN "Ampacity"
+F 6 "20%" V 5020 1500 50  0000 C CNN "Tolerance"
+F 7 "541-1013-1-ND" H 4670 1500 50  0001 C CNN "Digi-Key PN"
 	1    4670 1500
 	0    -1   -1   0
@@
 Wire Wire Line
 	6960 1500 7750 1500
-$Comp
-L Custom_Library:C_Custom C?
-U 1 1 5F2E7454
-P 6960 1810
-F 0 "C?" H 6985 1910 50  0000 L CNN
-F 1 "C_Custom" H 6985 1710 50  0000 L CNN
-F 2 "" H 6998 1660 50  0001 C CNN
-F 3 "" H 6985 1910 50  0001 C CNN
-F 4 "Foot" H 6810 1910 50  0000 R CNN "display_footprint"
-F 5 "V" H 6810 1810 50  0000 R CNN "Voltage"
-F 6 "Er" H 6810 1710 50  0000 R CNN "Dielectric"
-F 7 "PN" H 7385 2310 60  0001 C CNN "Digi-Key PN"
-	1    6960 1810
-	1    0    0    -1
-$EndComp
 $Comp
 L Custom_Library:R_Custom R?
@@
 	-1   0    0    -1
 $EndComp
+$Comp
+L Custom_Library:LT3757 U?
+U 1 1 5A0BD080
+P 3960 2890
+F 0 "U?" H 4460 1840 50  0000 C CNN
+F 1 "LT3757" H 3960 2890 50  0000 C CNN
+F 2 "Housings_DFN_QFN:DFN-10-1EP_3x3mm_Pitch0.5mm" H 3960 3590 60  0001 C CNN
+F 3 "" H 3960 3590 60  0001 C CNN
+F 4 "LT3757EDD#PBF-ND" H -1690 -80 50  0001 C CNN "Digi-Key PN"
+	1    3960 2890
+	1    0    0    -1
+$EndComp
+$Comp
+L Custom_Library:C_Custom C?
+U 1 1 5F2E7454
+P 6960 1810
+F 0 "C?" H 6985 1910 50  0000 L CNN
+F 1 "10uF" H 6985 1710 50  0000 L CNN
+F 2 "" H 6998 1660 50  0001 C CNN
+F 3 "" H 6985 1910 50  0001 C CNN
+F 4 "0805" H 6810 1910 50  0000 R CNN "display_footprint"
+F 5 "50V" H 6810 1810 50  0000 R CNN "Voltage"
+F 6 "X5R" H 6810 1710 50  0000 R CNN "Dielectric"
+F 7 "490-18664-1-ND" H 7385 2310 60  0001 C CNN "Digi-Key PN"
+	1    6960 1810
+	1    0    0    -1
+$EndComp
+$Comp
+L Custom_Library:FDC5612 Q?
+U 1 1 5F30CB26
+P 5340 2340
+F 0 "Q?" H 5540 2390 50  0000 L CNN
+F 1 "FDC5612" H 5540 2290 50  0000 L CNN
+F 2 "TO_SOT_Packages_SMD:SOT-23-6" H 5540 2440 50  0001 C CNN
+F 3 "https://www.onsemi.com/pub/Collateral/FDC5612-D.PDF" H 5340 2340 50  0001 C CNN
+F 4 "FDC5612CT-ND" H 5340 2340 50  0001 C CNN "Digi-Key PN"
+	1    5340 2340
+	1    0    0    -1
+$EndComp
+$Comp
+L Custom_Library:R_Custom R?
+U 1 1 5F3155DF
+P 4950 2340
+AR Path="/5EAE2D66/5F3155DF" Ref="R?"  Part="1"
+AR Path="/5EAE2D8A/5F3155DF" Ref="R?"  Part="1"
+AR Path="/5E939D31/5F3155DF" Ref="R?"  Part="1"
+F 0 "R?" V 4850 2340 50  0000 C CNN
+F 1 "10" V 4950 2340 50  0000 C CNN
+F 2 "Resistors_SMD:R_0402" H 4950 2340 50  0001 C CNN
+F 3 "" H 4950 2340 50  0001 C CNN
+F 4 "541-3964-1-ND" H 5250 2740 60  0001 C CNN "Digi-Key PN"
+F 5 "0402" V 5050 2340 50  0000 C CNN "display_footprint"
+F 6 "1%" V 5150 2340 50  0000 C CNN "Tolerance"
+F 7 "1/16W" V 5250 2340 50  0000 C CNN "Wattage"
+	1    4950 2340
+	0    1    1    0
+$EndComp
+Wire Wire Line
+	5140 2340 5100 2340
+Wire Wire Line
+	4800 2340 4760 2340
+$Comp
+L Custom_Library:+20V #PWR?
+U 1 1 5F31C1D1
+P 8750 1420
+F 0 "#PWR?" H 8750 1270 50  0001 C CNN
+F 1 "+20V" H 8750 1560 50  0000 C CNN
+F 2 "" H 8750 1420 50  0001 C CNN
+F 3 "" H 8750 1420 50  0001 C CNN
+	1    8750 1420
+	1    0    0    -1
+$EndComp
+$Comp
+L Custom_Library:+20V #PWR?
+U 1 1 5F31C768
+P 2050 5950
+F 0 "#PWR?" H 2050 5800 50  0001 C CNN
+F 1 "+20V" H 2050 6090 50  0000 C CNN
+F 2 "" H 2050 5950 50  0001 C CNN
+F 3 "" H 2050 5950 50  0001 C CNN
+	1    2050 5950
+	1    0    0    -1
+$EndComp
+$Comp
+L Custom_Library:C_Custom C?
+U 1 1 5F31FA8E
+P 4210 4480
+F 0 "C?" H 4235 4580 50  0000 L CNN
+F 1 "10uF" H 4235 4380 50  0000 L CNN
+F 2 "" H 4248 4330 50  0001 C CNN
+F 3 "" H 4235 4580 50  0001 C CNN
+F 4 "0805" H 4060 4580 50  0000 R CNN "display_footprint"
+F 5 "50V" H 4060 4480 50  0000 R CNN "Voltage"
+F 6 "X5R" H 4060 4380 50  0000 R CNN "Dielectric"
+F 7 "490-18664-1-ND" H 4635 4980 60  0001 C CNN "Digi-Key PN"
+	1    4210 4480
+	1    0    0    -1
+$EndComp
 $EndSCHEMATC

Commit message: more analog work, added some more sch stuff
Parts:
- R?: value R -> 1.87k
- R?: value R -> 383
- R?: value R -> 100k
Changed lines of the file:
@@
 $Descr A 11000 8500
 encoding utf-8
-Sheet 6 23
+Sheet 6 24
 Title "VFD Clock"
 Date "2019-04-11"
@@
 P 2050 7100
 F 0 "R?" H 2120 7230 50  0000 L CNN
-F 1 "R" V 2050 7100 40  0000 C CNN
+F 1 "1.87k" V 2050 7100 40  0000 C CNN
 F 2 "Resistors_SMD:R_0603" H 2050 7100 50  0001 C CNN
 F 3 "" H 2050 7100 50  0001 C CNN
@@
 P 2050 6600
 F 0 "R?" H 2120 6730 50  0000 L CNN
-F 1 "R" V 2050 6600 40  0000 C CNN
+F 1 "383" V 2050 6600 40  0000 C CNN
 F 2 "Resistors_SMD:R_0603" H 2050 6600 50  0001 C CNN
 F 3 "" H 2050 6600 50  0001 C CNN
@@
 P 2050 6100
 F 0 "R?" H 2120 6230 50  0000 L CNN
-F 1 "R" V 2050 6100 40  0000 C CNN
+F 1 "100k" V 2050 6100 40  0000 C CNN
 F 2 "Resistors_SMD:R_0603" H 2050 6100 50  0001 C CNN
 F 3 "" H 2050 6100 50  0001 C CNN
@@
 AR Path="/5EAE2D8A/5F3155DF" Ref="R?"  Part="1"
 AR Path="/5E939D31/5F3155DF" Ref="R?"  Part="1"
+AR Path="/5E939D51/5F3155DF" Ref="R?"  Part="1"
 F 0 "R?" V 4850 2340 50  0000 C CNN
 F 1 "10" V 4950 2340 50  0000 C CNN

Commit message: big sch push
Parts:
- removed C?: 0.1uF, Capacitors_SMD:C_0805, symbol Custom_Library:C_Custom
- C601, C602: renamed from C?; footprint Capacitors_SMD:C_1206 -> Capacitors_SMD:C_0805; Dielectric X7R -> X5R; Digi-Key PN 1276-1804-6-ND -> 490-18664-1-ND; Voltage 25V -> 50V; display_footprint 1206 -> 0805
- C603, C604, C606: renamed from C?; Digi-Key PN 399-6856-1-ND -> 399-7845-1-ND
- C605: renamed from C?; Digi-Key PN 311-1084-1-ND -> 399-1089-1-ND
- C607, C610: renamed from C?; footprint (none) -> Capacitors_SMD:C_0805
- C608: renamed from C?; Digi-Key PN 399-1092-1-ND -> 399-7842-1-ND
- L601: renamed from L?; footprint (none) -> Inductors_SMD:L_Vishay_IHLP-2525
- R605, R607: renamed from R?; Digi-Key PN P10.0KHCT-ND -> (none)
- R606: renamed from R?; Digi-Key PN A129704CT-ND -> (none)
- R608: renamed from R?; footprint Resistors_SMD:R_0402 -> Resistors_SMD:R_0603; Digi-Key PN 541-3964-1-ND -> (none); Wattage 1/16W -> 1/10W; display_footprint 0402 -> 0603
- R610, R612: renamed from R?; Digi-Key PN A106047CT-ND -> (none)
- gave numbers to parts that had none: 14

Commit message: Much more schematic progress
Parts:
- R601: Digi-Key PN (none) -> RMCF0603FT100KCT-ND
- R602: Digi-Key PN (none) -> 311-383HRCT-ND
- R603: Digi-Key PN (none) -> 311-1.87KHRCT-ND
- R604, R613: Digi-Key PN (none) -> 311-11.5KHRCT-ND
- R605, R607, R608: Digi-Key PN (none) -> YAG2321CT-ND
- R606: Digi-Key PN (none) -> 311-22KLDCT-ND
- R609: value 140m -> 130m; Digi-Key PN (none) -> RL12S.13FCT-ND
- R610, R612: Digi-Key PN (none) -> RMCF0603FT100RCT-ND
- R614: Digi-Key PN (none) -> 311-1.00KHRCT-ND
Changed lines of the file:
@@
 encoding utf-8
 Sheet 6 25
-Title "VFD Clock"
-Date "2019-04-11"
+Title "Analog Clock"
+Date "2020-08-15"
 Rev "A"
 Comp "Drew Maatman"
@@
 F 5 "1%" H 4160 6060 50  0000 L CNN "Tolerance"
 F 6 "1/10W" H 4160 5990 50  0000 L CNN "Wattage"
-F 7 "" H 0   470 50  0001 C CNN "Digi-Key PN"
+F 7 "YAG2321CT-ND" H 0   470 50  0001 C CNN "Digi-Key PN"
 	1    4090 6060
 	-1   0    0    1
@@
 F 5 "1%" H 2530 3530 50  0000 L CNN "Tolerance"
 F 6 "1/10W" H 2530 3440 50  0000 L CNN "Wattage"
+F 7 "311-11.5KHRCT-ND" H 2460 3570 50  0001 C CNN "Digi-Key PN"
 	1    2460 3570
 	-1   0    0    -1
@@
 F 5 "1%" H 9380 4070 50  0000 L CNN "Tolerance"
 F 6 "1/10W" H 9380 3980 50  0000 L CNN "Wattage"
+F 7 "311-1.00KHRCT-ND" H 9310 4110 50  0001 C CNN "Digi-Key PN"
 	1    9310 4110
 	1    0    0    -1
@@
 F 5 "1%" H 3780 4240 50  0000 L CNN "Tolerance"
 F 6 "1/10W" H 3780 4150 50  0000 L CNN "Wattage"
-F 7 "" H 4010 4680 60  0001 C CNN "Digi-Key PN"
+F 7 "311-22KLDCT-ND" H 4010 4680 60  0001 C CNN "Digi-Key PN"
 	1    3710 4280
 	-1   0    0    -1
@@
 P 5440 3380
 F 0 "R609" H 5510 3510 50  0000 L CNN
-F 1 "140m" V 5440 3380 40  0000 C CNN
+F 1 "130m" V 5440 3380 40  0000 C CNN
 F 2 "Resistors_SMD:R_0805" H 5440 3380 50  0001 C CNN
 F 3 "" H 5440 3380 50  0001 C CNN
@@
 F 5 "1%" H 5510 3340 50  0000 L CNN "Tolerance"
 F 6 "1/4W" H 5510 3250 50  0000 L CNN "Wattage"
+F 7 "RL12S.13FCT-ND" H 5440 3380 50  0001 C CNN "Digi-Key PN"
 	1    5440 3380
 	1    0    0    -1
@@
 F 5 "1%" H 2990 2530 50  0000 L CNN "Tolerance"
 F 6 "1/10W" H 2980 2600 50  0000 L CNN "Wattage"
-F 7 "" H -1690 -80 50  0001 C CNN "Digi-Key PN"
+F 7 "YAG2321CT-ND" H -1690 -80 50  0001 C CNN "Digi-Key PN"
 	1    2920 2550
 	-1   0    0    -1
@@
 F 5 "1%" V 7950 1810 50  0001 C CNN "Tolerance"
 F 6 "1/10W" V 8050 1810 50  0001 C CNN "Wattage"
-F 7 "" H 8050 2210 60  0001 C CNN "Digi-Key PN"
+F 7 "RMCF0603FT100RCT-ND" H 8050 2210 60  0001 C CNN "Digi-Key PN"
 	1    7750 1810
 	-1   0    0    1
@@
 F 5 "1%" V 8410 1810 50  0001 C CNN "Tolerance"
 F 6 "1/10W" V 8510 1810 50  0001 C CNN "Wattage"
-F 7 "" H 8510 2210 60  0001 C CNN "Digi-Key PN"
+F 7 "RMCF0603FT100RCT-ND" H 8510 2210 60  0001 C CNN "Digi-Key PN"
 	1    8210 1810
 	-1   0    0    1
@@
 F 5 "1%" H 9380 2720 50  0000 L CNN "Tolerance"
 F 6 "1/10W" H 9380 2630 50  0000 L CNN "Wattage"
+F 7 "311-11.5KHRCT-ND" H 9310 2760 50  0001 C CNN "Digi-Key PN"
 	1    9310 2760
 	1    0    0    -1
@@
 F 5 "1%" H 2120 7060 50  0000 L CNN "Tolerance"
 F 6 "1/10W" H 2120 6970 50  0000 L CNN "Wattage"
+F 7 "311-1.87KHRCT-ND" H 2050 7100 50  0001 C CNN "Digi-Key PN"
 	1    2050 7100
 	-1   0    0    -1
@@
 F 5 "1%" H 2120 6560 50  0000 L CNN "Tolerance"
 F 6 "1/10W" H 2120 6470 50  0000 L CNN "Wattage"
+F 7 "311-383HRCT-ND" H 2050 6600 50  0001 C CNN "Digi-Key PN"
 	1    2050 6600
 	-1   0    0    -1
@@
 F 5 "1%" H 2120 6060 50  0000 L CNN "Tolerance"
 F 6 "1/10W" H 2120 5970 50  0000 L CNN "Wattage"
+F 7 "RMCF0603FT100KCT-ND" H 2050 6100 50  0001 C CNN "Digi-Key PN"
 	1    2050 6100
 	-1   0    0    -1
@@
 F 2 "Resistors_SMD:R_0603" H 4950 2340 50  0001 C CNN
 F 3 "" H 4950 2340 50  0001 C CNN
-F 4 "" H 5250 2740 60  0001 C CNN "Digi-Key PN"
+F 4 "YAG2321CT-ND" H 5250 2740 60  0001 C CNN "Digi-Key PN"
 F 5 "0603" V 5050 2340 50  0000 C CNN "display_footprint"
 F 6 "1%" V 5150 2340 50  0000 C CNN "Tolerance"

Commit message: More PCB arrangement
Parts:
- removed C608: 10nF, Capacitors_SMD:C_0603, symbol Custom_Library:C_Custom
- removed C609: 1nF, Capacitors_SMD:C_0603, symbol Custom_Library:C_Custom
Changed lines of the file:
@@
 $Descr A 11000 8500
 encoding utf-8
-Sheet 6 25
+Sheet 6 24
 Title "Analog Clock"
 Date "2020-08-15"
@@
 Comment4 ""
 $EndDescr
-$Comp
-L power:GND #PWR0618
-U 1 1 5A4AC392
-P 4230 7580
-F 0 "#PWR0618" H 4230 7330 50  0001 C CNN
-F 1 "GND" H 4230 7430 50  0000 C CNN
-F 2 "" H 4230 7580 50  0000 C CNN
-F 3 "" H 4230 7580 50  0000 C CNN
-	1    4230 7580
-	1    0    0    -1
-$EndComp
 $Comp
 L Custom_Library:C_Custom C606
@@
 F 7 "399-7845-1-ND" H 0   470 50  0001 C CNN "Digi-Key PN"
 	1    3910 7350
-	1    0    0    -1
-$EndComp
-$Comp
-L Custom_Library:C_Custom C609
-U 1 1 5A4AC3AF
-P 4550 7350
-F 0 "C609" H 4575 7450 50  0000 L CNN
-F 1 "1nF" H 4575 7250 50  0000 L CNN
-F 2 "Capacitors_SMD:C_0603" H 4588 7200 50  0001 C CNN
-F 3 "" H 4575 7450 50  0001 C CNN
-F 4 "0603" H 4400 7450 50  0001 R CNN "display_footprint"
-F 5 "50V" H 4400 7350 50  0001 R CNN "Voltage"
-F 6 "X7R" H 4400 7250 50  0001 R CNN "Dielectric"
-F 7 "399-1083-1-ND" H 0   470 50  0001 C CNN "Digi-Key PN"
-	1    4550 7350
-	1    0    0    -1
-$EndComp
-$Comp
-L Custom_Library:C_Custom C608
-U 1 1 5A4AC3B9
-P 4230 7350
-F 0 "C608" H 4255 7450 50  0000 L CNN
-F 1 "10nF" H 4255 7250 50  0000 L CNN
-F 2 "Capacitors_SMD:C_0603" H 4268 7200 50  0001 C CNN
-F 3 "" H 4255 7450 50  0001 C CNN
-F 4 "0603" H 4080 7450 50  0001 R CNN "display_footprint"
-F 5 "50V" H 4080 7350 50  0001 R CNN "Voltage"
-F 6 "X7R" H 4080 7250 50  0001 R CNN "Dielectric"
-F 7 "399-7842-1-ND" H 0   470 50  0001 C CNN "Digi-Key PN"
-	1    4230 7350
-	1    0    0    -1
-$EndComp
-$Comp
-L power:+3.3V #PWR0617
-U 1 1 5A4AC3C0
-P 4230 7120
-F 0 "#PWR0617" H 4230 6970 50  0001 C CNN
-F 1 "+3.3V" H 4230 7260 50  0000 C CNN
-F 2 "" H 4230 7120 50  0000 C CNN
-F 3 "" H 4230 7120 50  0000 C CNN
-	1    4230 7120
 	1    0    0    -1
 $EndComp
@@
 	8750 1420 8750 1500
 Wire Wire Line
-	3910 7160 3910 7200
-Connection ~ 4230 7160
-Wire Wire Line
-	4550 7160 4550 7200
-Wire Wire Line
-	3910 7160 4230 7160
-Wire Wire Line
-	4230 7120 4230 7160
-Wire Wire Line
-	3910 7540 3910 7500
-Connection ~ 4230 7540
-Wire Wire Line
-	4550 7540 4550 7500
-Wire Wire Line
-	3910 7540 4230 7540
-Wire Wire Line
-	4230 7500 4230 7540
-Wire Wire Line
 	3490 6350 3490 6850
 Wire Wire Line
@@
 	1    0    0    -1
 $EndComp
-Wire Wire Line
-	4230 7160 4550 7160
-Wire Wire Line
-	4230 7160 4230 7200
-Wire Wire Line
-	4230 7540 4550 7540
-Wire Wire Line
-	4230 7540 4230 7580
 Wire Wire Line
 	2050 6850 2050 6950
@@
 	1    0    0    -1
 $EndComp
+$Comp
+L power:+3.3V #PWR0617
+U 1 1 5F53B335
+P 3910 7200
+F 0 "#PWR0617" H 3910 7050 50  0001 C CNN
+F 1 "+3.3V" H 3910 7340 50  0000 C CNN
+F 2 "" H 3910 7200 50  0001 C CNN
+F 3 "" H 3910 7200 50  0001 C CNN
+	1    3910 7200
+	1    0    0    -1
+$EndComp
+$Comp
+L power:GND #PWR0618
+U 1 1 5F53B7AC
+P 3910 7500
+F 0 "#PWR0618" H 3910 7250 50  0001 C CNN
+F 1 "GND" H 3910 7350 50  0000 C CNN
+F 2 "" H 3910 7500 50  0001 C CNN
+F 3 "" H 3910 7500 50  0001 C CNN
+	1    3910 7500
+	1    0    0    -1
+$EndComp
