File: hdw/Analog_Clock/Analog_Clock.kicad_pcb (KiCad board)
At the start: 2 copper layers, 417 parts, among them J1301 USB_B_Mini, J201 +12V IN, J2401 I2C, J2402 USB UART, J2403 DAC SPI, J801 PICKIT4, Q1601 BSS214NW, Q2401 BSS214NW, Q401 BSS214NW, Q402 ZXMS6004FFTA, Q601 FDC5612, Q801 BSS214NW, SW2201 Cap_Touch, SW2202 Cap_Touch, SW801 MRST, U1001 PIC32MZ0512EFE064T-I_PT, U1201 DS3231MZ, U1202 TLV6700, U1301 TLV6700, U1302 FT234XD, U1304 TXB0102DCU, U1305 TPD3S014DBVR, U1401 INA219BxDCN, U1402 MCP9804, U1501 DS1683, U1601 74LVC1G06, U1602 74LVC1G06, U1603 LP2985-3.3, U1604 74LVC1G06, U1605 74LVC1G07, U1606 74LVC1G06, U1701 74LVC1G06, U1702 74LVC1G06, U1703 74LVC1G06, U1704 74LVC1G06, U1801 74LVC1G07, U1802 LT1790-2.048, U1803 DAC8551, U1804 OPA2197xDGK, U1901 74LVC1G07, U1902 LT1790-2.048, U1903 DAC8551, U1904 OPA2197xDGK, U2001 74LVC1G07, U2002 LT1790-2.048, U2003 DAC8551, U2004 OPA2197xDGK, U201 TPS26600RHFT, U2101 LP5009, U2201 AT42QT1010-TSHR, U2202 AT42QT1010-TSHR, U2203 74LVC1G17, U2204 74LVC1G17, U2301 74LVC1G06, U2302 74LVC1G06, U2303 74LVC1G06, U2304 74LVC1G06, U2401 LTC6900, U2402 74LVC1G08, U2403 MCP9804, U301 INA219BxDCN, U302 MCP9804, U401 TPS62150, U501 INA219BxDCN, U502 MCP9804, U601 TLV6700, U602 LT3757, U701 INA219BxDCN, U702 MCP9804, X1101 ASE-8.000MHz, X1102 ECS-327KE

Commit message: Board outline
Parts:
- moved C603 275.8 mm to (490.4, 95.4)
- moved C605 275.8 mm to (490.4, 101.3)
- moved R604 275.8 mm to (490.4, 94.0)
- moved R606 275.8 mm to (490.4, 99.8)
- moved R613 275.8 mm to (490.4, 96.8)
- moved R614 275.8 mm to (490.4, 98.3)
- moved C1102 275.8 mm to (355.5, 174.4)
- moved C1104 275.8 mm to (354.2, 174.4)
- moved C1201 275.8 mm to (318.0, 81.4)
- moved C1203 275.8 mm to (307.4, 80.4)
- moved C1204 275.8 mm to (344.8, 90.5)
- moved C1205 275.8 mm to (339.2, 88.2)
- moved C1301 275.8 mm to (320.2, 27.9)
- moved C1303 275.8 mm to (321.9, 19.2)
- moved C1304 275.8 mm to (318.8, 27.9)
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Other:
- board outline added: 200 x 50 mm
