File: hdw/Analog_Clock/Analog_Clock.kicad_pcb (KiCad board)
At the start: 2 copper layers, 200 x 50 mm, 417 parts, among them J1301 USB_B_Mini, J201 +12V IN, J2401 I2C, J2402 USB UART, J2403 DAC SPI, J801 PICKIT4, Q1601 BSS214NW, Q2401 BSS214NW, Q401 BSS214NW, Q402 ZXMS6004FFTA, Q601 FDC5612, Q801 BSS214NW, SW2201 Cap_Touch, SW2202 Cap_Touch, SW801 MRST, U1001 PIC32MZ0512EFE064T-I_PT, U1201 DS3231MZ, U1202 TLV6700, U1301 TLV6700, U1302 FT234XD, U1304 TXB0102DCU, U1305 TPD3S014DBVR, U1401 INA219BxDCN, U1402 MCP9804, U1501 DS1683, U1601 74LVC1G06, U1602 74LVC1G06, U1603 LP2985-3.3, U1604 74LVC1G06, U1605 74LVC1G07, U1606 74LVC1G06, U1701 74LVC1G06, U1702 74LVC1G06, U1703 74LVC1G06, U1704 74LVC1G06, U1801 74LVC1G07, U1802 LT1790-2.048, U1803 DAC8551, U1804 OPA2197xDGK, U1901 74LVC1G07, U1902 LT1790-2.048, U1903 DAC8551, U1904 OPA2197xDGK, U2001 74LVC1G07, U2002 LT1790-2.048, U2003 DAC8551, U2004 OPA2197xDGK, U201 TPS26600RHFT, U2101 LP5009, U2201 AT42QT1010-TSHR, U2202 AT42QT1010-TSHR, U2203 74LVC1G17, U2204 74LVC1G17, U2301 74LVC1G06, U2302 74LVC1G06, U2303 74LVC1G06, U2304 74LVC1G06, U2401 LTC6900, U2402 74LVC1G08, U2403 MCP9804, U301 INA219BxDCN, U302 MCP9804, U401 TPS62150, U501 INA219BxDCN, U502 MCP9804, U601 TLV6700, U602 LT3757, U701 INA219BxDCN, U702 MCP9804, X1101 ASE-8.000MHz, X1102 ECS-327KE

Commit message: more PCB placement
Parts:
- C402, C601, C602, C603, C604, C605, C607, C610, D401, D601, L601, Q601, R401, R403, R601, R602, R603, R604, R605, R606, R607, R608, R609, R610, R611, R612, R613, R614, TP601, U601, U602: moved to B.Cu
- C606, C701, C702, C703, U701, U702: moved to F.Cu
- moved R607 542.7 mm to (-28.5, -39.4), turned to 270 degrees
- moved C606 539.4 mm to (-25.8, -39.4), turned to 0 degrees
- moved U601 539.4 mm to (-25.8, -39.4), turned to 180 degrees
- moved C605 538.5 mm to (-31.1, -33.4), turned to 270 degrees
- moved R603 538.1 mm to (-27.8, -36.2), turned to 270 degrees
- moved R606 536.7 mm to (-29.5, -33.4), turned to 90 degrees
- moved R602 536.3 mm to (-25.8, -36.8), turned to 180 degrees
- moved R614 534.9 mm to (-28.1, -33.4), turned to 90 degrees
- moved R613 533.1 mm to (-26.6, -33.4), turned to 270 degrees
- moved R601 533.1 mm to (-23.7, -36.2), turned to 90 degrees
- moved C603 531.4 mm to (-25.2, -33.4), turned to 90 degrees
- moved C604 529.8 mm to (-29.0, -28.2), turned to 90 degrees
- moved R604 529.7 mm to (-23.7, -33.4), turned to 90 degrees
- moved TP601 529.3 mm to (-20.7, -36.2), turned to 90 degrees
- moved C702 527.7 mm to (-19.2, -36.3), turned to 180 degrees
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Routing:
- net Net-(C201-Pad2): track 1.41 -> 0.00 mm
Other:
- board text added: "DAC0 WRITE"
- board text added: "DAC1 WRITE"
- board text added: "DAC2 WRITE"

Commit message: moar PCB placement
Parts:
- BT1202, C1101, C1102, C1103, C1104, C1105, C1106, C1201, C1202, C1203, C1204, C1205, C1501, C1502, C1503, C1504, C1812, C1912, C2012, C2101, C2102, C2103, C2403, C901, C902, C903, C904, C905, C906, C907, C908, C909, C910, C911, C912, C913, C914, C915, C916, C917, C918, C919, C920, C921, D1501, D1601, D1602, D1603, D1604, D1605, D1701, D1702, D1703, D1704, L1101, L1102, L901, L902, R1103, R1104, R1105, R1201, R1202, R1203, R1604, R1605, R1606, R1607, R1608, R1703, R1704, R1707, R1708, R2101, R2102, SW801, TP1102, TP1201, U1001, U1201, U1202, U1501, U1601, U1602, U1604, U1605, U1606, U1701, U1702, U1703, U1704, U2101, U2403, X1101, X1102: moved to B.Cu
- C1602, C1603, C1605, C1606, C1607, C1701, C1702, C1703, C1704, C801, Q801, R1001, R1002, R1106, R1107, R1601, R1603, R1701, R1702, R1705, R1706, R610, R612, R801, R802, R803, R804, R805: moved to F.Cu
- moved C2403 458.4 mm to (4.52, -15.7), turned to 0 degrees
- moved U2403 457.0 mm to (5.22, -13.7), turned to 180 degrees
- moved U1501 375.8 mm to (5.54, -32.0)
- moved C1504 371.7 mm to (8.59, -27.6), turned to 270 degrees
- moved C1501 371.7 mm to (7.25, -27.6), turned to 270 degrees
- moved C1502 371.7 mm to (4.58, -27.6), turned to 270 degrees
- moved C1503 371.7 mm to (5.92, -27.6), turned to 270 degrees
- moved D1501 371.6 mm to (2.81, -27.5), turned to 270 degrees
- moved C2102 339.4 mm to (99.5, -48.1), turned to 180 degrees
- moved C2103 339.4 mm to (99.5, -46.7), turned to 180 degrees
- moved U2101 335.0 mm to (101.9, -43.7), turned to 180 degrees
- moved R2101 333.1 mm to (102.9, -47.4)
- moved R2102 330.3 mm to (104.4, -47.4)
- moved C2101 327.5 mm to (105.9, -47.4)
- moved L1101 320.8 mm to (129.6, -35.9)
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Other:
- board text added: "+5V USB"
- board text added: "Double check clearance on meter connections and surrounding passives Also double check mounting hole clearance"

Commit message: finished first pass PCB placement
Parts:
- BZ2401, C2401, C2402, J2401, J2402, J2403, R2401, R2403, R2404, R2406, TP201, U2401, U2402: moved to B.Cu
- D2401, Q2401, R2402, R2405, R2407: moved to F.Cu
- moved J2403 159.3 mm to (84.8, 125.9), turned to 180 degrees
- moved C1102 140.1 mm to (174.6, 121.5)
- moved C1104 140.1 mm to (173.3, 121.5)
- moved C1106 140.1 mm to (171.9, 121.5)
- moved C1204 140.1 mm to (111.8, 87.3)
- moved C1205 140.1 mm to (114.0, 92.9)
- moved C1301 140.1 mm to (228.9, 119.9)
- moved C1302 140.1 mm to (220.2, 119.5)
- moved C1304 140.1 mm to (228.9, 121.3)
- moved C1310 140.1 mm to (222.0, 114.1)
- moved C1312 140.1 mm to (226.9, 114.1)
- moved C1401 140.1 mm to (228.3, 116.5)
- moved C1402 140.1 mm to (231.1, 113.2)
- moved C1501 140.1 mm to (46.3, 106.9)
- moved C1502 140.1 mm to (43.6, 106.9)
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Other:
- board text added: "MRST"

Commit message: A lot more PCB work
Routing:
- net Net-(U1803-Pad3): track 0.00 -> 18.0 mm
- net Net-(C1811-Pad1): track 0.00 -> 8.36 mm
- net Net-(R1812-Pad2): track 0.00 -> 7.45 mm
- net Net-(C1811-Pad2): track 0.00 -> 5.16 mm
- net Net-(C1807-Pad1): track 0.00 -> 3.51 mm
- net VDAC_0_ADC: track 0.00 -> 2.80 mm, vias 0 -> 1
- added copper zone on PWR, net +3V3
- added copper zone on GND, net GND
Other:
- copper layers 2 -> 4
- net class Default: clearance 0.2 -> 0.127; trace_width 0.25 -> 0.254; via_dia 0.8 -> 0.4318; via_drill 0.4 -> 0.2
- net class Power added: clearance 0.127, trace_width 0.635, via_dia 0.4318, via_drill 0.2
- net class Signal added: clearance 0.127, trace_width 0.254, via_dia 0.4318, via_drill 0.2
- rule trace_clearance: 0.2 -> 0.127
- rule trace_min: 0.2 -> 0.0508
- rule via_min_drill: 0.3 -> 0.199898
Changed lines of the file:
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@@
     (thickness 1.6)
     (drawings 51)
-    (tracks 0)
+    (tracks 37)
     (zones 0)
     (modules 417)
@@
   (page A)
   (layers
-    (0 F.Cu signal)
-    (31 B.Cu signal)
+    (0 F.Cu mixed)
+    (1 GND mixed)
+    (2 PWR mixed)
+    (31 B.Cu mixed)
     (32 B.Adhes user)
     (33 F.Adhes user)
@@
     (44 Edge.Cuts user)
     (45 Margin user)
-    (46 B.CrtYd user)
-    (47 F.CrtYd user)
+    (46 B.CrtYd user hide)
+    (47 F.CrtYd user hide)
     (48 B.Fab user hide)
     (49 F.Fab user hide)
   )
   (setup
-    (last_trace_width 0.25)
-    (trace_clearance 0.2)
-    (zone_clearance 0.508)
-    (zone_45_only no)
-    (trace_min 0.2)
-    (via_size 0.8)
-    (via_drill 0.4)
+    (last_trace_width 0.254)
+    (trace_clearance 0.127)
+    (zone_clearance 0.254)
+    (zone_45_only yes)
+    (trace_min 0.0508)
+    (via_size 0.4318)
+    (via_drill 0.2)
     (via_min_size 0.4)
-    (via_min_drill 0.3)
+    (via_min_drill 0.199898)
     (uvia_size 0.3)
     (uvia_drill 0.1)
@@
     (uvia_min_size 0.2)
     (uvia_min_drill 0.1)
-    (edge_width 0.05)
+    (edge_width 0.15)
     (segment_width 0.2)
     (pcb_text_width 0.3)
     (pcb_text_size 1.5 1.5)
-    (mod_edge_width 0.12)
+    (mod_edge_width 0.15)
     (mod_text_size 1 1)
     (mod_text_width 0.15)
@@
     (solder_mask_min_width 0.25)
     (aux_axis_origin 0 0)
-    (visible_elements 7FFFF77F)
+    (visible_elements 7FFFF67F)
     (pcbplotparams
       (layerselection 0x010fc_ffffffff)
@@
   (net 244 "Net-(U1402-Pad3)")
   (net_class Default "This is the default net class."
-    (clearance 0.2)
-    (trace_width 0.25)
-    (via_dia 0.8)
-    (via_drill 0.4)
+    (clearance 0.127)
+    (trace_width 0.254)
+    (via_dia 0.4318)
+    (via_drill 0.2)
+    (uvia_dia 0.3)
+    (uvia_drill 0.1)
+    (diff_pair_width 0.254)
+    (diff_pair_gap 0.127)
+  )
+  (net_class Power ""
+    (clearance 0.127)
+    (trace_width 0.635)
+    (via_dia 0.4318)
+    (via_drill 0.2)
     (uvia_dia 0.3)
     (uvia_drill 0.1)
@@
     (add_net +3V3)
     (add_net +5V_USB)
+    (add_net GND)
+    (add_net GNDA_MZ)
+  )
+  (net_class Signal ""
+    (clearance 0.127)
+    (trace_width 0.254)
+    (via_dia 0.4318)
+    (via_drill 0.2)
+    (uvia_dia 0.3)
+    (uvia_drill 0.1)
+    (diff_pair_width 0.254)
+    (diff_pair_gap 0.127)
     (add_net "/USB UART Bridge/BRIDGE_USB+")
     (add_net "/USB UART Bridge/BRIDGE_USB-")
@@
     (add_net Function_Time_LED)
     (add_net Function_Weekday_LED)
-    (add_net GND)
-    (add_net GNDA_MZ)
     (add_net Heartbeat_LED)
     (add_net I2C_SCL)
@@
       (net 25 "Net-(C1102-Pad1)"))
   )
-  (gr_text MRST (at 174.2694 86.4362) (layer B.SilkS)
-    (effects (font (size 1 1) (thickness 0.15)) (justify left mirror))
+  (gr_text MRST (at 179.3748 93.1672) (layer B.SilkS)
+    (effects (font (size 1 1) (thickness 0.15)) (justify mirror))
   )
   (gr_text GND (at 93.2942 89.0524) (layer B.SilkS)
@@
     (effects (font (size 1 1) (thickness 0.15)) (justify mirror))
   )
+  (segment (start 87.2751 114.9858) (end 87.0966 115.1643) (width 0.254) (layer B.Cu) (net 34))
+  (segment (start 88.6326 114.9858) (end 87.2751 114.9858) (width 0.254) (layer B.Cu) (net 34))
+  (segment (start 88.6326 114.0028) (end 89.2781 113.3573) (width 0.254) (layer B.Cu) (net 34))
+  (segment (start 88.6326 114.9858) (end 88.6326 114.0028) (width 0.254) (layer B.Cu) (net 34))
+  (segment (start 95.7281 112.0573) (end 95.8596 111.9258) (width 0.254) (layer B.Cu) (net 36))
+  (segment (start 93.6781 112.0573) (end 95.7281 112.0573) (width 0.254) (layer B.Cu) (net 36))
+  (segment (start 95.8596 111.9258) (end 98.7806 111.9258) (width 0.254) (layer B.Cu) (net 36))
+  (segment (start 92.6991 111.4073) (end 93.6781 111.4073) (width 0.254) (layer B.Cu) (net 37))
+  (segment (start 90.1326 114.9858) (end 90.1326 115.1858) (width 0.254) (layer B.Cu) (net 37))
+  (segment (start 90.1326 115.1858) (end 90.974 116.0272) (width 0.254) (layer B.Cu) (net 37))
+  (segment (start 90.974 116.0272) (end 92.1004 116.0272) (width 0.254) (layer B.Cu) (net 37))
+  (segment (start 92.1004 116.0272) (end 92.3036 115.824) (width 0.254) (layer B.Cu) (net 37))
+  (segment (start 92.3036 115.824) (end 92.3036 111.8028) (width 0.254) (layer B.Cu) (net 37))
+  (segment (start 92.3036 111.8028) (end 92.6991 111.4073) (width 0.254) (layer B.Cu) (net 37))
+  (via (at 94.6404 114.5032) (size 0.4318) (drill 0.2) (layers F.Cu B.Cu) (net 38))
+  (segment (start 93.0536 114.9858) (end 94.1578 114.9858) (width 0.254) (layer B.Cu) (net 38))
+  (segment (start 94.1578 114.9858) (end 94.6404 114.5032) (width 0.254) (layer B.Cu) (net 38))
+  (segment (start 95.6015 114.5032) (end 95.6396 114.5413) (width 0.254) (layer F.Cu) (net 38))
+  (segment (start 94.6404 114.5032) (end 95.6015 114.5032) (width 0.254) (layer F.Cu) (net 38))
+  (segment (start 90.8125 112.7073) (end 89.2781 112.7073) (width 0.254) (layer B.Cu) (net 165))
+  (segment (start 91.5536 114.9858) (end 91.5536 113.4484) (width 0.254) (layer B.Cu) (net 165))
+  (segment (start 91.5536 113.4484) (end 90.8125 112.7073) (width 0.254) (layer B.Cu) (net 165))
+  (segment (start 91.5536 113.4484) (end 91.5536 112.6356) (width 0.254) (layer B.Cu) (net 165))
+  (segment (start 90.9753 112.0573) (end 89.2781 112.0573) (width 0.254) (layer B.Cu) (net 165))
+  (segment (start 91.5536 112.6356) (end 90.9753 112.0573) (width 0.254) (layer B.Cu) (net 165))
+  (segment (start 87.4286 116.9318) (end 86.9286 116.9318) (width 0.254) (layer B.Cu) (net 222))
+  (segment (start 87.9076 116.4528) (end 87.4286 116.9318) (width 0.254) (layer B.Cu) (net 222))
+  (segment (start 92.21363 116.452799) (end 87.9076 116.4528) (width 0.254) (layer B.Cu) (net 222))
+  (segment (start 94.6571 112.7073) (end 95.110301 113.160501) (width 0.254) (layer B.Cu) (net 222))
+  (segment (start 93.6781 112.7073) (end 94.6571 112.7073) (width 0.254) (layer B.Cu) (net 222))
+  (segment (start 95.110301 113.160501) (end 95.110301 114.728753) (width 0.254) (layer B.Cu) (net 222))
+  (segment (start 95.110301 114.728753) (end 94.096755 115.742299) (width 0.254) (layer B.Cu) (net 222))
+  (segment (start 94.096755 115.742299) (end 92.92413 115.742299) (width 0.254) (layer B.Cu) (net 222))
+  (segment (start 92.92413 115.742299) (end 92.21363 116.452799) (width 0.254) (layer B.Cu) (net 222))
+  (segment (start 86.9286 117.5818) (end 88.2598 117.5818) (width 0.254) (layer B.Cu) (net 222))
+  (segment (start 89.388801 116.452799) (end 92.21363 116.452799) (width 0.254) (layer B.Cu) (net 222))
+  (segment (start 88.2598 117.5818) (end 89.388801 116.452799) (width 0.254) (layer B.Cu) (net 222))
+  (zone (net 5) (net_name GND) (layer GND) (hatch edge 0.508)
+    (connect_pads yes (clearance 0.254))
+    (min_thickness 0.254)
+    (fill yes (arc_segments 32) (thermal_gap 0.508) (thermal_bridge_width 0.508) (smoothing fillet) (radius 0.254))
+    (polygon
+      (pts
+        (xy 39.0652 84.5312) (xy 239.0648 84.5312) (xy 239.0648 134.5184) (xy 39.0652 134.5184)
+      )
+    )
+  )
+  (zone (net 1) (net_name +3V3) (layer PWR) (hatch edge 0.508)
+    (connect_pads yes (clearance 0.254))
+    (min_thickness 0.254)
+    (fill yes (arc_segments 32) (thermal_gap 0.508) (thermal_bridge_width 0.508) (smoothing fillet) (radius 0.254))
+    (polygon
+      (pts
+        (xy 39.063881 84.5312) (xy 239.063481 84.5312) (xy 239.063481 134.5184) (xy 39.063881 134.5184)
+      )
+    )
+  )
 )

Commit message: started routing
Parts:
- C1205: moved to F.Cu
- moved C1205 53.8 mm to (165.1, 110.1), turned to 270 degrees
- moved D801 0.38 mm to (162.9, 89.8)
Routing:
- net GND: track 0.00 -> 240.2 mm, vias 0 -> 63
- net +3V3: track 0.00 -> 116.5 mm, vias 0 -> 29
- net ~PIC32MZ_MCLR: track 0.00 -> 32.5 mm, vias 0 -> 1
- net PIC32MZ_ICSPCLK: track 0.00 -> 29.3 mm, vias 0 -> 2
- net VBAT: track 0.00 -> 26.6 mm
- net PIC32MZ_ICSPDAT: track 0.00 -> 25.2 mm
- net +20V: track 0.00 -> 18.6 mm, vias 0 -> 4
- net Net-(U2003-Pad3): track 0.00 -> 18.0 mm
- net Net-(U1903-Pad3): track 0.00 -> 18.0 mm
- net +12Vin: track 0.00 -> 12.9 mm
- net Net-(C2011-Pad1): track 0.00 -> 12.7 mm
- net Net-(C1911-Pad1): track 0.00 -> 12.7 mm
- net Net-(C201-Pad2): track 0.00 -> 11.5 mm, vias 0 -> 6
- net DAC0_VREF: track 0.00 -> 11.0 mm
- net DAC2_VREF: track 0.00 -> 11.0 mm
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- added copper zone on F.Cu, net +12Vin
- added copper zone on PWR, net Net-(C201-Pad2)

Commit message: more routing
Routing:
- net GND: track 240.2 -> 304.5 mm, vias 63 -> 85
- net +3V3: track 116.5 -> 161.1 mm, vias 29 -> 38
- net +3.3V_USB: track 0.00 -> 25.1 mm, vias 0 -> 1
- net Net-(J1301-Pad6): track 0.00 -> 23.3 mm
- net /USB UART Bridge/CONN_USB+: track 0.00 -> 16.7 mm, vias 0 -> 1
- net /USB UART Bridge/CONN_USB-: track 0.00 -> 16.2 mm, vias 0 -> 1
- net USB_UART_TX_BUF: track 0.00 -> 13.8 mm, vias 0 -> 1
- net POS5_USB_SNS+: track 0.00 -> 8.03 mm, vias 0 -> 1
- net Net-(C1501-Pad1): track 0.00 -> 7.72 mm
- net Net-(L1301-Pad2): track 0.00 -> 7.31 mm
- net Net-(R1310-Pad2): track 0.00 -> 7.31 mm
- net POS5_USB_SNS-: track 0.00 -> 7.28 mm, vias 0 -> 1
- net +12Vin: track 12.9 -> 19.9 mm
- net +5V_USB: track 0.00 -> 6.57 mm
- net USB_UART_RX_BUF: track 0.00 -> 5.14 mm, vias 0 -> 2
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- added copper zone on F.Cu, net Net-(R205-Pad2)

Commit message: moar routing
Parts:
- moved C502 9.06 mm to (56.5, 92.1), turned to 180 degrees
- moved U501 7.33 mm to (56.5, 89.6), turned to 180 degrees
- moved L801 4.98 mm to (166.4, 94.7)
- moved L802 4.98 mm to (162.5, 94.7)
- moved C501 3.47 mm to (59.1, 88.9), turned to 270 degrees
- moved C402 0.95 mm to (62.9, 101.5)
- moved R401 0.95 mm to (61.5, 101.5)
Routing:
- net +20V: track 18.6 -> 160.4 mm, vias 4 -> 5
- net GND: track 304.5 -> 354.2 mm, vias 85 -> 104
- net +12V: track 6.78 -> 40.5 mm, vias 0 -> 7
- net ~DAC_SPI_SYNC_0: track 0.00 -> 19.2 mm, vias 0 -> 2
- net ~DAC_SPI_SYNC_2: track 0.00 -> 19.2 mm, vias 0 -> 2
- net ~DAC_SPI_SYNC_1: track 0.00 -> 19.2 mm, vias 0 -> 2
- net +3V3: track 161.1 -> 173.2 mm, vias 38 -> 41
- net +12Vin: track 19.9 -> 27.7 mm
- net POS3P3_RUN: track 0.00 -> 7.26 mm, vias 0 -> 1
- net Net-(J801-Pad3): track 2.71 -> 8.66 mm
- net Net-(D801-Pad3): track 8.91 -> 14.8 mm
- net Net-(R608-Pad2): track 0.00 -> 5.45 mm
- net ~PIC32MZ_MCLR: track 32.5 -> 27.6 mm
- net POS3P3_SNS-: track 3.19 -> 7.94 mm
- net POS3P3_SNS+: track 3.18 -> 7.37 mm
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- added copper zone on B.Cu, net +12V
- added copper zone on F.Cu, net +12V
- added copper zone on F.Cu, net Net-(C405-Pad1)
- added copper zone on B.Cu, net Net-(C610-Pad1)
- added copper zone on B.Cu, net Net-(D601-Pad2)
- added copper zone on F.Cu, net Net-(L401-Pad1)

Commit message: finished routing subcircuits
Parts:
- C1306: moved to B.Cu
- moved R1301 1.62 mm to (228.4, 112.5), turned to 270 degrees
- moved R2302 0.08 mm to (215.9, 90.2)
Routing:
- net GND: track 354.2 -> 463.4 mm, vias 104 -> 131
- net +3V3: track 173.2 -> 243.1 mm, vias 41 -> 63
- net +5V_USB: track 6.57 -> 36.2 mm, vias 0 -> 2
- net POS5_USB_PGOOD: track 3.93 -> 28.7 mm, vias 0 -> 1
- net +3.3V_PGL: track 0.00 -> 22.1 mm, vias 0 -> 6
- net ~USB_ACTIVE: track 0.00 -> 19.9 mm, vias 0 -> 3
- net +20V: track 160.4 -> 175.6 mm, vias 5 -> 6
- net Net-(C1811-Pad1): track 12.7 -> 24.0 mm, vias 0 -> 1
- net ~PIC32MZ_MCLR: track 27.6 -> 37.5 mm
- net Net-(R801-Pad1): track 0.00 -> 9.76 mm
- net Net-(C2011-Pad1): track 12.7 -> 22.0 mm
- net Net-(C1911-Pad1): track 12.7 -> 22.0 mm
- net +12V: track 40.5 -> 49.6 mm, vias 7 -> 8
- net Net-(BZ2401-Pad2): track 0.00 -> 8.23 mm
- net Net-(C801-Pad1): track 0.00 -> 5.41 mm
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- added copper zone on F.Cu, net +3V3
Other:
- board text added: "VBAT LOW"
- board text removed: "VBAT"
