File: hdw/Analog_Clock/Analog_Clock.kicad_pcb (KiCad board)
At the start: 4 copper layers, 200 x 50 mm, 417 parts, among them J1301 USB_B_Mini, J201 +12V IN, J2401 I2C, J2402 USB UART, J2403 DAC SPI, J801 PICKIT4, Q1601 BSS214NW, Q2401 BSS214NW, Q401 BSS214NW, Q402 ZXMS6004FFTA, Q601 FDC5612, Q801 BSS214NW, SW2201 Cap_Touch, SW2202 Cap_Touch, SW801 MRST, U1001 PIC32MZ0512EFE064T-I_PT, U1201 DS3231MZ, U1202 TLV6700, U1301 TLV6700, U1302 FT234XD, U1304 TXB0102DCU, U1305 TPD3S014DBVR, U1401 INA219BxDCN, U1402 MCP9804, U1501 DS1683, U1601 74LVC1G06, U1602 74LVC1G06, U1603 LP2985-3.3, U1604 74LVC1G06, U1605 74LVC1G07, U1606 74LVC1G06, U1701 74LVC1G06, U1702 74LVC1G06, U1703 74LVC1G06, U1704 74LVC1G06, U1801 74LVC1G07, U1802 LT1790-2.048, U1803 DAC8551, U1804 OPA2197xDGK, U1901 74LVC1G07, U1902 LT1790-2.048, U1903 DAC8551, U1904 OPA2197xDGK, U2001 74LVC1G07, U2002 LT1790-2.048, U2003 DAC8551, U2004 OPA2197xDGK, U201 TPS26600RHFT, U2101 LP5009, U2201 AT42QT1010-TSHR, U2202 AT42QT1010-TSHR, U2203 74LVC1G17, U2204 74LVC1G17, U2301 74LVC1G06, U2302 74LVC1G06, U2303 74LVC1G06, U2304 74LVC1G06, U2401 LTC6900, U2402 74LVC1G08, U2403 MCP9804, U301 INA219BxDCN, U302 MCP9804, U401 TPS62150, U501 INA219BxDCN, U502 MCP9804, U601 TLV6700, U602 LT3757, U701 INA219BxDCN, U702 MCP9804, X1101 ASE-8.000MHz, X1102 ECS-327KE

Commit message: autorouting, cleanups
Routing:
- net I2C_SCL: track 2.31 -> 375.6 mm, vias 1 -> 14
- net I2C_SDA: track 4.62 -> 373.3 mm, vias 1 -> 14
- net POS3P3_PGOOD: track 4.15 -> 241.5 mm, vias 0 -> 9
- net POS12_PGOOD: track 6.67 -> 229.3 mm, vias 0 -> 6
- net POS20_PGOOD: track 3.88 -> 224.5 mm, vias 0 -> 4
- net +12V: track 49.6 -> 241.2 mm, vias 8 -> 15
- net VBAT_PGOOD: track 1.80 -> 186.0 mm, vias 0 -> 4
- net DAC_SPI_SCLK: track 0.00 -> 148.2 mm, vias 0 -> 9
- net DAC_SPI_MOSI: track 0.00 -> 144.9 mm, vias 0 -> 2
- net Cap_Touch_Function: track 4.02 -> 137.6 mm, vias 0 -> 1
- net Cap_Touch_Power: track 4.32 -> 131.9 mm, vias 0 -> 7
- net POS20_RUN: track 3.35 -> 119.7 mm, vias 0 -> 3
- net USB_UART_RX: track 1.81 -> 92.8 mm, vias 1 -> 5
- net POS3P3_PGL_SHDN: track 0.00 -> 89.6 mm, vias 0 -> 3
- net DAC0_VREF: track 11.0 -> 100.2 mm, vias 0 -> 2
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
Commit message: Added BOM
Parts:
- added G***: Microchip_Logo, Custom Footprints Library:Microchip_Logo, B.Cu at (163.8, 111.6)
- added G***: Owl_1_Logo, Custom Footprints Library:Owl_1_Logo, B.Cu at (217.7, 102.4)
- added G***: PIC32_Logo, Custom Footprints Library:PIC32_Logo, B.Cu at (160.4, 97.1)
- added REF**: KiCAD Logo, Symbols:Symbol_KiCAD-Logo_CopperAndSilkScreenTop, B.Cu at (81.0, 91.2)
- added REF**: Symbol_Barrel_Polarity, Symbol:Symbol_Barrel_Polarity, F.Cu at (64.0, 129.9)
- added REF***: ESD-Logo_6.6x6mm_SilkScreen, Symbols:ESD-Logo_6.6x6mm_SilkScreen, B.Cu at (149.5, 91.8)
Routing:
- net Net-(U1803-Pad3): track 18.0 -> 15.2 mm
- net METER0_LED_R: track 65.5 -> 68.1 mm
- net METER0_LED_B: track 60.6 -> 62.2 mm
- net METER2_LED_B: track 55.6 -> 56.8 mm
- net METER0_LED_G: track 62.0 -> 63.1 mm
- net METER2_LED_G: track 60.8 -> 61.4 mm
Other:
- board text added: "1"
- board text added: "2"
- board text added: "3"
- board text added: "4"
- board text added: "Analog Clock Rev A - October, 2020"
- board text added: "CR1616"
- board text added: "JLCJLCJLCJLC"
- board text removed: "Double check clearance on meter connections and surrounding passives Also double check mounting hole clearance"
